Commit message: new naming fixed

File: src/rviz_basic/urdf/moonbot.urdf (robot description, URDF)
Before this commit: robot Moonbot1, 14 links, 13 joints
Links:
- link BODY: geometry collision mesh filename=package://rviz_basic/base_link.STL; visual mesh filename=package://rviz_basic/base_link.STL
- link Leg1_Link1: geometry collision mesh filename=package://rviz_basic/Leg1_Link1.STL; visual mesh filename=package://rviz_basic/Leg1_Link1.STL
- link Leg1_Link2: geometry collision mesh filename=package://rviz_basic/Leg1_Link2.STL; visual mesh filename=package://rviz_basic/Leg1_Link2.STL
- link Leg1_Link3: geometry collision mesh filename=package://rviz_basic/Leg1_Link3.STL; visual mesh filename=package://rviz_basic/Leg1_Link3.STL
- link Leg2_Link1: geometry collision mesh filename=package://rviz_basic/Leg2_Link1.STL; visual mesh filename=package://rviz_basic/Leg2_Link1.STL
- link Leg2_Link2: geometry collision mesh filename=package://rviz_basic/Leg2_Link2.STL; visual mesh filename=package://rviz_basic/Leg2_Link2.STL
- link Leg2_Link3: geometry collision mesh filename=package://rviz_basic/Leg2_Link3.STL; visual mesh filename=package://rviz_basic/Leg2_Link3.STL
- link Leg3_Link1: geometry collision mesh filename=package://rviz_basic/Leg3_Link1.STL; visual mesh filename=package://rviz_basic/Leg3_Link1.STL
- link Leg3_Link2: geometry collision mesh filename=package://rviz_basic/Leg3_Link2.STL; visual mesh filename=package://rviz_basic/Leg3_Link2.STL
- link Leg3_Link3: geometry collision mesh filename=package://rviz_basic/Leg3_Link3.STL; visual mesh filename=package://rviz_basic/Leg3_Link3.STL
- link Leg4_Link1: geometry collision mesh filename=package://rviz_basic/Leg4_Link1.STL; visual mesh filename=package://rviz_basic/Leg4_Link1.STL
- link Leg4_Link2: geometry collision mesh filename=package://rviz_basic/Leg4_Link2.STL; visual mesh filename=package://rviz_basic/Leg4_Link2.STL
- link Leg4_Link3: geometry collision mesh filename=package://rviz_basic/Leg4_Link3.STL; visual mesh filename=package://rviz_basic/Leg4_Link3.STL

Commit message: rviz with robot body movements

File: src/rviz_basic/urdf/moonbot.urdf (robot description, URDF)
Before this commit: robot Moonbot1, 14 links, 13 joints
Links:
- removed link base_link
- link BODY: mass 1.7613 -> None
Joints:
- removed joint moonbot_attachment

Commit message: body movements working

File: src/rviz_basic/urdf/moonbot.urdf (robot description, URDF)
Before this commit: robot Moonbot1, 13 links, 12 joints
Links:
- added link base_link
Joints:
- added joint moonbot_attachment: type fixed, parent base_link, child BODY, origin xyz=0 0 0 rpy=0 0 2.35619449
