Commit message: bash fix and moonbot2 trails

File: src/rviz_basic/urdf/moonbot2.urdf (robot description, URDF)
Before this commit: robot Moonbot_1_urdf, 13 links, 12 joints
Links:
- removed link Leg1_Link1
- removed link Leg1_Link2
- removed link Leg1_Link3
- removed link Leg2_Link1
- removed link Leg2_Link2
- removed link Leg2_Link3
- removed link Leg3_Link1
- removed link Leg3_Link2
- removed link Leg3_Link3
- removed link Leg4_Link1
- removed link Leg4_Link2
- removed link Leg4_Link3
- added link Body_connector_5, mass 1.00227146305622; collision mesh filename=package://rviz_basic/meshes/Body_connector_5.stl scale=0.001 0.001 0.001; visual mesh filename=package://rviz_basic/meshes/Body_connector_5.stl scale=0.001 0.001 0.001
- added link Body_connector__2__1, mass 1.00227146305622; collision mesh filename=package://rviz_basic/meshes/Body_connector__2__1.stl scale=0.001 0.001 0.001; visual mesh filename=package://rviz_basic/meshes/Body_connector__2__1.stl scale=0.001 0.001 0.001
- added link Body_connector__3__1, mass 1.00227146305622; collision mesh filename=package://rviz_basic/meshes/Body_connector__3__1.stl scale=0.001 0.001 0.001; visual mesh filename=package://rviz_basic/meshes/Body_connector__3__1.stl scale=0.001 0.001 0.001
- added link Connector4_1, mass 0.41151751450909346; collision mesh filename=package://rviz_basic/meshes/Connector4_1.stl scale=0.001 0.001 0.001; visual mesh filename=package://rviz_basic/meshes/Connector4_1.stl scale=0.001 0.001 0.001
- added link Limb0Connector1_1, mass 0.41151751450909346; collision mesh filename=package://rviz_basic/meshes/Limb0Connector1_1.stl scale=0.001 0.001 0.001; visual mesh filename=package://rviz_basic/meshes/Limb0Connector1_1.stl scale=0.001 0.001 0.001
- added link Limb0Connector1__1__1, mass 0.41151751450909346; collision mesh filename=package://rviz_basic/meshes/Limb0Connector1__1__1.stl scale=0.001 0.001 0.001; visual mesh filename=package://rviz_basic/meshes/Limb0Connector1__1__1.stl scale=0.001 0.001 0.001
- added link Limb0Connector2_2, mass 0.028818583393616055; collision mesh filename=package://rviz_basic/meshes/Limb0Connector2_2.stl scale=0.001 0.001 0.001; visual mesh filename=package://rviz_basic/meshes/Limb0Connector2_2.stl scale=0.001 0.001 0.001
- added link Limb0Connector2__1__1, mass 0.028818583393616055; collision mesh filename=package://rviz_basic/meshes/Limb0Connector2__1__1.stl scale=0.001 0.001 0.001; visual mesh filename=package://rviz_basic/meshes/Limb0Connector2__1__1.stl scale=0.001 0.001 0.001
- added link Limb0Connector3_3, mass 0.028067093486926365; collision mesh filename=package://rviz_basic/meshes/Limb0Connector3_3.stl scale=0.001 0.001 0.001; visual mesh filename=package://rviz_basic/meshes/Limb0Connector3_3.stl scale=0.001 0.001 0.001
- added link Limb0Connector3__1__1, mass 0.028067093486926365; collision mesh filename=package://rviz_basic/meshes/Limb0Connector3__1__1.stl scale=0.001 0.001 0.001; visual mesh filename=package://rviz_basic/meshes/Limb0Connector3__1__1.stl scale=0.001 0.001 0.001
- added link Limb0Pitch1A_2, mass 3.3477117479193077; collision mesh filename=package://rviz_basic/meshes/Limb0Pitch1A_2.stl scale=0.001 0.001 0.001; visual mesh filename=package://rviz_basic/meshes/Limb0Pitch1A_2.stl scale=0.001 0.001 0.001
- added link Limb0Pitch1A__1__1, mass 3.3477117479193077; collision mesh filename=package://rviz_basic/meshes/Limb0Pitch1A__1__1.stl scale=0.001 0.001 0.001; visual mesh filename=package://rviz_basic/meshes/Limb0Pitch1A__1__1.stl scale=0.001 0.001 0.001
- added link Limb0Pitch1B_2, mass 0.7729993259283914; collision mesh filename=package://rviz_basic/meshes/Limb0Pitch1B_2.stl scale=0.001 0.001 0.001; visual mesh filename=package://rviz_basic/meshes/Limb0Pitch1B_2.stl scale=0.001 0.001 0.001
- added link Limb0Pitch1B__1__1, mass 0.7729993259283914; collision mesh filename=package://rviz_basic/meshes/Limb0Pitch1B__1__1.stl scale=0.001 0.001 0.001; visual mesh filename=package://rviz_basic/meshes/Limb0Pitch1B__1__1.stl scale=0.001 0.001 0.001
- added link Limb0Pitch2A_2, mass 0.18660217560053788; collision mesh filename=package://rviz_basic/meshes/Limb0Pitch2A_2.stl scale=0.001 0.001 0.001; visual mesh filename=package://rviz_basic/meshes/Limb0Pitch2A_2.stl scale=0.001 0.001 0.001
- added link Limb0Pitch2A__1__1, mass 0.18660217560053788; collision mesh filename=package://rviz_basic/meshes/Limb0Pitch2A__1__1.stl scale=0.001 0.001 0.001; visual mesh filename=package://rviz_basic/meshes/Limb0Pitch2A__1__1.stl scale=0.001 0.001 0.001
- added link Limb0Pitch3A_2, mass 0.07127174173566476; collision mesh filename=package://rviz_basic/meshes/Limb0Pitch3A_2.stl scale=0.001 0.001 0.001; visual mesh filename=package://rviz_basic/meshes/Limb0Pitch3A_2.stl scale=0.001 0.001 0.001
- added link Limb0Pitch3A__1__1, mass 0.07127174173566476; collision mesh filename=package://rviz_basic/meshes/Limb0Pitch3A__1__1.stl scale=0.001 0.001 0.001; visual mesh filename=package://rviz_basic/meshes/Limb0Pitch3A__1__1.stl scale=0.001 0.001 0.001
- added link Limb0Pitch3B_2, mass 0.07127174173566476; collision mesh filename=package://rviz_basic/meshes/Limb0Pitch3B_2.stl scale=0.001 0.001 0.001; visual mesh filename=package://rviz_basic/meshes/Limb0Pitch3B_2.stl scale=0.001 0.001 0.001
- added link Limb0Pitch3B__1__1, mass 0.07127174173566476; collision mesh filename=package://rviz_basic/meshes/Limb0Pitch3B__1__1.stl scale=0.001 0.001 0.001; visual mesh filename=package://rviz_basic/meshes/Limb0Pitch3B__1__1.stl scale=0.001 0.001 0.001
- added link Limb0Roll1A_2, mass 0.8458457350592995; collision mesh filename=package://rviz_basic/meshes/Limb0Roll1A_2.stl scale=0.001 0.001 0.001; visual mesh filename=package://rviz_basic/meshes/Limb0Roll1A_2.stl scale=0.001 0.001 0.001
- added link Limb0Roll1A__1__1, mass 0.8458457350592995; collision mesh filename=package://rviz_basic/meshes/Limb0Roll1A__1__1.stl scale=0.001 0.001 0.001; visual mesh filename=package://rviz_basic/meshes/Limb0Roll1A__1__1.stl scale=0.001 0.001 0.001
- added link Limb0Roll1B_2, mass 0.1621742617893587; collision mesh filename=package://rviz_basic/meshes/Limb0Roll1B_2.stl scale=0.001 0.001 0.001; visual mesh filename=package://rviz_basic/meshes/Limb0Roll1B_2.stl scale=0.001 0.001 0.001
- added link Limb0Roll1B__1__1, mass 0.1621742617893587; collision mesh filename=package://rviz_basic/meshes/Limb0Roll1B__1__1.stl scale=0.001 0.001 0.001; visual mesh filename=package://rviz_basic/meshes/Limb0Roll1B__1__1.stl scale=0.001 0.001 0.001
- added link Limb0Roll2A_3, mass 0.09449902324417689; collision mesh filename=package://rviz_basic/meshes/Limb0Roll2A_3.stl scale=0.001 0.001 0.001; visual mesh filename=package://rviz_basic/meshes/Limb0Roll2A_3.stl scale=0.001 0.001 0.001
- added link Limb0Roll2A__1__1, mass 0.09449902324417689; collision mesh filename=package://rviz_basic/meshes/Limb0Roll2A__1__1.stl scale=0.001 0.001 0.001; visual mesh filename=package://rviz_basic/meshes/Limb0Roll2A__1__1.stl scale=0.001 0.001 0.001
- added link Limb0Roll2B_2, mass 0.14254348347132964; collision mesh filename=package://rviz_basic/meshes/Limb0Roll2B_2.stl scale=0.001 0.001 0.001; visual mesh filename=package://rviz_basic/meshes/Limb0Roll2B_2.stl scale=0.001 0.001 0.001
- added link Limb0Roll2B__1__1, mass 0.14254348347132964; collision mesh filename=package://rviz_basic/meshes/Limb0Roll2B__1__1.stl scale=0.001 0.001 0.001; visual mesh filename=package://rviz_basic/meshes/Limb0Roll2B__1__1.stl scale=0.001 0.001 0.001
- added link Limb0Roll2C_2, mass 5.5447698039525; collision mesh filename=package://rviz_basic/meshes/Limb0Roll2C_2.stl scale=0.001 0.001 0.001; visual mesh filename=package://rviz_basic/meshes/Limb0Roll2C_2.stl scale=0.001 0.001 0.001
- added link Limb0Roll2C__1__1, mass 5.5447698039525; collision mesh filename=package://rviz_basic/meshes/Limb0Roll2C__1__1.stl scale=0.001 0.001 0.001; visual mesh filename=package://rviz_basic/meshes/Limb0Roll2C__1__1.stl scale=0.001 0.001 0.001
- added link Limb0Roll3A_2, mass 2.8490901932138626; collision mesh filename=package://rviz_basic/meshes/Limb0Roll3A_2.stl scale=0.001 0.001 0.001; visual mesh filename=package://rviz_basic/meshes/Limb0Roll3A_2.stl scale=0.001 0.001 0.001
- added link Limb0Roll3A__1__1, mass 2.8490901932138626; collision mesh filename=package://rviz_basic/meshes/Limb0Roll3A__1__1.stl scale=0.001 0.001 0.001; visual mesh filename=package://rviz_basic/meshes/Limb0Roll3A__1__1.stl scale=0.001 0.001 0.001
- added link Limb0Roll3B_2, mass 0.28508696694265934; collision mesh filename=package://rviz_basic/meshes/Limb0Roll3B_2.stl scale=0.001 0.001 0.001; visual mesh filename=package://rviz_basic/meshes/Limb0Roll3B_2.stl scale=0.001 0.001 0.001
- added link Limb0Roll3B__1__1, mass 0.28508696694265934; collision mesh filename=package://rviz_basic/meshes/Limb0Roll3B__1__1.stl scale=0.001 0.001 0.001; visual mesh filename=package://rviz_basic/meshes/Limb0Roll3B__1__1.stl scale=0.001 0.001 0.001
- added link Limb0Wheel_1, mass 20.629366559155358; collision mesh filename=package://rviz_basic/meshes/Limb0Wheel_1.stl scale=0.001 0.001 0.001; visual mesh filename=package://rviz_basic/meshes/Limb0Wheel_1.stl scale=0.001 0.001 0.001
- added link Limb1Connector1_1, mass 0.41151751450909346; collision mesh filename=package://rviz_basic/meshes/Limb1Connector1_1.stl scale=0.001 0.001 0.001; visual mesh filename=package://rviz_basic/meshes/Limb1Connector1_1.stl scale=0.001 0.001 0.001
- added link Limb1Connector2_1, mass 0.028818583393616055; collision mesh filename=package://rviz_basic/meshes/Limb1Connector2_1.stl scale=0.001 0.001 0.001; visual mesh filename=package://rviz_basic/meshes/Limb1Connector2_1.stl scale=0.001 0.001 0.001
- added link Limb1Connector3_1, mass 0.028067093486926365; collision mesh filename=package://rviz_basic/meshes/Limb1Connector3_1.stl scale=0.001 0.001 0.001; visual mesh filename=package://rviz_basic/meshes/Limb1Connector3_1.stl scale=0.001 0.001 0.001
- added link Limb1Pitch1A_1, mass 3.3477117479193077; collision mesh filename=package://rviz_basic/meshes/Limb1Pitch1A_1.stl scale=0.001 0.001 0.001; visual mesh filename=package://rviz_basic/meshes/Limb1Pitch1A_1.stl scale=0.001 0.001 0.001
- added link Limb1Pitch1B_1, mass 0.7729993259283914; collision mesh filename=package://rviz_basic/meshes/Limb1Pitch1B_1.stl scale=0.001 0.001 0.001; visual mesh filename=package://rviz_basic/meshes/Limb1Pitch1B_1.stl scale=0.001 0.001 0.001
- added link Limb1Pitch2A_1, mass 0.18660217560053788; collision mesh filename=package://rviz_basic/meshes/Limb1Pitch2A_1.stl scale=0.001 0.001 0.001; visual mesh filename=package://rviz_basic/meshes/Limb1Pitch2A_1.stl scale=0.001 0.001 0.001
- added link Limb1Pitch3A_1, mass 0.07127174173566476; collision mesh filename=package://rviz_basic/meshes/Limb1Pitch3A_1.stl scale=0.001 0.001 0.001; visual mesh filename=package://rviz_basic/meshes/Limb1Pitch3A_1.stl scale=0.001 0.001 0.001
- added link Limb1Pitch3B_1, mass 0.07127174173566476; collision mesh filename=package://rviz_basic/meshes/Limb1Pitch3B_1.stl scale=0.001 0.001 0.001; visual mesh filename=package://rviz_basic/meshes/Limb1Pitch3B_1.stl scale=0.001 0.001 0.001
- added link Limb1Roll1A_1, mass 0.8458457350592995; collision mesh filename=package://rviz_basic/meshes/Limb1Roll1A_1.stl scale=0.001 0.001 0.001; visual mesh filename=package://rviz_basic/meshes/Limb1Roll1A_1.stl scale=0.001 0.001 0.001
- added link Limb1Roll1B_1, mass 0.1621742617893587; collision mesh filename=package://rviz_basic/meshes/Limb1Roll1B_1.stl scale=0.001 0.001 0.001; visual mesh filename=package://rviz_basic/meshes/Limb1Roll1B_1.stl scale=0.001 0.001 0.001
- added link Limb1Roll2A_1, mass 0.09449902324417689; collision mesh filename=package://rviz_basic/meshes/Limb1Roll2A_1.stl scale=0.001 0.001 0.001; visual mesh filename=package://rviz_basic/meshes/Limb1Roll2A_1.stl scale=0.001 0.001 0.001
- added link Limb1Roll2B_1, mass 0.14254348347132964; collision mesh filename=package://rviz_basic/meshes/Limb1Roll2B_1.stl scale=0.001 0.001 0.001; visual mesh filename=package://rviz_basic/meshes/Limb1Roll2B_1.stl scale=0.001 0.001 0.001
- added link Limb1Roll3A_1, mass 2.8490901932138626; collision mesh filename=package://rviz_basic/meshes/Limb1Roll3A_1.stl scale=0.001 0.001 0.001; visual mesh filename=package://rviz_basic/meshes/Limb1Roll3A_1.stl scale=0.001 0.001 0.001
- added link Limb1Roll3B_1, mass 0.28508696694265934; collision mesh filename=package://rviz_basic/meshes/Limb1Roll3B_1.stl scale=0.001 0.001 0.001; visual mesh filename=package://rviz_basic/meshes/Limb1Roll3B_1.stl scale=0.001 0.001 0.001
- added link Limb1Wheel_1, mass 20.629366559155358; collision mesh filename=package://rviz_basic/meshes/Limb1Wheel_1.stl scale=0.001 0.001 0.001; visual mesh filename=package://rviz_basic/meshes/Limb1Wheel_1.stl scale=0.001 0.001 0.001
- added link Limb2Wheel_1, mass 20.629366559155358; collision mesh filename=package://rviz_basic/meshes/Limb2Wheel_1.stl scale=0.001 0.001 0.001; visual mesh filename=package://rviz_basic/meshes/Limb2Wheel_1.stl scale=0.001 0.001 0.001
- added link Limb3BodyConnector_1, mass 1.00227146305622; collision mesh filename=package://rviz_basic/meshes/Limb3BodyConnector_1.stl scale=0.001 0.001 0.001; visual mesh filename=package://rviz_basic/meshes/Limb3BodyConnector_1.stl scale=0.001 0.001 0.001
- added link Limb3Connector2_1, mass 0.028818583393616055; collision mesh filename=package://rviz_basic/meshes/Limb3Connector2_1.stl scale=0.001 0.001 0.001; visual mesh filename=package://rviz_basic/meshes/Limb3Connector2_1.stl scale=0.001 0.001 0.001
- added link Limb3Connector3_1, mass 0.028067093486926365; collision mesh filename=package://rviz_basic/meshes/Limb3Connector3_1.stl scale=0.001 0.001 0.001; visual mesh filename=package://rviz_basic/meshes/Limb3Connector3_1.stl scale=0.001 0.001 0.001
- added link Limb3Pitch1A_1, mass 3.3477117479193077; collision mesh filename=package://rviz_basic/meshes/Limb3Pitch1A_1.stl scale=0.001 0.001 0.001; visual mesh filename=package://rviz_basic/meshes/Limb3Pitch1A_1.stl scale=0.001 0.001 0.001
- added link Limb3Pitch1B_1, mass 0.7729993259283914; collision mesh filename=package://rviz_basic/meshes/Limb3Pitch1B_1.stl scale=0.001 0.001 0.001; visual mesh filename=package://rviz_basic/meshes/Limb3Pitch1B_1.stl scale=0.001 0.001 0.001
- added link Limb3Pitch2A_1, mass 0.18660217560053788; collision mesh filename=package://rviz_basic/meshes/Limb3Pitch2A_1.stl scale=0.001 0.001 0.001; visual mesh filename=package://rviz_basic/meshes/Limb3Pitch2A_1.stl scale=0.001 0.001 0.001
- added link Limb3Pitch3A_1, mass 0.07127174173566476; collision mesh filename=package://rviz_basic/meshes/Limb3Pitch3A_1.stl scale=0.001 0.001 0.001; visual mesh filename=package://rviz_basic/meshes/Limb3Pitch3A_1.stl scale=0.001 0.001 0.001
- added link Limb3Pitch3B_1, mass 0.07127174173566476; collision mesh filename=package://rviz_basic/meshes/Limb3Pitch3B_1.stl scale=0.001 0.001 0.001; visual mesh filename=package://rviz_basic/meshes/Limb3Pitch3B_1.stl scale=0.001 0.001 0.001
- added link Limb3Roll1A_1, mass 0.8458457350592995; collision mesh filename=package://rviz_basic/meshes/Limb3Roll1A_1.stl scale=0.001 0.001 0.001; visual mesh filename=package://rviz_basic/meshes/Limb3Roll1A_1.stl scale=0.001 0.001 0.001
- added link Limb3Roll1B_1, mass 0.1621742617893587; collision mesh filename=package://rviz_basic/meshes/Limb3Roll1B_1.stl scale=0.001 0.001 0.001; visual mesh filename=package://rviz_basic/meshes/Limb3Roll1B_1.stl scale=0.001 0.001 0.001
- added link Limb3Roll2A_1, mass 0.09449902324417689; collision mesh filename=package://rviz_basic/meshes/Limb3Roll2A_1.stl scale=0.001 0.001 0.001; visual mesh filename=package://rviz_basic/meshes/Limb3Roll2A_1.stl scale=0.001 0.001 0.001
- added link Limb3Roll2B_1, mass 0.14254348347132964; collision mesh filename=package://rviz_basic/meshes/Limb3Roll2B_1.stl scale=0.001 0.001 0.001; visual mesh filename=package://rviz_basic/meshes/Limb3Roll2B_1.stl scale=0.001 0.001 0.001
- added link Limb3Roll2C_1, mass 5.5447698039525; collision mesh filename=package://rviz_basic/meshes/Limb3Roll2C_1.stl scale=0.001 0.001 0.001; visual mesh filename=package://rviz_basic/meshes/Limb3Roll2C_1.stl scale=0.001 0.001 0.001
- added link Limb3Roll3A_1, mass 2.8490901932138626; collision mesh filename=package://rviz_basic/meshes/Limb3Roll3A_1.stl scale=0.001 0.001 0.001; visual mesh filename=package://rviz_basic/meshes/Limb3Roll3A_1.stl scale=0.001 0.001 0.001
- added link Limb3Roll3B_1, mass 0.28508696694265934; collision mesh filename=package://rviz_basic/meshes/Limb3Roll3B_1.stl scale=0.001 0.001 0.001; visual mesh filename=package://rviz_basic/meshes/Limb3Roll3B_1.stl scale=0.001 0.001 0.001
- added link Limb3Wheel_1, mass 20.629366559155358; collision mesh filename=package://rviz_basic/meshes/Limb3Wheel_1.stl scale=0.001 0.001 0.001; visual mesh filename=package://rviz_basic/meshes/Limb3Wheel_1.stl scale=0.001 0.001 0.001
- added link LimbRoll2C__1__1, mass 5.5447698039525; collision mesh filename=package://rviz_basic/meshes/LimbRoll2C__1__1.stl scale=0.001 0.001 0.001; visual mesh filename=package://rviz_basic/meshes/LimbRoll2C__1__1.stl scale=0.001 0.001 0.001
- link base_link: mass 1.7613 -> 83.58553795695674; geometry collision mesh filename=package://rviz_basic/meshes/base_link.stl scale=0.001 0.001 0.001; visual mesh filename=package://rviz_basic/meshes/base_link.stl scale=0.001 0.001 0.001
Joints:
- removed joint LEg4_Joint2
- removed joint Leg1_Joint1
- removed joint Leg1_Joint2
- removed joint Leg1_Joint3
- removed joint Leg2_Joint1
- removed joint Leg2_Joint2
- removed joint Leg2_joint3
- removed joint Leg3_Joint1
- removed joint Leg3_Joint2
- removed joint Leg3_Joint3
- removed joint Leg4_Joint1
- removed joint Leg4_Joint3
- added joint Limb0Pitch1: type continuous, parent Limb0Pitch1A_2, child Limb0Pitch1B_2, origin xyz=0.034163 -0.034169 -0.043437 rpy=0 0 0, axis 0.527675 0.818143 -0.228478
- added joint Limb0Pitch2: type continuous, parent Limb0Pitch1B_2, child Limb0Pitch2A_2, origin xyz=0.097284 -0.097284 -0.123679 rpy=0 0 0, axis 0.527675 0.818143 -0.228478
- added joint Limb0Pitch3: type continuous, parent Limb0Pitch3A_2, child Limb0Pitch3B_2, origin xyz=0.001594 0.00191 -0.000248 rpy=0 0 0, axis 0.637539 0.763972 -0.09945
- added joint Limb0Roll1: type continuous, parent Limb0Roll1A_2, child Limb0Roll1B_2, origin xyz=0.013673 -0.013672 -0.017382 rpy=0 0 0, axis 0.52586 -0.52586 -0.668537
- added joint Limb0Roll2: type continuous, parent Limb0Roll2A_3, child Limb0Roll2B_2, origin xyz=0.013147 -0.013146 -0.016714 rpy=0 0 0, axis -0.52586 0.52586 0.668537
- added joint Limb0Roll3: type continuous, parent Limb0Roll3A_2, child Limb0Roll3B_2, origin xyz=0.052911 0.017165 -0.031713 rpy=0 0 0, axis 0.52586 -0.52586 -0.668537
- added joint Limb1Pitch1: type continuous, parent Limb1Pitch1A_1, child Limb1Pitch1B_1, origin xyz=0.034168 0.034164 -0.043438 rpy=0 0 0, axis -0.713693 0.70038 -0.010471
- added joint Limb1Pitch2: type continuous, parent Limb1Pitch1B_1, child Limb1Pitch2A_1, origin xyz=0.097284 0.097284 -0.123679 rpy=0 0 0, axis 0.713693 -0.70038 0.010471
- added joint Limb1Roll2: type continuous, parent Limb1Roll2A_1, child Limb1Roll2B_1, origin xyz=0.013147 0.013146 -0.016714 rpy=0 0 0, axis 0.52586 0.52586 -0.668537
- added joint Limb2Pitch1: type continuous, parent Limb0Pitch1A__1__1, child Limb0Pitch1B__1__1, origin xyz=-0.034163 0.034168 -0.043437 rpy=0 0 0, axis -0.70038 -0.713693 -0.010471
- added joint Limb2Pitch2: type continuous, parent Limb0Pitch1B__1__1, child Limb0Pitch2A__1__1, origin xyz=-0.097284 0.097284 -0.12368 rpy=0 0 0, axis -0.70038 -0.713693 -0.010471
- added joint Limb2Pitch3: type continuous, parent Limb0Pitch3A__1__1, child Limb0Pitch3B__1__1, origin xyz=-0.001751 -0.001784 -2.6e-05 rpy=0 0 0, axis -0.70038 -0.713693 -0.010471
- added joint Limb2Roll1: type continuous, parent Limb0Roll1A__1__1, child Limb0Roll1B__1__1, origin xyz=-0.013672 0.013672 -0.017382 rpy=0 0 0, axis -0.52586 0.52586 -0.668537
- added joint Limb2Roll2: type continuous, parent Limb0Roll2A__1__1, child Limb0Roll2B__1__1, origin xyz=-0.013146 0.013147 -0.016713 rpy=0 0 0, axis -0.52586 0.52586 -0.668537
- added joint Limb2Roll3: type continuous, parent Limb0Roll3A__1__1, child Limb0Roll3B__1__1, origin xyz=-0.056052 -0.014651 -0.027264 rpy=0 0 0, axis -0.52586 0.52586 -0.668537
- added joint Limb3Pitch1: type continuous, parent Limb3Pitch1A_1, child Limb3Pitch1B_1, origin xyz=-0.034165 -0.034169 -0.043435 rpy=0 0 0, axis -0.713693 0.70038 0.010471
- added joint Limb3Pitch2: type continuous, parent Limb3Pitch1B_1, child Limb3Pitch2A_1, origin xyz=-0.097284 -0.097284 -0.123679 rpy=0 0 0, axis -0.713693 0.70038 0.010471
- added joint Limb3Pitch3: type continuous, parent Limb3Pitch3A_1, child Limb3Pitch3B_1, origin xyz=0.001784 -0.001751 -2.6e-05 rpy=0 0 0, axis 0.713693 -0.70038 -0.010471
- added joint Limb3Roll1: type continuous, parent Limb3Roll1A_1, child Limb3Roll1B_1, origin xyz=-0.013673 -0.013672 -0.017382 rpy=0 0 0, axis -0.52586 -0.52586 -0.668537
- added joint Limb3Roll2: type continuous, parent Limb3Roll2A_1, child Limb3Roll2B_1, origin xyz=-0.013146 -0.013147 -0.016714 rpy=0 0 0, axis -0.52586 -0.52586 -0.668537
- added joint Limb3Roll3: type continuous, parent Limb3Roll3A_1, child Limb3Roll3B_1, origin xyz=0.014651 -0.056052 -0.027264 rpy=0 0 0, axis -0.52586 -0.52586 -0.668537
- added joint Revolute 53: type continuous, parent Limb1Roll1A_1, child Limb1Roll1B_1, origin xyz=0.013672 0.013672 -0.017382 rpy=0 0 0, axis 0.52586 0.52586 -0.668537
- added joint Revolute 63: type continuous, parent Limb1Pitch3A_1, child Limb1Pitch3B_1, origin xyz=-0.001784 0.001751 -2.6e-05 rpy=0 0 0, axis -0.713693 0.70038 -0.010471
- added joint Revolute 65: type continuous, parent Limb1Roll3A_1, child Limb1Roll3B_1, origin xyz=-0.014652 0.056053 -0.027264 rpy=0 0 0, axis 0.52586 0.52586 -0.668537
- added joint Rigid 101: type fixed, parent Limb0Pitch3B__1__1, child Limb0Roll3A__1__1, origin xyz=0.0 0.0 0.0 rpy=0 0 0
- added joint Rigid 103: type fixed, parent Limb3Roll3B_1, child Limb3Wheel_1, origin xyz=-0.005259 -0.005259 -0.006685 rpy=0 0 0
- added joint Rigid 104: type fixed, parent Limb0Roll3B__1__1, child Limb2Wheel_1, origin xyz=-0.005259 0.005258 -0.006685 rpy=0 0 0
- added joint Rigid 105: type fixed, parent Limb0Roll3B_2, child Limb0Wheel_1, origin xyz=0.005258 -0.005259 -0.006685 rpy=0 0 0
- added joint Rigid 106: type fixed, parent Limb1Roll3B_1, child Limb1Wheel_1, origin xyz=0.005259 0.005258 -0.006685 rpy=0 0 0
- added joint Rigid 107: type fixed, parent Limb3BodyConnector_1, child Connector4_1, origin xyz=-0.014196 -0.014254 -0.018009 rpy=0 0 0
- added joint Rigid 12: type fixed, parent base_link, child Body_connector_5, origin xyz=-0.104123 0.099642 0.676307 rpy=0 0 0
- added joint Rigid 14: type fixed, parent Limb0Pitch2A_2, child Limb0Connector2_2, origin xyz=0.044699 -0.044698 -0.056826 rpy=0 0 0
- added joint Rigid 17: type fixed, parent Limb0Roll1B_2, child Limb0Pitch1A_2, origin xyz=0.002629 -0.002629 -0.003343 rpy=0 0 0
- added joint Rigid 43: type fixed, parent Limb0Connector2_2, child Limb0Connector3_3, origin xyz=0.004206 -0.004207 -0.005348 rpy=0 0 0
- added joint Rigid 44: type fixed, parent Limb0Connector3_3, child Limb0Roll2A_3, origin xyz=0.004207 -0.004207 -0.005348 rpy=0 0 0
- added joint Rigid 46: type fixed, parent Limb0Roll2B_2, child Limb0Roll2C_2, origin xyz=0.002629 -0.00263 -0.003342 rpy=0 0 0
- added joint Rigid 47: type fixed, parent Limb0Roll2C_2, child Limb0Pitch3A_2, origin xyz=0.02541 -0.102493 -0.071414 rpy=0 0 0
- added joint Rigid 49: type fixed, parent Limb0Pitch3B_2, child Limb0Roll3A_2, origin xyz=0.001594 0.00191 -0.000249 rpy=0 0 0
- added joint Rigid 54: type fixed, parent Limb1Roll1B_1, child Limb1Pitch1A_1, origin xyz=0.002629 0.002629 -0.003343 rpy=0 0 0
- added joint Rigid 57: type fixed, parent Limb1Pitch2A_1, child Limb1Connector2_1, origin xyz=0.044698 0.044698 -0.056826 rpy=0 0 0
- added joint Rigid 58: type fixed, parent Limb1Connector2_1, child Limb1Connector3_1, origin xyz=0.004207 0.004207 -0.005348 rpy=0 0 0
- added joint Rigid 59: type fixed, parent Limb1Connector3_1, child Limb1Roll2A_1, origin xyz=0.004207 0.004207 -0.005348 rpy=0 0 0
- added joint Rigid 61: type fixed, parent Limb1Roll2B_1, child LimbRoll2C__1__1, origin xyz=0.002629 0.002629 -0.003342 rpy=0 0 0
- added joint Rigid 62: type fixed, parent LimbRoll2C__1__1, child Limb1Pitch3A_1, origin xyz=0.099728 0.021954 -0.076308 rpy=0 0 0
- added joint Rigid 64: type fixed, parent Limb1Pitch3B_1, child Limb1Roll3A_1, origin xyz=-0.001784 0.001751 -2.6e-05 rpy=0 0 0
- added joint Rigid 66: type fixed, parent Body_connector__2__1, child Limb0Connector1_1, origin xyz=0.014166 -0.014166 -0.018102 rpy=0 0 0
- added joint Rigid 67: type fixed, parent base_link, child Body_connector__2__1, origin xyz=0.099583 -0.104063 0.676307 rpy=0 0 0
- added joint Rigid 68: type fixed, parent Limb0Connector1_1, child Limb0Roll1A_2, origin xyz=0.005784 -0.005785 -0.007354 rpy=0 0 0
- added joint Rigid 69: type fixed, parent Limb1Connector1_1, child Limb1Roll1A_1, origin xyz=0.005785 0.005785 -0.007354 rpy=0 0 0
- added joint Rigid 70: type fixed, parent Body_connector__3__1, child Limb1Connector1_1, origin xyz=0.014196 0.014253 -0.018009 rpy=0 0 0
- added joint Rigid 71: type fixed, parent base_link, child Limb3BodyConnector_1, origin xyz=-0.104123 -0.104063 0.676307 rpy=0 0 0
- added joint Rigid 72: type fixed, parent base_link, child Body_connector__3__1, origin xyz=0.099583 0.099642 0.676307 rpy=0 0 0
- added joint Rigid 74: type fixed, parent Connector4_1, child Limb3Roll1A_1, origin xyz=-0.005784 -0.005784 -0.007354 rpy=0 0 0
- added joint Rigid 76: type fixed, parent Limb3Roll1B_1, child Limb3Pitch1A_1, origin xyz=-0.002629 -0.00263 -0.003343 rpy=0 0 0
- added joint Rigid 79: type fixed, parent Limb3Pitch2A_1, child Limb3Connector2_1, origin xyz=-0.044698 -0.044698 -0.056826 rpy=0 0 0
- added joint Rigid 80: type fixed, parent Limb3Connector2_1, child Limb3Connector3_1, origin xyz=-0.004207 -0.004207 -0.005348 rpy=0 0 0
- added joint Rigid 81: type fixed, parent Limb3Connector3_1, child Limb3Roll2A_1, origin xyz=-0.004207 -0.004207 -0.005348 rpy=0 0 0
- added joint Rigid 83: type fixed, parent Limb3Roll2B_1, child Limb3Roll2C_1, origin xyz=-0.00263 -0.002629 -0.003343 rpy=0 0 0
- added joint Rigid 84: type fixed, parent Limb3Roll2C_1, child Limb3Pitch3A_1, origin xyz=-0.099728 -0.021954 -0.076307 rpy=0 0 0
- added joint Rigid 86: type fixed, parent Limb3Pitch3B_1, child Limb3Roll3A_1, origin xyz=0.001785 -0.001751 -2.6e-05 rpy=0 0 0
- added joint Rigid 88: type fixed, parent Body_connector_5, child Limb0Connector1__1__1, origin xyz=-0.014255 0.014167 -0.01803 rpy=0 0 0
- added joint Rigid 89: type fixed, parent Limb0Connector1__1__1, child Limb0Roll1A__1__1, origin xyz=-0.005785 0.005785 -0.007354 rpy=0 0 0
- added joint Rigid 91: type fixed, parent Limb0Roll1B__1__1, child Limb0Pitch1A__1__1, origin xyz=-0.00263 0.002629 -0.003343 rpy=0 0 0
- added joint Rigid 94: type fixed, parent Limb0Pitch2A__1__1, child Limb0Connector2__1__1, origin xyz=-0.044698 0.044698 -0.056825 rpy=0 0 0
- added joint Rigid 95: type fixed, parent Limb0Connector2__1__1, child Limb0Connector3__1__1, origin xyz=-0.004207 0.004207 -0.005349 rpy=0 0 0
- added joint Rigid 96: type fixed, parent Limb0Connector3__1__1, child Limb0Roll2A__1__1, origin xyz=-0.004207 0.004207 -0.005348 rpy=0 0 0
- added joint Rigid 98: type fixed, parent Limb0Roll2B__1__1, child Limb0Roll2C__1__1, origin xyz=-0.00263 0.002629 -0.003343 rpy=0 0 0
- added joint Rigid 99: type fixed, parent Limb0Roll2C__1__1, child Limb0Pitch3A__1__1, origin xyz=-0.021954 0.099728 -0.076307 rpy=0 0 0
