Commit message: Margin added and moonbot7 with tips

File: src/rviz_basic/urdf/moonbot7.urdf (robot description, URDF)
Before this commit: robot Moonbot_ver7, 15 links, 14 joints
Links:
- added link end1
- added link end2
- added link end3
Joints:
- removed joint end_effector
- added joint end_effector1: type fixed, parent Leg1_Link3, child end1, origin xyz=-0.16 0 0 rpy=0 0 0
- added joint end_effector2: type fixed, parent Leg2_Link3, child end2, origin xyz=-0.16 0 0 rpy=0 0 0
- added joint end_effector3: type fixed, parent Leg3_Link3, child end3, origin xyz=-0.16 0 0 rpy=0 0 0
- added joint end_effector4: type fixed, parent Leg4_Link3, child end4, origin xyz=-0.16 0 0 rpy=0 0 0
