Commit message: utomatic urdf load

File: src/rviz_basic/urdf/hero_3wheel_1hand/hero_3wheel_1hand.xacro (robot description, xacro)
@@ -3,7 +3,9 @@
 <xacro:property name="ThisPackage" value="rviz_basic" />
 <xacro:property name="Filename" value="hero_3wheel_1hand" />
-<xacro:include filename="$(find ${ThisPackage})/urdf/${Filename}/materials.xacro" />
-<xacro:include filename="$(find ${ThisPackage})/urdf/${Filename}/hero_3wheel_1hand.trans" />
-<xacro:include filename="$(find ${ThisPackage})/urdf/${Filename}/hero_3wheel_1hand.gazebo" />
+<xacro:property name="UrdfDataPath" value="package://${ThisPackage}/urdf/${Filename}" />
+<xacro:property name="MeshPath" value="package://${ThisPackage}/meshes/${Filename}" />
+<xacro:include filename="materials.xacro" />
+<xacro:include filename="${Filename}.trans" />
+<xacro:include filename="${Filename}.gazebo" />
 <link name="base_link">
   <inertial>
@@ -15,5 +17,5 @@
     <origin xyz="0 0 0" rpy="0 0 0"/>
     <geometry>
-    <mesh filename="package://${ThisPackage}/meshes/${Filename}/base_link.stl" scale="0.001 0.001 0.001"/>
+    <mesh filename="${MeshPath}/base_link.stl" scale="0.001 0.001 0.001"/>
     </geometry>
     <material name="silver"/>
@@ -22,5 +24,5 @@
     <origin xyz="0 0 0" rpy="0 0 0"/>
     <geometry>
-    <mesh filename="package://${ThisPackage}/meshes/${Filename}/base_link.stl" scale="0.001 0.001 0.001"/>
+    <mesh filename="${MeshPath}/base_link.stl" scale="0.001 0.001 0.001"/>
     </geometry>
   </collision>
@@ -35,5 +37,5 @@
     <origin xyz="0.048782 0.161811 -0.129376" rpy="0 0 0"/>
     <geometry>
-    <mesh filename="package://${ThisPackage}/meshes/${Filename}/Leg1_Hip_2.stl" scale="0.001 0.001 0.001"/>
+    <mesh filename="${MeshPath}/Leg1_Hip_2.stl" scale="0.001 0.001 0.001"/>
     </geometry>
     <material name="silver"/>
@@ -42,5 +44,5 @@
     <origin xyz="0.048782 0.161811 -0.129376" rpy="0 0 0"/>
     <geometry>
-    <mesh filename="package://${ThisPackage}/meshes/${Filename}/Leg1_Hip_2.stl" scale="0.001 0.001 0.001"/>
+    <mesh filename="${MeshPath}/Leg1_Hip_2.stl" scale="0.001 0.001 0.001"/>
     </geometry>
   </collision>
@@ -55,5 +57,5 @@
     <origin xyz="0.029926 0.194471 -0.116043" rpy="0 0 0"/>
     <geometry>
-    <mesh filename="package://${ThisPackage}/meshes/${Filename}/Leg1_RollLink1_2.stl" scale="0.001 0.001 0.001"/>
+    <mesh filename="${MeshPath}/Leg1_RollLink1_2.stl" scale="0.001 0.001 0.001"/>
     </geometry>
     <material name="silver"/>
@@ -62,5 +64,5 @@
     <origin xyz="0.029926 0.194471 -0.116043" rpy="0 0 0"/>
     <geometry>
-    <mesh filename="package://${ThisPackage}/meshes/${Filename}/Leg1_RollLink1_2.stl" scale="0.001 0.001 0.001"/>
+    <mesh filename="${MeshPath}/Leg1_RollLink1_2.stl" scale="0.001 0.001 0.001"/>
     </geometry>
   </collision>
@@ -75,5 +77,5 @@
     <origin xyz="0.026086 0.30112 -0.082709" rpy="0 0 0"/>
     <geometry>
-    <mesh filename="package://${ThisPackage}/meshes/${Filename}/Leg1_PitchLink1_2.stl" scale="0.001 0.001 0.001"/>
+    <mesh filename="${MeshPath}/Leg1_PitchLink1_2.stl" scale="0.001 0.001 0.001"/>
     </geometry>
     <material name="silver"/>
@@ -82,5 +84,5 @@
     <origin xyz="0.026086 0.30112 -0.082709" rpy="0 0 0"/>
     <geometry>
-    <mesh filename="package://${ThisPackage}/meshes/${Filename}/Leg1_PitchLink1_2.stl" scale="0.001 0.001 0.001"/>
+    <mesh filename="${MeshPath}/Leg1_PitchLink1_2.stl" scale="0.001 0.001 0.001"/>
     </geometry>
   </collision>
@@ -95,5 +97,5 @@
     <origin xyz="-0.035874 0.304437 -0.129805" rpy="0 0 0"/>
     <geometry>
-    <mesh filename="package://${ThisPackage}/meshes/${Filename}/Leg1_RollLink2_2.stl" scale="0.001 0.001 0.001"/>
+    <mesh filename="${MeshPath}/Leg1_RollLink2_2.stl" scale="0.001 0.001 0.001"/>
     </geometry>
     <material name="silver"/>
@@ -102,5 +104,5 @@
     <origin xyz="-0.035874 0.304437 -0.129805" rpy="0 0 0"/>
     <geometry>
-    <mesh filename="package://${ThisPackage}/meshes/${Filename}/Leg1_RollLink2_2.stl" scale="0.001 0.001 0.001"/>
+    <mesh filename="${MeshPath}/Leg1_RollLink2_2.stl" scale="0.001 0.001 0.001"/>
     </geometry>
   </collision>
@@ -115,5 +117,5 @@
     <origin xyz="-0.387924 0.6809 0.030367" rpy="0 0 0"/>
     <geometry>
-    <mesh filename="package://${ThisPackage}/meshes/${Filename}/Leg1_Ankle_2.stl" scale="0.001 0.001 0.001"/>
+    <mesh filename="${MeshPath}/Leg1_Ankle_2.stl" scale="0.001 0.001 0.001"/>
     </geometry>
     <material name="silver"/>
@@ -122,5 +124,5 @@
     <origin xyz="-0.387924 0.6809 0.030367" rpy="0 0 0"/>
     <geometry>
-    <mesh filename="package://${ThisPackage}/meshes/${Filename}/Leg1_Ankle_2.stl" scale="0.001 0.001 0.001"/>
+    <mesh filename="${MeshPath}/Leg1_Ankle_2.stl" scale="0.001 0.001 0.001"/>
     </geometry>
   </collision>
@@ -135,5 +137,5 @@
     <origin xyz="-0.387924 0.6809 0.070367" rpy="0 0 0"/>
     <geometry>
-    <mesh filename="package://${ThisPackage}/meshes/${Filename}/Leg1_WheelBody_2.stl" scale="0.001 0.001 0.001"/>
+    <mesh filename="${MeshPath}/Leg1_WheelBody_2.stl" scale="0.001 0.001 0.001"/>
     </geometry>
     <material name="silver"/>
@@ -142,5 +144,5 @@
     <origin xyz="-0.387924 0.6809 0.070367" rpy="0 0 0"/>
     <geometry>
-    <mesh filename="package://${ThisPackage}/meshes/${Filename}/Leg1_WheelBody_2.stl" scale="0.001 0.001 0.001"/>
+    <mesh filename="${MeshPath}/Leg1_WheelBody_2.stl" scale="0.001 0.001 0.001"/>
     </geometry>
   </collision>
@@ -155,5 +157,5 @@
     <origin xyz="-0.387924 0.6109 0.161367" rpy="0 0 0"/>
     <geometry>
-    <mesh filename="package://${ThisPackage}/meshes/${Filename}/Leg1_Wheel1_2.stl" scale="0.001 0.001 0.001"/>
+    <mesh filename="${MeshPath}/Leg1_Wheel1_2.stl" scale="0.001 0.001 0.001"/>
     </geometry>
     <material name="silver"/>
@@ -162,5 +164,5 @@
     <origin xyz="-0.387924 0.6109 0.161367" rpy="0 0 0"/>
     <geometry>
-    <mesh filename="package://${ThisPackage}/meshes/${Filename}/Leg1_Wheel1_2.stl" scale="0.001 0.001 0.001"/>
+    <mesh filename="${MeshPath}/Leg1_Wheel1_2.stl" scale="0.001 0.001 0.001"/>
     </geometry>
   </collision>
@@ -175,5 +177,5 @@
     <origin xyz="-0.387924 0.7509 0.161367" rpy="0 0 0"/>
     <geometry>
-    <mesh filename="package://${ThisPackage}/meshes/${Filename}/Leg1_Wheel2_2.stl" scale="0.001 0.001 0.001"/>
+    <mesh filename="${MeshPath}/Leg1_Wheel2_2.stl" scale="0.001 0.001 0.001"/>
     </geometry>
     <material name="silver"/>
@@ -182,5 +184,5 @@
     <origin xyz="-0.387924 0.7509 0.161367" rpy="0 0 0"/>
     <geometry>
-    <mesh filename="package://${ThisPackage}/meshes/${Filename}/Leg1_Wheel2_2.stl" scale="0.001 0.001 0.001"/>
+    <mesh filename="${MeshPath}/Leg1_Wheel2_2.stl" scale="0.001 0.001 0.001"/>
     </geometry>
   </collision>
@@ -195,5 +197,5 @@
     <origin xyz="0.141408 -0.000459 -0.393612" rpy="0 0 0"/>
     <geometry>
-    <mesh filename="package://${ThisPackage}/meshes/${Filename}/Arm_Hip_2.stl" scale="0.001 0.001 0.001"/>
+    <mesh filename="${MeshPath}/Arm_Hip_2.stl" scale="0.001 0.001 0.001"/>
     </geometry>
     <material name="silver"/>
@@ -202,5 +204,5 @@
     <origin xyz="0.141408 -0.000459 -0.393612" rpy="0 0 0"/>
     <geometry>
-    <mesh filename="package://${ThisPackage}/meshes/${Filename}/Arm_Hip_2.stl" scale="0.001 0.001 0.001"/>
+    <mesh filename="${MeshPath}/Arm_Hip_2.stl" scale="0.001 0.001 0.001"/>
     </geometry>
   </collision>
@@ -215,5 +217,5 @@
     <origin xyz="0.141408 -0.000459 -0.433612" rpy="0 0 0"/>
     <geometry>
-    <mesh filename="package://${ThisPackage}/meshes/${Filename}/Arm_RollLink1_2.stl" scale="0.001 0.001 0.001"/>
+    <mesh filename="${MeshPath}/Arm_RollLink1_2.stl" scale="0.001 0.001 0.001"/>
     </geometry>
     <material name="silver"/>
@@ -222,5 +224,5 @@
     <origin xyz="0.141408 -0.000459 -0.433612" rpy="0 0 0"/>
     <geometry>
-    <mesh filename="package://${ThisPackage}/meshes/${Filename}/Arm_RollLink1_2.stl" scale="0.001 0.001 0.001"/>
+    <mesh filename="${MeshPath}/Arm_RollLink1_2.stl" scale="0.001 0.001 0.001"/>
     </geometry>
   </collision>
@@ -235,5 +237,5 @@
     <origin xyz="0.141408 -0.050459 -0.533612" rpy="0 0 0"/>
     <geometry>
-    <mesh filename="package://${ThisPackage}/meshes/${Filename}/Arm_PitchLink1_2.stl" scale="0.001 0.001 0.001"/>
+    <mesh filename="${MeshPath}/Arm_PitchLink1_2.stl" scale="0.001 0.001 0.001"/>
     </geometry>
     <material name="silver"/>
@@ -242,5 +244,5 @@
     <origin xyz="0.141408 -0.050459 -0.533612" rpy="0 0 0"/>
     <geometry>
-    <mesh filename="package://${ThisPackage}/meshes/${Filename}/Arm_PitchLink1_2.stl" scale="0.001 0.001 0.001"/>
+    <mesh filename="${MeshPath}/Arm_PitchLink1_2.stl" scale="0.001 0.001 0.001"/>
     </geometry>
   </collision>
@@ -255,5 +257,5 @@
     <origin xyz="0.102841 -0.004459 -0.579575" rpy="0 0 0"/>
     <geometry>
-    <mesh filename="package://${ThisPackage}/meshes/${Filename}/Arm_RollLink2_2.stl" scale="0.001 0.001 0.001"/>
+    <mesh filename="${MeshPath}/Arm_RollLink2_2.stl" scale="0.001 0.001 0.001"/>
     </geometry>
     <material name="silver"/>
@@ -262,5 +264,5 @@
     <origin xyz="0.102841 -0.004459 -0.579575" rpy="0 0 0"/>
     <geometry>
-    <mesh filename="package://${ThisPackage}/meshes/${Filename}/Arm_RollLink2_2.stl" scale="0.001 0.001 0.001"/>
+    <mesh filename="${MeshPath}/Arm_RollLink2_2.stl" scale="0.001 0.001 0.001"/>
     </geometry>
   </collision>
@@ -275,5 +277,5 @@
     <origin xyz="-0.179986 -0.004459 -0.916634" rpy="0 0 0"/>
     <geometry>
-    <mesh filename="package://${ThisPackage}/meshes/${Filename}/Arm_PitchLink2_2.stl" scale="0.001 0.001 0.001"/>
+    <mesh filename="${MeshPath}/Arm_PitchLink2_2.stl" scale="0.001 0.001 0.001"/>
     </geometry>
     <material name="silver"/>
@@ -282,5 +284,5 @@
     <origin xyz="-0.179986 -0.004459 -0.916634" rpy="0 0 0"/>
     <geometry>
-    <mesh filename="package://${ThisPackage}/meshes/${Filename}/Arm_PitchLink2_2.stl" scale="0.001 0.001 0.001"/>
+    <mesh filename="${MeshPath}/Arm_PitchLink2_2.stl" scale="0.001 0.001 0.001"/>
     </geometry>
   </collision>
@@ -295,5 +297,5 @@
     <origin xyz="-0.460884 -0.004459 -0.577966" rpy="0 0 0"/>
     <geometry>
-    <mesh filename="package://${ThisPackage}/meshes/${Filename}/Arm_RollLink3_2.stl" scale="0.001 0.001 0.001"/>
+    <mesh filename="${MeshPath}/Arm_RollLink3_2.stl" scale="0.001 0.001 0.001"/>
     </geometry>
     <material name="silver"/>
@@ -302,5 +304,5 @@
     <origin xyz="-0.460884 -0.004459 -0.577966" rpy="0 0 0"/>
     <geometry>
-    <mesh filename="package://${ThisPackage}/meshes/${Filename}/Arm_RollLink3_2.stl" scale="0.001 0.001 0.001"/>
+    <mesh filename="${MeshPath}/Arm_RollLink3_2.stl" scale="0.001 0.001 0.001"/>
     </geometry>
   </collision>
@@ -315,5 +317,5 @@
     <origin xyz="-0.533628 -0.053103 -0.508381" rpy="0 0 0"/>
     <geometry>
-    <mesh filename="package://${ThisPackage}/meshes/${Filename}/Arm_PitchLink3_2.stl" scale="0.001 0.001 0.001"/>
+    <mesh filename="${MeshPath}/Arm_PitchLink3_2.stl" scale="0.001 0.001 0.001"/>
     </geometry>
     <material name="silver"/>
@@ -322,5 +324,5 @@
     <origin xyz="-0.533628 -0.053103 -0.508381" rpy="0 0 0"/>
     <geometry>
-    <mesh filename="package://${ThisPackage}/meshes/${Filename}/Arm_PitchLink3_2.stl" scale="0.001 0.001 0.001"/>
+    <mesh filename="${MeshPath}/Arm_PitchLink3_2.stl" scale="0.001 0.001 0.001"/>
     </geometry>
   </collision>
@@ -335,5 +337,5 @@
     <origin xyz="-0.576209 -0.002185 -0.474216" rpy="0 0 0"/>
     <geometry>
-    <mesh filename="package://${ThisPackage}/meshes/${Filename}/Arm_Gripper_2.stl" scale="0.001 0.001 0.001"/>
+    <mesh filename="${MeshPath}/Arm_Gripper_2.stl" scale="0.001 0.001 0.001"/>
     </geometry>
     <material name="silver"/>
@@ -342,5 +344,5 @@
     <origin xyz="-0.576209 -0.002185 -0.474216" rpy="0 0 0"/>
     <geometry>
-    <mesh filename="package://${ThisPackage}/meshes/${Filename}/Arm_Gripper_2.stl" scale="0.001 0.001 0.001"/>
+    <mesh filename="${MeshPath}/Arm_Gripper_2.stl" scale="0.001 0.001 0.001"/>
     </geometry>
   </collision>
@@ -355,5 +357,5 @@
     <origin xyz="0.048252 -0.161811 -0.130126" rpy="0 0 0"/>
     <geometry>
-    <mesh filename="package://${ThisPackage}/meshes/${Filename}/Leg2_Hip_2.stl" scale="0.001 0.001 0.001"/>
+    <mesh filename="${MeshPath}/Leg2_Hip_2.stl" scale="0.001 0.001 0.001"/>
     </geometry>
     <material name="silver"/>
@@ -362,5 +364,5 @@
     <origin xyz="0.048252 -0.161811 -0.130126" rpy="0 0 0"/>
     <geometry>
-    <mesh filename="package://${ThisPackage}/meshes/${Filename}/Leg2_Hip_2.stl" scale="0.001 0.001 0.001"/>
+    <mesh filename="${MeshPath}/Leg2_Hip_2.stl" scale="0.001 0.001 0.001"/>
     </geometry>
   </collision>
@@ -375,5 +377,5 @@
     <origin xyz="0.029396 -0.194471 -0.116793" rpy="0 0 0"/>
     <geometry>
-    <mesh filename="package://${ThisPackage}/meshes/${Filename}/Leg2_RollLink1_2.stl" scale="0.001 0.001 0.001"/>
+    <mesh filename="${MeshPath}/Leg2_RollLink1_2.stl" scale="0.001 0.001 0.001"/>
     </geometry>
     <material name="silver"/>
@@ -382,5 +384,5 @@
     <origin xyz="0.029396 -0.194471 -0.116793" rpy="0 0 0"/>
     <geometry>
-    <mesh filename="package://${ThisPackage}/meshes/${Filename}/Leg2_RollLink1_2.stl" scale="0.001 0.001 0.001"/>
+    <mesh filename="${MeshPath}/Leg2_RollLink1_2.stl" scale="0.001 0.001 0.001"/>
     </geometry>
   </collision>
@@ -395,5 +397,5 @@
     <origin xyz="-0.05628 -0.247865 -0.068746" rpy="0 0 0"/>
     <geometry>
-    <mesh filename="package://${ThisPackage}/meshes/${Filename}/Leg2_PitchLink1_2.stl" scale="0.001 0.001 0.001"/>
+    <mesh filename="${MeshPath}/Leg2_PitchLink1_2.stl" scale="0.001 0.001 0.001"/>
     </geometry>
     <material name="silver"/>
@@ -402,5 +404,5 @@
     <origin xyz="-0.05628 -0.247865 -0.068746" rpy="0 0 0"/>
     <geometry>
-    <mesh filename="package://${ThisPackage}/meshes/${Filename}/Leg2_PitchLink1_2.stl" scale="0.001 0.001 0.001"/>
+    <mesh filename="${MeshPath}/Leg2_PitchLink1_2.stl" scale="0.001 0.001 0.001"/>
     </geometry>
   </collision>
@@ -415,5 +417,5 @@
     <origin xyz="-0.04822 -0.298225 -0.127626" rpy="0 0 0"/>
     <geometry>
-    <mesh filename="package://${ThisPackage}/meshes/${Filename}/Leg2_RollLink2_2.stl" scale="0.001 0.001 0.001"/>
+    <mesh filename="${MeshPath}/Leg2_RollLink2_2.stl" scale="0.001 0.001 0.001"/>
     </geometry>
     <material name="silver"/>
@@ -422,5 +424,5 @@
     <origin xyz="-0.04822 -0.298225 -0.127626" rpy="0 0 0"/>
     <geometry>
-    <mesh filename="package://${ThisPackage}/meshes/${Filename}/Leg2_RollLink2_2.stl" scale="0.001 0.001 0.001"/>
+    <mesh filename="${MeshPath}/Leg2_RollLink2_2.stl" scale="0.001 0.001 0.001"/>
     </geometry>
   </collision>
@@ -435,5 +437,5 @@
     <origin xyz="-0.164283 0.526848 -0.487079" rpy="0 0 0"/>
     <geometry>
-    <mesh filename="package://${ThisPackage}/meshes/${Filename}/Leg1_PitchRollLink3_2.stl" scale="0.001 0.001 0.001"/>
+    <mesh filename="${MeshPath}/Leg1_PitchRollLink3_2.stl" scale="0.001 0.001 0.001"/>
     </geometry>
     <material name="silver"/>
@@ -442,5 +444,5 @@
     <origin xyz="-0.164283 0.526848 -0.487079" rpy="0 0 0"/>
     <geometry>
-    <mesh filename="package://${ThisPackage}/meshes/${Filename}/Leg1_PitchRollLink3_2.stl" scale="0.001 0.001 0.001"/>
+    <mesh filename="${MeshPath}/Leg1_PitchRollLink3_2.stl" scale="0.001 0.001 0.001"/>
     </geometry>
   </collision>
@@ -455,5 +457,5 @@
     <origin xyz="-0.359864 0.722284 -0.069633" rpy="0 0 0"/>
     <geometry>
-    <mesh filename="package://${ThisPackage}/meshes/${Filename}/Leg1_SteeringLink3_2.stl" scale="0.001 0.001 0.001"/>
+    <mesh filename="${MeshPath}/Leg1_SteeringLink3_2.stl" scale="0.001 0.001 0.001"/>
     </geometry>
     <material name="silver"/>
@@ -462,5 +464,5 @@
     <origin xyz="-0.359864 0.722284 -0.069633" rpy="0 0 0"/>
     <geometry>
-    <mesh filename="package://${ThisPackage}/meshes/${Filename}/Leg1_SteeringLink3_2.stl" scale="0.001 0.001 0.001"/>
+    <mesh filename="${MeshPath}/Leg1_SteeringLink3_2.stl" scale="0.001 0.001 0.001"/>
     </geometry>
   </collision>
@@ -475,5 +477,5 @@
     <origin xyz="-0.291111 -0.45733 -0.458216" rpy="0 0 0"/>
     <geometry>
-    <mesh filename="package://${ThisPackage}/meshes/${Filename}/Leg2_PitchLink2_2.stl" scale="0.001 0.001 0.001"/>
+    <mesh filename="${MeshPath}/Leg2_PitchLink2_2.stl" scale="0.001 0.001 0.001"/>
     </geometry>
     <material name="silver"/>
@@ -482,5 +484,5 @@
     <origin xyz="-0.291111 -0.45733 -0.458216" rpy="0 0 0"/>
     <geometry>
-    <mesh filename="package://${ThisPackage}/meshes/${Filename}/Leg2_PitchLink2_2.stl" scale="0.001 0.001 0.001"/>
+    <mesh filename="${MeshPath}/Leg2_PitchLink2_2.stl" scale="0.001 0.001 0.001"/>
     </geometry>
   </collision>
@@ -495,5 +497,5 @@
     <origin xyz="-0.47637 -0.660815 -0.11489" rpy="0 0 0"/>
     <geometry>
-    <mesh filename="package://${ThisPackage}/meshes/${Filename}/Leg2_RollLink3_2.stl" scale="0.001 0.001 0.001"/>
+    <mesh filename="${MeshPath}/Leg2_RollLink3_2.stl" scale="0.001 0.001 0.001"/>
     </geometry>
     <material name="silver"/>
@@ -502,5 +504,5 @@
     <origin xyz="-0.47637 -0.660815 -0.11489" rpy="0 0 0"/>
     <geometry>
-    <mesh filename="package://${ThisPackage}/meshes/${Filename}/Leg2_RollLink3_2.stl" scale="0.001 0.001 0.001"/>
+    <mesh filename="${MeshPath}/Leg2_RollLink3_2.stl" scale="0.001 0.001 0.001"/>
     </geometry>
   </collision>
@@ -515,5 +517,5 @@
     <origin xyz="-0.539241 -0.652631 -0.069633" rpy="0 0 0"/>
     <geometry>
-    <mesh filename="package://${ThisPackage}/meshes/${Filename}/Leg2_SteeringLink3_2.stl" scale="0.001 0.001 0.001"/>
+    <mesh filename="${MeshPath}/Leg2_SteeringLink3_2.stl" scale="0.001 0.001 0.001"/>
     </geometry>
     <material name="silver"/>
@@ -522,5 +524,5 @@
     <origin xyz="-0.539241 -0.652631 -0.069633" rpy="0 0 0"/>
     <geometry>
-    <mesh filename="package://${ThisPackage}/meshes/${Filename}/Leg2_SteeringLink3_2.stl" scale="0.001 0.001 0.001"/>
+    <mesh filename="${MeshPath}/Leg2_SteeringLink3_2.stl" scale="0.001 0.001 0.001"/>
     </geometry>
   </collision>
@@ -535,5 +537,5 @@
     <origin xyz="-0.502269 -0.686292 0.030367" rpy="0 0 0"/>
     <geometry>
-    <mesh filename="package://${ThisPackage}/meshes/${Filename}/Leg2_Ankle_2.stl" scale="0.001 0.001 0.001"/>
+    <mesh filename="${MeshPath}/Leg2_Ankle_2.stl" scale="0.001 0.001 0.001"/>
     </geometry>
     <material name="silver"/>
@@ -542,5 +544,5 @@
     <origin xyz="-0.502269 -0.686292 0.030367" rpy="0 0 0"/>
     <geometry>
-    <mesh filename="package://${ThisPackage}/meshes/${Filename}/Leg2_Ankle_2.stl" scale="0.001 0.001 0.001"/>
+    <mesh filename="${MeshPath}/Leg2_Ankle_2.stl" scale="0.001 0.001 0.001"/>
     </geometry>
   </collision>
@@ -555,5 +557,5 @@
     <origin xyz="-0.502269 -0.686292 0.070367" rpy="0 0 0"/>
     <geometry>
-    <mesh filename="package://${ThisPackage}/meshes/${Filename}/Leg2_WheelBody_2.stl" scale="0.001 0.001 0.001"/>
+    <mesh filename="${MeshPath}/Leg2_WheelBody_2.stl" scale="0.001 0.001 0.001"/>
     </geometry>
     <material name="silver"/>
@@ -562,5 +564,5 @@
     <origin xyz="-0.502269 -0.686292 0.070367" rpy="0 0 0"/>
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