Commit message: utomatic urdf load

File: src/rviz_basic/urdf/moonbot_7/moonbot_7.xacro (robot description, xacro)
@@ -1,8 +1,8 @@
-<?xml version="1.0" encoding="utf-8"?>
-<!-- This URDF was automatically created by SolidWorks to URDF Exporter! Originally created by Stephen Brawner (brawner@gmail.com)
-     Commit Version: 1.6.0-4-g7f85cfe  Build Version: 1.6.7995.38578
-     For more information, please see http://wiki.ros.org/sw_urdf_exporter -->
-<robot
-  name="Moonbot_ver7">
+<?xml version="1.0" ?>
+<robot name="moonbot_7" xmlns:xacro="http://www.ros.org/wiki/xacro">
+<xacro:property name="ThisPackage" value="rviz_basic" />
+<xacro:property name="Filename" value="moonbot_7" />
+<xacro:property name="UrdfDataPath" value="package://${ThisPackage}/urdf/${Filename}" />
+<xacro:property name="MeshPath" value="package://${ThisPackage}/meshes/${Filename}" />
   <material name="Grey">
       <color rgba="0.9 0.9 0.98 1" />
@@ -26,17 +26,17 @@
       <geometry>
         <mesh
-        filename="package://rviz_basic/base_link.STL" />
-      </geometry>
-      <material
-        name="Black">
-      </material>
-    </visual>
-    <collision>
-      <origin
-        xyz="0 0 0"
-        rpy="0 0 0" />
-      <geometry>
-        <mesh
-        filename="package://rviz_basic/base_link.STL" />
+        filename="${MeshPath}/base_link.STL" />
+      </geometry>
+      <material
+        name="Black">
+      </material>
+    </visual>
+    <collision>
+      <origin
+        xyz="0 0 0"
+        rpy="0 0 0" />
+      <geometry>
+        <mesh
+        filename="${MeshPath}/base_link.STL" />
       </geometry>
     </collision>
@@ -64,5 +64,5 @@
       <geometry>
         <mesh
-        filename="package://rviz_basic/Leg4_Link1.STL" />
+        filename="${MeshPath}/Leg4_Link1.STL" />
       </geometry>
       <material
@@ -76,5 +76,5 @@
       <geometry>
         <mesh
-        filename="package://rviz_basic/Leg4_Link1.STL" />
+        filename="${MeshPath}/Leg4_Link1.STL" />
       </geometry>
     </collision>
@@ -120,17 +120,17 @@
       <geometry>
         <mesh
-        filename="package://rviz_basic/Leg4_Link2.STL" />
-      </geometry>
-      <material
-        name="Black">
-      </material>
-    </visual>
-    <collision>
-      <origin
-        xyz="0 0 0"
-        rpy="0 0 0" />
-      <geometry>
-        <mesh
-        filename="package://rviz_basic/Leg4_Link2.STL" />
+        filename="${MeshPath}/Leg4_Link2.STL" />
+      </geometry>
+      <material
+        name="Black">
+      </material>
+    </visual>
+    <collision>
+      <origin
+        xyz="0 0 0"
+        rpy="0 0 0" />
+      <geometry>
+        <mesh
+        filename="${MeshPath}/Leg4_Link2.STL" />
       </geometry>
     </collision>
@@ -176,17 +176,17 @@
       <geometry>
         <mesh
-        filename="package://rviz_basic/Leg4_Link3.STL" />
-      </geometry>
-      <material
-        name="Black">
-      </material>
-    </visual>
-    <collision>
-      <origin
-        xyz="0 0 0"
-        rpy="0 0 0" />
-      <geometry>
-        <mesh
-        filename="package://rviz_basic/Leg4_Link3.STL" />
+        filename="${MeshPath}/Leg4_Link3.STL" />
+      </geometry>
+      <material
+        name="Black">
+      </material>
+    </visual>
+    <collision>
+      <origin
+        xyz="0 0 0"
+        rpy="0 0 0" />
+      <geometry>
+        <mesh
+        filename="${MeshPath}/Leg4_Link3.STL" />
       </geometry>
     </collision>
@@ -232,5 +232,5 @@
       <geometry>
         <mesh
-        filename="package://rviz_basic/Leg1_Link1.STL" />
+        filename="${MeshPath}/Leg1_Link1.STL" />
       </geometry>
       <material
@@ -244,5 +244,5 @@
       <geometry>
         <mesh
-        filename="package://rviz_basic/Leg1_Link1.STL" />
+        filename="${MeshPath}/Leg1_Link1.STL" />
       </geometry>
     </collision>
@@ -288,17 +288,17 @@
       <geometry>
         <mesh
-        filename="package://rviz_basic/Leg1_Link2.STL" />
-      </geometry>
-      <material
-        name="Black">
-      </material>
-    </visual>
-    <collision>
-      <origin
-        xyz="0 0 0"
-        rpy="0 0 0" />
-      <geometry>
-        <mesh
-        filename="package://rviz_basic/Leg1_Link2.STL" />
+        filename="${MeshPath}/Leg1_Link2.STL" />
+      </geometry>
+      <material
+        name="Black">
+      </material>
+    </visual>
+    <collision>
+      <origin
+        xyz="0 0 0"
+        rpy="0 0 0" />
+      <geometry>
+        <mesh
+        filename="${MeshPath}/Leg1_Link2.STL" />
       </geometry>
     </collision>
@@ -344,17 +344,17 @@
       <geometry>
         <mesh
-        filename="package://rviz_basic/Leg1_Link3.STL" />
-      </geometry>
-      <material
-        name="Black">
-      </material>
-    </visual>
-    <collision>
-      <origin
-        xyz="0 0 0"
-        rpy="0 0 0" />
-      <geometry>
-        <mesh
-        filename="package://rviz_basic/Leg1_Link3.STL" />
+        filename="${MeshPath}/Leg1_Link3.STL" />
+      </geometry>
+      <material
+        name="Black">
+      </material>
+    </visual>
+    <collision>
+      <origin
+        xyz="0 0 0"
+        rpy="0 0 0" />
+      <geometry>
+        <mesh
+        filename="${MeshPath}/Leg1_Link3.STL" />
       </geometry>
     </collision>
@@ -400,5 +400,5 @@
       <geometry>
         <mesh
-        filename="package://rviz_basic/Leg2_Link1.STL" />
+        filename="${MeshPath}/Leg2_Link1.STL" />
       </geometry>
       <material
@@ -412,5 +412,5 @@
       <geometry>
         <mesh
-        filename="package://rviz_basic/Leg2_Link1.STL" />
+        filename="${MeshPath}/Leg2_Link1.STL" />
       </geometry>
     </collision>
@@ -456,17 +456,17 @@
       <geometry>
         <mesh
-        filename="package://rviz_basic/Leg2_Link2.STL" />
-      </geometry>
-      <material
-        name="Black">
-      </material>
-    </visual>
-    <collision>
-      <origin
-        xyz="0 0 0"
-        rpy="0 0 0" />
-      <geometry>
-        <mesh
-        filename="package://rviz_basic/Leg2_Link2.STL" />
+        filename="${MeshPath}/Leg2_Link2.STL" />
+      </geometry>
+      <material
+        name="Black">
+      </material>
+    </visual>
+    <collision>
+      <origin
+        xyz="0 0 0"
+        rpy="0 0 0" />
+      <geometry>
+        <mesh
+        filename="${MeshPath}/Leg2_Link2.STL" />
       </geometry>
     </collision>
@@ -512,17 +512,17 @@
       <geometry>
         <mesh
-        filename="package://rviz_basic/Leg2_Link3.STL" />
-      </geometry>
-      <material
-        name="Black">
-      </material>
-    </visual>
-    <collision>
-      <origin
-        xyz="0 0 0"
-        rpy="0 0 0" />
-      <geometry>
-        <mesh
-        filename="package://rviz_basic/Leg2_Link3.STL" />
+        filename="${MeshPath}/Leg2_Link3.STL" />
+      </geometry>
+      <material
+        name="Black">
+      </material>
+    </visual>
+    <collision>
+      <origin
+        xyz="0 0 0"
+        rpy="0 0 0" />
+      <geometry>
+        <mesh
+        filename="${MeshPath}/Leg2_Link3.STL" />
       </geometry>
     </collision>
@@ -568,5 +568,5 @@
       <geometry>
         <mesh
-        filename="package://rviz_basic/Leg3_Link1.STL" />
+        filename="${MeshPath}/Leg3_Link1.STL" />
       </geometry>
       <material
@@ -580,5 +580,5 @@
       <geometry>
         <mesh
-        filename="package://rviz_basic/Leg3_Link1.STL" />
+        filename="${MeshPath}/Leg3_Link1.STL" />
       </geometry>
     </collision>
@@ -624,17 +624,17 @@
       <geometry>
         <mesh
-        filename="package://rviz_basic/Leg3_Link2.STL" />
-      </geometry>
-      <material
-        name="Black">
-      </material>
-    </visual>
-    <collision>
-      <origin
-        xyz="0 0 0"
-        rpy="0 0 0" />
-      <geometry>
-        <mesh
-        filename="package://rviz_basic/Leg3_Link2.STL" />
+        filename="${MeshPath}/Leg3_Link2.STL" />
+      </geometry>
+      <material
+        name="Black">
+      </material>
+    </visual>
+    <collision>
+      <origin
+        xyz="0 0 0"
+        rpy="0 0 0" />
+      <geometry>
+        <mesh
+        filename="${MeshPath}/Leg3_Link2.STL" />
       </geometry>
     </collision>
@@ -680,17 +680,17 @@
       <geometry>
         <mesh
-        filename="package://rviz_basic/Leg3_Link3.STL" />
-      </geometry>
-      <material
-        name="Black">
-      </material>
-    </visual>
-    <collision>
-      <origin
-        xyz="0 0 0"
-        rpy="0 0 0" />
-      <geometry>
-        <mesh
-        filename="package://rviz_basic/Leg3_Link3.STL" />
+        filename="${MeshPath}/Leg3_Link3.STL" />
+      </geometry>
+      <material
+        name="Black">
+      </material>
+    </visual>
+    <collision>
+      <origin
+        xyz="0 0 0"
+        rpy="0 0 0" />
+      <geometry>
+        <mesh
+        filename="${MeshPath}/Leg3_Link3.STL" />
       </geometry>
     </collision>

Commit message: source fixed

File: src/rviz_basic/urdf/hero_3wheel_1hand/hero_3wheel_1hand.xacro (robot description, xacro)
@@ -915,5 +915,5 @@
   <parent link="Arm_PitchLink1_2"/>
   <child link="Arm_RollLink2_2"/>
-  <axis xyz="0.642788 -0.0 0.766044"/>
+  <axis xyz="0.642788 0.0 0.766044"/>
 </joint>
 <joint name="Arm_Pitch2" type="continuous">

File: src/rviz_basic/urdf/moonbot_hero/moonbot_hero.xacro (robot description, xacro)
@@ -1074,9 +1074,9 @@
 </joint>
 <joint name="Revolute 34" type="continuous">
-<!-- <origin xyz="0.0 -0.03266 -0.023094" rpy="${0 * 3.14 / 180} ${0 * 3.14 / 180} ${0 * 3.14 / 180}"/> -->
+<!-- <origin xyz="0.0 -0.03266 -0.023094" rpy="${-35 * 3.14 / 180} ${-35 * 3.14 / 180} ${90 * 3.14 / 180}"/> -->
   <origin xyz="0.0 -0.03266 -0.023094" rpy="0.0 -0.0 -0.0"/>
   <parent link="LegHip_2"/>
   <child link="LegRoll1Link_2"/>
-  <!-- <axis xyz="0.0 0.0 1.0"/> -->
+  <!-- <axis xyz="1.0 0.0 0.0"/> -->
   <axis xyz="0.0 -0.816497 -0.57735"/>
 </joint>
