Commit message: it owrks but rot quat is needed

File: src/rviz_basic/urdf/moonbot_hero/moonbot_hero.xacro (robot description, xacro)
@@ -1224,7 +1224,9 @@
 </joint>
 <joint name="Revolute 103" type="continuous">
+<!-- <joint name="Revolute 103" type="fixed"> -->
   <origin xyz="-0.017532 -0.043284 -0.101582" rpy="0 0 0"/>
   <parent link="Leg2_Pitch3Link_1"/>
   <child link="Leg2_Ankle_1"/>
+  <!-- <axis xyz="0 0 -1"/> -->
   <axis xyz="0.022311 0.026135 -0.999409"/>
 </joint>
