Commit message: urdf up

File: src/rviz_basic/urdf/moonbot_7/moonbot_7.xacro (robot description, xacro)
@@ -5,4 +5,10 @@
 <xacro:property name="UrdfDataPath" value="package://${ThisPackage}/urdf/${Filename}" />
 <xacro:property name="MeshPath" value="package://${ThisPackage}/meshes/${Filename}" />
+<xacro:property name="LimUpJ3" value="2.1" />
+<xacro:property name="LimLowJ3" value="0" />
+<xacro:property name="LimUpJ2" value="2.1" />
+<xacro:property name="LimLowJ2" value="0" />
+<xacro:property name="LimUpJ1" value="1.57" />
+<xacro:property name="LimLowJ1" value="1.57" />
   <material name="Grey">
       <color rgba="0.9 0.9 0.98 1" />
@@ -205,6 +211,6 @@
       xyz="0 0 -1" />
     <limit
-      lower="0"
-      upper="0"
+      lower="${LimLowJ3}"
+      upper="${LimUpJ3}"
       effort="0"
       velocity="0" />

Commit message: demo

File: src/rviz_basic/urdf/moonbot_7/moonbot_7.xacro (robot description, xacro)
@@ -5,10 +5,10 @@
 <xacro:property name="UrdfDataPath" value="package://${ThisPackage}/urdf/${Filename}" />
 <xacro:property name="MeshPath" value="package://${ThisPackage}/meshes/${Filename}" />
-<xacro:property name="LimUpJ3" value="2.1" />
-<xacro:property name="LimLowJ3" value="0" />
+<xacro:property name="LimUpJ3" value="3.1" />
+<xacro:property name="LimLowJ3" value="-0.25" />
 <xacro:property name="LimUpJ2" value="2.1" />
-<xacro:property name="LimLowJ2" value="0" />
+<xacro:property name="LimLowJ2" value="-2.1" />
 <xacro:property name="LimUpJ1" value="1.57" />
-<xacro:property name="LimLowJ1" value="1.57" />
+<xacro:property name="LimLowJ1" value="-1.57" />
   <material name="Grey">
       <color rgba="0.9 0.9 0.98 1" />
@@ -99,6 +99,6 @@
       xyz="0 0 -1" />
     <limit
-      lower="0"
-      upper="0"
+      lower="${LimLowJ1}"
+      upper="${LimUpJ1}"
       effort="0"
       velocity="0" />
@@ -155,6 +155,6 @@
       xyz="0 0 1" />
     <limit
-      lower="0"
-      upper="0"
+      lower="${LimLowJ2}"
+      upper="${LimUpJ2}"
       effort="0"
       velocity="0" />
@@ -267,6 +267,6 @@
       xyz="0 0 -1" />
     <limit
-      lower="0"
-      upper="0"
+      lower="${LimLowJ1}"
+      upper="${LimUpJ1}"
       effort="0"
       velocity="0" />
@@ -323,6 +323,6 @@
       xyz="0 0 1" />
     <limit
-      lower="0"
-      upper="0"
+      lower="${LimLowJ2}"
+      upper="${LimUpJ2}"
       effort="0"
       velocity="0" />
@@ -379,6 +379,6 @@
       xyz="0 0 -1" />
     <limit
-      lower="0"
-      upper="0"
+      lower="${LimLowJ3}"
+      upper="${LimUpJ3}"
       effort="0"
       velocity="0" />
@@ -435,6 +435,6 @@
       xyz="0 0 -1" />
     <limit
-      lower="0"
-      upper="0"
+      lower="${LimLowJ1}"
+      upper="${LimUpJ1}"
       effort="0"
       velocity="0" />
@@ -491,6 +491,6 @@
       xyz="0 0 1" />
     <limit
-      lower="0"
-      upper="0"
+      lower="${LimLowJ2}"
+      upper="${LimUpJ2}"
       effort="0"
       velocity="0" />
@@ -547,6 +547,6 @@
       xyz="0 0 -1" />
     <limit
-      lower="0"
-      upper="0"
+      lower="${LimLowJ3}"
+      upper="${LimUpJ3}"
       effort="0"
       velocity="0" />
@@ -603,6 +603,6 @@
       xyz="0 0 -1" />
     <limit
-      lower="0"
-      upper="0"
+      lower="${LimLowJ1}"
+      upper="${LimUpJ1}"
       effort="0"
       velocity="0" />
@@ -659,6 +659,6 @@
       xyz="0 0 1" />
     <limit
-      lower="0"
-      upper="0"
+      lower="${LimLowJ2}"
+      upper="${LimUpJ2}"
       effort="0"
       velocity="0" />
@@ -715,6 +715,6 @@
       xyz="0 0 -1" />
     <limit
-      lower="0"
-      upper="0"
+      lower="${LimLowJ3}"
+      upper="${LimUpJ3}"
       effort="0"
       velocity="0" />

Commit message: moonwalk fast

File: src/rviz_basic/urdf/moonbot_7/moonbot_7.xacro (robot description, xacro)
@@ -5,10 +5,10 @@
 <xacro:property name="UrdfDataPath" value="package://${ThisPackage}/urdf/${Filename}" />
 <xacro:property name="MeshPath" value="package://${ThisPackage}/meshes/${Filename}" />
-<xacro:property name="LimUpJ3" value="3.1" />
-<xacro:property name="LimLowJ3" value="-0.25" />
-<xacro:property name="LimUpJ2" value="2.1" />
-<xacro:property name="LimLowJ2" value="-2.1" />
-<xacro:property name="LimUpJ1" value="1.57" />
-<xacro:property name="LimLowJ1" value="-1.57" />
+<xacro:property name="LimUpJ3" value="2.5" />
+<xacro:property name="LimLowJ3" value="-0.5" />
+<xacro:property name="LimUpJ2" value="1.8" />
+<xacro:property name="LimLowJ2" value="-1.8" />
+<xacro:property name="LimUpJ1" value="1.8" />
+<xacro:property name="LimLowJ1" value="-1.8" />
   <material name="Grey">
       <color rgba="0.9 0.9 0.98 1" />
