Commit message: better funcs and dragon pose pretty

File: src/urdf_packer/urdf/hero_7dof/wheel_macro.xacro (robot description, xacro)
@@ -87,5 +87,5 @@
     <parent link="${prefix}wheel_body"/>
     <child link="${prefix}wheel_left"/>
-    <axis xyz="0.0 1.0 0.0"/>
+    <axis xyz="0 1 0"/>
   </joint>
   <joint name="${prefix}wheel_right_joint" type="continuous">
@@ -93,5 +93,5 @@
     <parent link="${prefix}wheel_body"/>
     <child link="${prefix}wheel_right"/>
-    <axis xyz="-0.0 -1.0 -0.0"/>
+    <axis xyz="0 1 0"/>
   </joint>
   <joint name="${prefix}wheel_cen2out" type="fixed">
