Commit message: single launch changed to all testing everything

File: src/urdf_packer/urdf/hero_7dof/hero_7dofm1.xacro (robot description, xacro)
@@ -1,18 +1,17 @@
 <?xml version="1.0"?>
-<robot xmlns:xacro="http://www.ros.org/wiki/xacro" name="hero_7dofm3">
+<robot xmlns:xacro="http://www.ros.org/wiki/xacro" name="hero_7dofm1">
 <xacro:property name="ThisPackage" value="urdf_packer" />
 <xacro:property name="Filename" value="hero_7dof" />
 <xacro:property name="UrdfDataPath" value="package://${ThisPackage}/urdf/${Filename}" />
 <xacro:property name="MeshPath" value="package://${ThisPackage}/meshes/${Filename}" />
-  <!-- Include the original xacro file -->
 <xacro:include filename="${Filename}.xacro"/>
-  <!-- Override specific properties -->
-<xacro:property name="off_base_link_link2" value="-1.5968164926267214" />
-<xacro:property name="off_link2_link3" value="-1.5249186659861529" />
-<xacro:property name="off_link3_link4" value="-1.1246189568997114" />
-<xacro:property name="off_link4_link5" value="-1.2173329162057398" />
-<xacro:property name="off_link5_link6" value="-0.4995871839710359" />
-<xacro:property name="off_link6_link7" value="-1.6035269564465078" />
-<xacro:property name="off_link7_link8" value="-0.8002183286638307" />
-  <!-- Rest of your new robot description -->
+<xacro:get_hero prefix = "leg1"
+off_base_link_link2 = "-1.5968164926267214"
+off_link2_link3 = "-1.5249186659861529"
+off_link3_link4 = "-1.1246189568997114"
+off_link4_link5 = "-1.2173329162057398"
+off_link5_link6 = "-0.4995871839710359"
+off_link6_link7 = "-1.6035269564465078"
+off_link7_link8 = "-0.8002183286638307"
+/>
 </robot>

File: src/urdf_packer/urdf/hero_7dof/hero_7dofm2.xacro (robot description, xacro)
@@ -1,9 +1,8 @@
 <?xml version="1.0"?>
-<robot xmlns:xacro="http://www.ros.org/wiki/xacro" name="hero_7dofm4">
+<robot xmlns:xacro="http://www.ros.org/wiki/xacro" name="hero_7dofm2">
 <xacro:property name="ThisPackage" value="urdf_packer" />
 <xacro:property name="Filename" value="hero_7dof" />
 <xacro:property name="UrdfDataPath" value="package://${ThisPackage}/urdf/${Filename}" />
 <xacro:property name="MeshPath" value="package://${ThisPackage}/meshes/${Filename}" />
-  <!-- Include the original xacro file -->
 <xacro:include filename="${Filename}.xacro"/>
 <xacro:get_hero prefix = "leg2"
