Commit message: gragon fixed

File: src/urdf_packer/urdf/hero_7dof/hero_7dofflipped.xacro (robot description, xacro)
@@ -1,2 +1,24 @@
+<!-- THIS DOES NOT WORK -->
+<!-- THIS DOES NOT WORK -->
+<!-- THIS DOES NOT WORK -->
+<!-- THIS DOES NOT WORK -->
+<!-- THIS DOES NOT WORK -->
+<!-- THIS DOES NOT WORK -->
+<!-- THIS DOES NOT WORK -->
+<!-- THIS DOES NOT WORK -->
+<!-- THIS DOES NOT WORK -->
+<!-- THIS DOES NOT WORK -->
+<!-- THIS DOES NOT WORK -->
+<!-- THIS DOES NOT WORK -->
+<!-- THIS DOES NOT WORK -->
+<!-- THIS DOES NOT WORK -->
+<!-- THIS DOES NOT WORK -->
+<!-- THIS DOES NOT WORK -->
+<!-- THIS DOES NOT WORK -->
+<!-- THIS DOES NOT WORK -->
+<!-- THIS DOES NOT WORK -->
+<!-- THIS DOES NOT WORK -->
+<!-- THIS DOES NOT WORK -->
+<!-- THIS DOES NOT WORK -->
 <?xml version="1.0" encoding="utf-8"?>
 <robot name="hero_7dof" xmlns:xacro="http://www.ros.org/wiki/xacro">
@@ -108,5 +130,5 @@
     </collision>
   </link>
-  <joint name="${prefix}base_link-link2" type="continuous">
+  <joint name="${prefix}link7-link8" type="continuous">
     <origin xyz="0 0 0.05" rpy="0 0 0" />
     <parent link="${prefix}gripper1" />
@@ -155,5 +177,5 @@
     </collision>
   </link>
-  <joint name="${prefix}link2-link3" type="continuous">
+  <joint name="${prefix}link6-link7" type="continuous">
     <origin xyz="0.00016471 -0.090096 0.16854" rpy="0 1.57 0" />
     <parent link="${prefix}link2" />
@@ -202,5 +224,5 @@
     </collision>
   </link>
-  <joint name="${prefix}link3-link4" type="continuous">
+  <joint name="${prefix}link5-link6" type="continuous">
     <origin xyz="0 -0.058547 0.071444" rpy="0 0 1.57" />
     <parent link="${prefix}link3" />
@@ -296,5 +318,5 @@
     </collision>
   </link>
-  <joint name="${prefix}link5-link6" type="continuous">
+  <joint name="${prefix}link3-link4" type="continuous">
     <origin xyz="0.12633 0 0.42742" rpy="0 0 1.57" />
     <parent link="${prefix}link5" />
@@ -342,5 +364,5 @@
     </collision>
   </link>
-  <joint name="${prefix}link6-link7" type="continuous">
+  <joint name="${prefix}link2-link3" type="continuous">
     <origin xyz="0 0.12032 0.072384" rpy="0 -1.57 0" />
     <parent link="${prefix}link6" />
@@ -389,5 +411,5 @@
     </collision>
   </link>
-  <joint name="${prefix}link7-link8" type="continuous">
+  <joint name="${prefix}base_link-link2" type="continuous">
     <origin xyz="0 0.029477 0.15419" rpy="0 0 0" />
     <parent link="${prefix}link7" />

File: src/urdf_packer/urdf/hero_7dof/hero_dragon.xacro (robot description, xacro)
@@ -15,5 +15,5 @@
 <xacro:include filename="wheel_macro.xacro"/>
 <joint name="bfix" type="fixed">
-<origin xyz="0 0 0" rpy="${1*pi/4} 0 0"/>
+<origin xyz="0 0 0" rpy="${1*pi/4} 0 ${-pi/2}"/>
 <parent link="base_link"/>
 <child link="base_link45"/>
