Commit message: working on all 3 legs

File: src/urdf_packer/urdf/hero_7dof/hero_3leg.xacro (robot description, xacro)
@@ -32,15 +32,15 @@
 <joint name="fix2" type="fixed">
 <origin xyz="${R} 0 0" rpy="0 ${pi/2} 0"/>
-<parent link="d2"/>
+<parent link="d3"/>
 <child link="leg2gripper1"/>
 </joint>
 <joint name="fix3" type="fixed">
 <origin xyz="${R} 0 0" rpy="0 ${pi/2} 0"/>
-<parent link="d3"/>
-<child link="leg3gripper1"/>
+<parent link="d2"/>
+<child link="leg4gripper1"/>
 </joint>
 <xacro:include filename="hero_7dofm1.xacro"/>
 <xacro:include filename="hero_7dofm2.xacro"/>
-<xacro:include filename="hero_7dofm3.xacro"/>
+<xacro:include filename="hero_7dofm4.xacro"/>
 <!-- <xacro:include filename="hero_7dofm4.xacro"/> -->
 <!-- <joint name="fix4" type="fixed"> -->

Commit message: pi checked and leg up

File: src/urdf_packer/urdf/hero_7dof/hero_3leg.xacro (robot description, xacro)
@@ -9,5 +9,5 @@
 <link name="d1" />
 <joint name="orient1" type="fixed">
-<origin xyz="0 0 0" rpy="0 0 0"/>
+<origin xyz="0 0 0" rpy="${pi} 0 0"/>
 <parent link="base_link"/>
 <child link="d1"/>
@@ -15,5 +15,5 @@
 <link name="d2" />
 <joint name="orient2" type="fixed">
-<origin xyz="0 0 0" rpy="0 0 ${2*pi/3}"/>
+<origin xyz="0 0 0" rpy="${pi} 0 ${2*pi/3}"/>
 <parent link="base_link"/>
 <child link="d2"/>
@@ -21,5 +21,5 @@
 <link name="d3" />
 <joint name="orient3" type="fixed">
-<origin xyz="0 0 0" rpy="0 0 ${2*2*pi/3}"/>
+<origin xyz="0 0 0" rpy="${pi} 0 ${-1*2*pi/3}"/>
 <parent link="base_link"/>
 <child link="d3"/>

Commit message: leg 3 front tricycle

File: src/urdf_packer/urdf/hero_7dof/hero_3leg.xacro (robot description, xacro)
@@ -21,5 +21,5 @@
 <link name="d3" />
 <joint name="orient3" type="fixed">
-<origin xyz="0 0 0" rpy="${pi} 0 ${-1*2*pi/3}"/>
+<origin xyz="0 0 0" rpy="${pi} 0 ${2*2*pi/3}"/>
 <parent link="base_link"/>
 <child link="d3"/>
@@ -28,19 +28,19 @@
 <origin xyz="${R} 0 0" rpy="0 ${pi/2} 0"/>
 <parent link="d1"/>
-<child link="leg1gripper1"/>
+<child link="leg3gripper1"/>
 </joint>
 <joint name="fix2" type="fixed">
 <origin xyz="${R} 0 0" rpy="0 ${pi/2} 0"/>
 <parent link="d3"/>
-<child link="leg2gripper1"/>
+<child link="leg1gripper1"/>
 </joint>
 <joint name="fix3" type="fixed">
 <origin xyz="${R} 0 0" rpy="0 ${pi/2} 0"/>
 <parent link="d2"/>
-<child link="leg4gripper1"/>
+<child link="leg2gripper1"/>
 </joint>
 <xacro:include filename="hero_7dofm1.xacro"/>
 <xacro:include filename="hero_7dofm2.xacro"/>
-<xacro:include filename="hero_7dofm4.xacro"/>
+<xacro:include filename="hero_7dofm3.xacro"/>
 <!-- <xacro:include filename="hero_7dofm4.xacro"/> -->
 <!-- <joint name="fix4" type="fixed"> -->

Commit message: leg 4 instead of 1

File: src/urdf_packer/urdf/hero_7dof/hero_3leg.xacro (robot description, xacro)
@@ -33,5 +33,5 @@
 <origin xyz="${R} 0 0" rpy="0 ${pi/2} 0"/>
 <parent link="d3"/>
-<child link="leg1gripper1"/>
+<child link="leg4gripper1"/>
 </joint>
 <joint name="fix3" type="fixed">
@@ -40,5 +40,5 @@
 <child link="leg2gripper1"/>
 </joint>
-<xacro:include filename="hero_7dofm1.xacro"/>
+<xacro:include filename="hero_7dofm4.xacro"/>
 <xacro:include filename="hero_7dofm2.xacro"/>
 <xacro:include filename="hero_7dofm3.xacro"/>

Commit message: leg2 flipped on tricycle

File: src/urdf_packer/urdf/hero_7dof/hero_3leg.xacro (robot description, xacro)
@@ -7,4 +7,6 @@
 <xacro:property name="R" value="0.300" />
 <link name="base_link" />
+<link name="base_linkp" />
+<!-- fake end of gripper 3-2 -->
 <link name="d1" />
 <joint name="orient1" type="fixed">
@@ -12,4 +14,10 @@
 <parent link="base_link"/>
 <child link="d1"/>
+</joint>
+<link name="d1p" />
+<joint name="orient1p" type="fixed">
+<origin xyz="0 0 0" rpy="0 0 0"/>
+<parent link="d1p"/>
+<child link="base_linkp"/>
 </joint>
 <link name="d2" />
@@ -29,4 +37,9 @@
 <parent link="d1"/>
 <child link="leg3gripper1"/>
+</joint>
+<joint name="fix1p" type="fixed">
+<origin xyz="${R} 0 0" rpy="${pi} 0 ${pi}"/>
+<parent link="leg3gripper2_straight"/>
+<child link="d1p"/>
 </joint>
 <joint name="fix2" type="fixed">

Commit message: replaced leg 3 with 4, better james bond

File: src/urdf_packer/urdf/hero_7dof/hero_3leg.xacro (robot description, xacro)
@@ -36,9 +36,9 @@
 <origin xyz="${R} 0 0" rpy="0 ${pi/2} 0"/>
 <parent link="d1"/>
-<child link="leg3gripper1"/>
+<child link="leg1gripper1"/>
 </joint>
 <joint name="fix1p" type="fixed">
 <origin xyz="${R} 0 0" rpy="${pi} 0 ${pi}"/>
-<parent link="leg3gripper2_straight"/>
+<parent link="leg1gripper2_straight"/>
 <child link="d1p"/>
 </joint>
@@ -55,5 +55,5 @@
 <xacro:include filename="hero_7dofm4.xacro"/>
 <xacro:include filename="hero_7dofm2.xacro"/>
-<xacro:include filename="hero_7dofm3.xacro"/>
+<xacro:include filename="hero_7dofm1.xacro"/>
 <!-- <xacro:include filename="hero_7dofm4.xacro"/> -->
 <!-- <joint name="fix4" type="fixed"> -->

File: src/urdf_packer/urdf/hero_7dof/hero_7dof_all.xacro (robot description, xacro)
@@ -7,20 +7,20 @@
 <link name="base_link" />
 <joint name="fix1" type="fixed">
-<origin xyz="0 0 0" rpy="0 0 0"/>
+<origin xyz="-0.6 0 0" rpy="0 0 0"/>
 <parent link="base_link"/>
 <child link="leg1gripper1"/>
 </joint>
 <joint name="fix2" type="fixed">
-<origin xyz="0 0 0.4" rpy="0 0 0"/>
+<origin xyz="0.6 0 0" rpy="0 0 0"/>
 <parent link="base_link"/>
 <child link="leg2gripper1"/>
 </joint>
 <joint name="fix3" type="fixed">
-<origin xyz="0 0 0.8" rpy="0 0 0"/>
+<origin xyz="-1.4 0 0" rpy="0 0 0"/>
 <parent link="base_link"/>
 <child link="leg3gripper1"/>
 </joint>
 <joint name="fix4" type="fixed">
-<origin xyz="1 0 0.12" rpy="0 0 0"/>
+<origin xyz="1.4 0 0" rpy="0 0 0"/>
 <parent link="base_link"/>
 <child link="leg4gripper1"/>
@@ -33,5 +33,5 @@
 <xacro:add_wheel prefix="11" />
 <joint name="fix11" type="fixed">
-<origin xyz="0 0 0" rpy="0 0 0"/>
+<origin xyz="0.2 2 0" rpy="0 0 ${pi/2}"/>
 <parent link="base_link"/>
 <child link="11wheel_in"/>
@@ -39,5 +39,5 @@
 <xacro:add_wheel prefix="12" />
 <joint name="fix12" type="fixed">
-<origin xyz="0 0 0" rpy="0 0 0"/>
+<origin xyz="0.6 2 0" rpy="0 0 ${pi/2}"/>
 <parent link="base_link"/>
 <child link="12wheel_in"/>
@@ -45,5 +45,5 @@
 <xacro:add_wheel prefix="13" />
 <joint name="fix13" type="fixed">
-<origin xyz="0 0 0" rpy="0 0 0"/>
+<origin xyz="1 2 0" rpy="0 0 ${pi/2}"/>
 <parent link="base_link"/>
 <child link="13wheel_in"/>
@@ -51,5 +51,5 @@
 <xacro:add_wheel prefix="14" />
 <joint name="fix14" type="fixed">
-<origin xyz="0 0 0" rpy="0 0 0"/>
+<origin xyz="1.4 2 0" rpy="0 0 ${pi/2}"/>
 <parent link="base_link"/>
 <child link="14wheel_in"/>

File: src/urdf_packer/urdf/hero_7dof/hero_dragon.xacro (robot description, xacro)
@@ -8,7 +8,7 @@
 <!-- also change that here !!!!    V   -->
 <xacro:include filename="hero_7dofm2.xacro" ns="leg${main_leg}"/>
-<xacro:property name="manip_leg" value="3" />
+<xacro:property name="manip_leg" value="4" />
 <!-- also change that here !!!!    V   -->
-<xacro:include filename="hero_7dofm3.xacro" ns="leg${manip_leg}"/>
+<xacro:include filename="hero_7dofm4.xacro" ns="leg${manip_leg}"/>
   <!-- Include the original xacro file -->
 <link name="base_link" />

Commit message: Add central hub visual mesh

File: src/urdf_packer/urdf/hero_7dof/hero_3leg.xacro (robot description, xacro)
@@ -6,5 +6,18 @@
 <xacro:property name="MeshPath" value="package://${ThisPackage}/meshes/${Filename}" />
 <xacro:property name="R" value="0.300" />
-<link name="base_link" />
+<link name="base_link">
+    <visual>
+	<origin xyz="0 0 0" rpy="0 0 1.04" />
+      <geometry>
+        <mesh filename="${MeshPath}/hero_hub_unit.stl" scale="0.001 0.001 0.001">
+	</mesh>
+      </geometry>
+	<material
+        name="">
+        <color
+          rgba="0.627450980392157 0.627450980392157 0.627450980392157 1" />
+      </material>
+    </visual>
+</link>
 <link name="base_linkp" />
 <!-- fake end of gripper 3-2 -->

Commit message: Fix limb/hub attachment position

File: src/urdf_packer/urdf/hero_7dof/hero_3leg.xacro (robot description, xacro)
@@ -5,5 +5,5 @@
 <xacro:property name="UrdfDataPath" value="package://${ThisPackage}/urdf/${Filename}" />
 <xacro:property name="MeshPath" value="package://${ThisPackage}/meshes/${Filename}" />
-<xacro:property name="R" value="0.300" />
+<xacro:property name="R" value="0.200" />
 <link name="base_link" />
 <link name="base_linkp" />
