Commit message: vehicle mode

File: src/urdf_packer/urdf/hero_7dof/hero_vehicle.xacro (robot description, xacro)
@@ -5,11 +5,7 @@
   <xacro:property name="UrdfDataPath" value="package://${ThisPackage}/urdf/${Filename}"></xacro:property>
   <xacro:property name="MeshPath" value="package://${ThisPackage}/meshes/${Filename}"></xacro:property>
-  <xacro:property name="main_leg" value="2"></xacro:property>
+  <xacro:property name="main_leg" value="4"></xacro:property>
   <!-- also change that here !!!!    V   -->
-  <xacro:include filename="hero_7dofm2.xacro" ns="leg${main_leg}"></xacro:include>
-  <xacro:property name="manip_leg" value="4"></xacro:property>
-  <!-- also change that here !!!!    V   -->
-  <xacro:include filename="hero_7dofm4.xacro" ns="leg${manip_leg}"></xacro:include>
-  <!-- Include the original xacro file -->
+  <xacro:include filename="hero_7dofm4.xacro" ns="leg${main_leg}"></xacro:include>
   <link name="base_link"></link>
   <xacro:include filename="wheel_macro.xacro"></xacro:include>
@@ -21,6 +17,6 @@
   <link name="base_link45"></link>
   <joint name="bfixstraight" type="fixed">
-    <origin rpy="0 0 0" xyz="0 0 0.165"></origin>
-    <parent link="base_link45"></parent>
+    <origin rpy="0 0 ${-pi/2}" xyz="0 0 0.165"></origin>
+    <parent link="base_link"></parent>
     <child link="1wheel_in"></child>
   </joint>
@@ -49,15 +45,3 @@
     <child link="wheel2c45"></child>
   </joint>
-  <joint name="fixwheel1-2" type="fixed">
-    <origin rpy="0 0 0" xyz="0 0 0"></origin>
-    <parent link="1wheel_out"></parent>
-    <child link="leg${manip_leg}gripper1"></child>
-  </joint>
-  <!-- <xacro:add_wheel  prefix="${manip_leg}" /> -->
-  <!---->
-  <!-- <joint name="fixwheel1-${manip_leg}" type="fixed"> -->
-  <!-- <origin xyz="0 0 0" rpy="0 0 0"/> -->
-  <!-- <parent link="leg4gripper2"/> -->
-  <!-- <child link="${manip_leg}wheel_in"/> -->
-  <!-- </joint> -->
 </robot>
