Commit message: why is it broken

File: src/urdf_packer/urdf/hero_7dof/hero_7dof.xacro (robot description, xacro)
@@ -9,4 +9,6 @@
 <xacro:property name="UrdfDataPath" value="package://${ThisPackage}/urdf/${Filename}" />
 <xacro:property name="MeshPath" value="package://${ThisPackage}/meshes/${Filename}" />
+<!-- use this instead for moveit or other stuff -->
+<!-- <xacro:property name="MeshPath" value="package://new_hero/meshes" /> -->
   <link name="base_link">
     <inertial>
@@ -375,4 +377,18 @@
     <limit effort="100.0" velocity="1300"/>
   </joint>
+  <link
+  name="gripper2">
+  </link>
+  <joint
+    name="eefix"
+    type="fixed">
+    <origin
+      xyz="0 0 0.06"
+      rpy="0 0 0" />
+    <parent
+      link="link8" />
+    <child
+      link="gripper2" />
+  </joint>
   <transmission name="link2_trans">
     <type>transmission_interface/SimpleTransmission</type>

Commit message: working on the arm

File: src/urdf_packer/urdf/hero_7dof/hero_7dof.xacro (robot description, xacro)
@@ -140,5 +140,5 @@
     <parent link="link2" />
     <child link="link3" />
-    <axis xyz="0 1 0" />
+    <axis xyz="0 -1 0" />
     <dynamics damping="0.7"/>
     <limit effort="100.0" velocity="1300"/>
@@ -234,5 +234,5 @@
     <parent link="link4" />
     <child link="link5" />
-    <axis xyz="-1 0 0" />
+    <axis xyz="1 0 0" />
     <dynamics damping="0.7"/>
     <limit effort="100.0" velocity="1300"/>
@@ -326,5 +326,5 @@
     <parent link="link6" />
     <child link="link7" />
-    <axis xyz="0 -1 0" />
+    <axis xyz="0 1 0" />
     <dynamics damping="0.7"/>
     <limit effort="100.0" velocity="1300"/>

Commit message: oh my god it keeps crashing

File: src/urdf_packer/urdf/hero_7dof/hero_7dof.xacro (robot description, xacro)
@@ -373,5 +373,5 @@
     <parent link="link7" />
     <child link="link8" />
-    <axis xyz="0 0 -1" />
+    <axis xyz="0 0 1" />
     <dynamics damping="0.7"/>
     <limit effort="100.0" velocity="1300"/>

Commit message: joint limit

File: src/urdf_packer/urdf/hero_7dof/hero_7dof.xacro (robot description, xacro)
@@ -11,4 +11,25 @@
 <!-- use this instead for moveit or other stuff -->
 <!-- <xacro:property name="MeshPath" value="package://new_hero/meshes" /> -->
+<xacro:property name="off_base_link_link2" value="-1.5968164926267214" />
+<xacro:property name="off_link2_link3" value="-1.5249186659861529" />
+<xacro:property name="off_link3_link4" value="-1.1246189568997114" />
+<xacro:property name="off_link4_link5" value="-1.2173329162057398" />
+<xacro:property name="off_link5_link6" value="-0.4995871839710359" />
+<xacro:property name="off_link6_link7" value="-1.6035269564465078" />
+<xacro:property name="off_link7_link8" value="-0.8002183286638307" />
+<xacro:property name="max_base_link_link2" value="${-1 * off_base_link_link2}" />
+<xacro:property name="max_link2_link3" value="${-1 * off_link2_link3}" />
+<xacro:property name="max_link3_link4" value="${-1 * off_link3_link4}" />
+<xacro:property name="max_link4_link5" value="${-1 * off_link4_link5}" />
+<xacro:property name="max_link5_link6" value="${-1 * off_link5_link6}" />
+<xacro:property name="max_link6_link7" value="${-1 * off_link6_link7}" />
+<xacro:property name="max_link7_link8" value="${-1 * off_link7_link8}" />
+<xacro:property name="min_base_link_link2" value="${-1 * off_base_link_link2 - pi}" />
+<xacro:property name="min_link2_link3" value="${-1 * off_link2_link3 - pi}" />
+<xacro:property name="min_link3_link4" value="${-1 * off_link3_link4 - pi}" />
+<xacro:property name="min_link4_link5" value="${-1 * off_link4_link5 - pi}" />
+<xacro:property name="min_link5_link6" value="${-1 * off_link5_link6 - pi}" />
+<xacro:property name="min_link6_link7" value="${-1 * off_link6_link7 - pi}" />
+<xacro:property name="min_link7_link8" value="${-1 * off_link7_link8 - pi}" />
   <link name="base_link">
     <inertial>
@@ -95,5 +116,5 @@
     <axis xyz="0 0 1" />
     <dynamics damping="0.7"/>
-    <limit effort="100.0" velocity="1300"/>
+    <limit upper="${max_base_link_link2}" lower="${min_base_link_link2}" effort="100.0" velocity="1300"/>
   </joint>
   <link name="link3">
@@ -142,5 +163,5 @@
     <axis xyz="0 -1 0" />
     <dynamics damping="0.7"/>
-    <limit effort="100.0" velocity="1300"/>
+    <limit upper="${max_link2_link3}" lower="${min_link2_link3}" effort="100.0" velocity="1300"/>
   </joint>
   <link name="link4">
@@ -189,5 +210,5 @@
     <axis xyz="0 0 1" />
     <dynamics damping="0.7"/>
-    <limit effort="100.0" velocity="1300"/>
+    <limit upper="${max_link3_link4}" lower="${min_link3_link4}" effort="100.0" velocity="1300"/>
   </joint>
   <link name="link5">
@@ -236,5 +257,5 @@
     <axis xyz="1 0 0" />
     <dynamics damping="0.7"/>
-    <limit effort="100.0" velocity="1300"/>
+    <limit upper="${max_link4_link5}" lower="${min_link4_link5}" effort="100.0" velocity="1300"/>
   </joint>
   <link  name="link6">
@@ -282,4 +303,5 @@
     <child link="link6" />
     <axis xyz="0 0 1" />
+    <limit upper="${max_link5_link6}" lower="${min_link5_link6}" effort="100.0" velocity="1300"/>
   </joint>
   <link name="link7">
@@ -328,5 +350,5 @@
     <axis xyz="0 1 0" />
     <dynamics damping="0.7"/>
-    <limit effort="100.0" velocity="1300"/>
+    <limit upper="${max_link6_link7}" lower="${min_link6_link7}" effort="100.0" velocity="1300"/>
   </joint>
   <link  name="link8">
@@ -375,5 +397,5 @@
     <axis xyz="0 0 1" />
     <dynamics damping="0.7"/>
-    <limit effort="100.0" velocity="1300"/>
+    <limit upper="${max_link7_link8}" lower="${min_link7_link8}" effort="100.0" velocity="1300"/>
   </joint>
   <link

Commit message: new colored mesh

File: src/urdf_packer/urdf/hero_7dof/hero_7dof.xacro (robot description, xacro)
@@ -32,4 +32,5 @@
 <xacro:property name="min_link6_link7" value="${-1 * off_link6_link7 - pi}" />
 <xacro:property name="min_link7_link8" value="${-1 * off_link7_link8 - pi}" />
+<xacro:property name="mesh_extension" value="dae" />
   <link name="base_link">
     <inertial>
@@ -53,5 +54,5 @@
       <geometry>
         <mesh
-        filename="${MeshPath}/base_link.STL" />
+        filename="${MeshPath}/base_link.${mesh_extension}" />
       </geometry>
       <material
@@ -67,5 +68,5 @@
       <geometry>
         <mesh
-        filename="${MeshPath}/base_link.STL" />
+        filename="${MeshPath}/base_link.${mesh_extension}" />
       </geometry>
     </collision>
@@ -92,5 +93,5 @@
       <geometry>
         <mesh
-        filename="${MeshPath}/link2.STL" />
+        filename="${MeshPath}/link2.${mesh_extension}" />
       </geometry>
       <material
@@ -106,5 +107,5 @@
       <geometry>
         <mesh
-        filename="${MeshPath}/link2.STL" />
+        filename="${MeshPath}/link2.${mesh_extension}" />
       </geometry>
     </collision>
@@ -139,5 +140,5 @@
       <geometry>
         <mesh
-        filename="${MeshPath}/link3.STL" />
+        filename="${MeshPath}/link3.${mesh_extension}" />
       </geometry>
       <material
@@ -153,5 +154,5 @@
       <geometry>
         <mesh
-        filename="${MeshPath}/link3.STL" />
+        filename="${MeshPath}/link3.${mesh_extension}" />
       </geometry>
     </collision>
@@ -186,5 +187,5 @@
       <geometry>
         <mesh
-        filename="${MeshPath}/link4.STL" />
+        filename="${MeshPath}/link4.${mesh_extension}" />
       </geometry>
       <material
@@ -200,5 +201,5 @@
       <geometry>
         <mesh
-        filename="${MeshPath}/link4.STL" />
+        filename="${MeshPath}/link4.${mesh_extension}" />
       </geometry>
     </collision>
@@ -233,5 +234,5 @@
       <geometry>
         <mesh
-        filename="${MeshPath}/link5.STL" />
+        filename="${MeshPath}/link5.${mesh_extension}" />
       </geometry>
       <material
@@ -247,5 +248,5 @@
       <geometry>
         <mesh
-        filename="${MeshPath}/link5.STL" />
+        filename="${MeshPath}/link5.${mesh_extension}" />
       </geometry>
     </collision>
@@ -280,5 +281,5 @@
       <geometry>
         <mesh
-        filename="${MeshPath}/link6.STL" />
+        filename="${MeshPath}/link6.${mesh_extension}" />
       </geometry>
       <material
@@ -294,5 +295,5 @@
       <geometry>
         <mesh
-        filename="${MeshPath}/link6.STL" />
+        filename="${MeshPath}/link6.${mesh_extension}" />
       </geometry>
     </collision>
@@ -326,5 +327,5 @@
       <geometry>
         <mesh
-        filename="${MeshPath}/link7.STL" />
+        filename="${MeshPath}/link7.${mesh_extension}" />
       </geometry>
       <material
@@ -340,5 +341,5 @@
       <geometry>
         <mesh
-        filename="${MeshPath}/link7.STL" />
+        filename="${MeshPath}/link7.${mesh_extension}" />
       </geometry>
     </collision>
@@ -373,5 +374,5 @@
       <geometry>
         <mesh
-        filename="${MeshPath}/link8.STL" />
+        filename="${MeshPath}/link8.${mesh_extension}" />
       </geometry>
       <material
@@ -387,5 +388,5 @@
       <geometry>
         <mesh
-        filename="${MeshPath}/link8.STL" />
+        filename="${MeshPath}/link8.${mesh_extension}" />
       </geometry>
     </collision>
@@ -407,5 +408,5 @@
     <origin
       xyz="0 0 0.06"
-      rpy="0 0 0" />
+    rpy="0 ${-pi} ${-pi}" />
     <parent
       link="link8" />

Commit message: dragon moving rviz

File: src/urdf_packer/urdf/hero_7dof/hero_7dof.xacro (robot description, xacro)
@@ -33,5 +33,5 @@
 <xacro:property name="min_link7_link8" value="${-1 * off_link7_link8 - pi}" />
 <xacro:property name="mesh_extension" value="dae" />
-  <link name="base_link">
+  <link name="gripper1">
     <inertial>
       <origin
@@ -113,5 +113,5 @@
   <joint name="base_link-link2" type="continuous">
     <origin xyz="0 0 0.05" rpy="0 0 0" />
-    <parent link="base_link" />
+    <parent link="gripper1" />
     <child link="link2" />
     <axis xyz="0 0 1" />

Commit message: it does not work with this xacro

File: src/urdf_packer/urdf/hero_7dof/hero_7dof.xacro (robot description, xacro)
@@ -3,10 +3,11 @@
      Commit Version: 1.6.0-4-g7f85cfe  Build Version: 1.6.7995.38578
      For more information, please see http://wiki.ros.org/sw_urdf_exporter -->
-<robot
-  name="hero_7dof" xmlns:xacro="http://www.ros.org/wiki/xacro">
+<robot name="hero_7dof" xmlns:xacro="http://www.ros.org/wiki/xacro">
 <xacro:property name="ThisPackage" value="urdf_packer" />
 <xacro:property name="Filename" value="hero_7dof" />
 <xacro:property name="UrdfDataPath" value="package://${ThisPackage}/urdf/${Filename}" />
 <xacro:property name="MeshPath" value="package://${ThisPackage}/meshes/${Filename}" />
+<xacro:property name="mesh_extension" value="dae" />
+<xacro:macro name="get_hero" params="prefix">
 <!-- use this instead for moveit or other stuff -->
 <!-- <xacro:property name="MeshPath" value="package://new_hero/meshes" /> -->
@@ -32,6 +33,5 @@
 <xacro:property name="min_link6_link7" value="${-1 * off_link6_link7 - pi}" />
 <xacro:property name="min_link7_link8" value="${-1 * off_link7_link8 - pi}" />
-<xacro:property name="mesh_extension" value="dae" />
-  <link name="gripper1">
+<link name="${prefix}gripper1">
     <inertial>
       <origin
@@ -72,5 +72,5 @@
     </collision>
   </link>
-  <link name="link2">
+  <link name="${prefix}link2">
     <inertial>
       <origin
@@ -111,13 +111,13 @@
     </collision>
   </link>
-  <joint name="base_link-link2" type="continuous">
+  <joint name="${prefix}base_link-link2" type="continuous">
     <origin xyz="0 0 0.05" rpy="0 0 0" />
-    <parent link="gripper1" />
-    <child link="link2" />
+    <parent link="${prefix}gripper1" />
+    <child link="${prefix}link2" />
     <axis xyz="0 0 1" />
     <dynamics damping="0.7"/>
     <limit upper="${max_base_link_link2}" lower="${min_base_link_link2}" effort="100.0" velocity="1300"/>
   </joint>
-  <link name="link3">
+  <link name="${prefix}link3">
     <inertial>
       <origin
@@ -158,13 +158,13 @@
     </collision>
   </link>
-  <joint name="link2-link3" type="continuous">
+  <joint name="${prefix}link2-link3" type="continuous">
     <origin xyz="0.00016471 -0.090096 0.16854" rpy="0 1.57 0" />
-    <parent link="link2" />
-    <child link="link3" />
+    <parent link="${prefix}link2" />
+    <child link="${prefix}link3" />
     <axis xyz="0 -1 0" />
     <dynamics damping="0.7"/>
     <limit upper="${max_link2_link3}" lower="${min_link2_link3}" effort="100.0" velocity="1300"/>
   </joint>
-  <link name="link4">
+  <link name="${prefix}link4">
     <inertial>
       <origin
@@ -205,13 +205,13 @@
     </collision>
   </link>
-  <joint name="link3-link4" type="continuous">
+  <joint name="${prefix}link3-link4" type="continuous">
     <origin xyz="0 -0.058547 0.071444" rpy="0 0 1.57" />
-    <parent link="link3" />
-    <child  link="link4" />
+    <parent link="${prefix}link3" />
+    <child  link="${prefix}link4" />
     <axis xyz="0 0 1" />
     <dynamics damping="0.7"/>
     <limit upper="${max_link3_link4}" lower="${min_link3_link4}" effort="100.0" velocity="1300"/>
   </joint>
-  <link name="link5">
+  <link name="${prefix}link5">
     <inertial>
       <origin
@@ -252,13 +252,13 @@
     </collision>
   </link>
-  <joint name="link4-link5" type="continuous">
+  <joint name="${prefix}link4-link5" type="continuous">
     <origin xyz="0.023568 0 0.42835" rpy="-1.57 0 0" />
-    <parent link="link4" />
-    <child link="link5" />
+    <parent link="${prefix}link4" />
+    <child link="${prefix}link5" />
     <axis xyz="1 0 0" />
     <dynamics damping="0.7"/>
     <limit upper="${max_link4_link5}" lower="${min_link4_link5}" effort="100.0" velocity="1300"/>
   </joint>
-  <link  name="link6">
+  <link name="${prefix}link6">
     <inertial>
       <origin
@@ -299,12 +299,12 @@
     </collision>
   </link>
-  <joint name="link5-link6" type="continuous">
+  <joint name="${prefix}link5-link6" type="continuous">
     <origin xyz="0.12633 0 0.42742" rpy="0 0 1.57" />
-    <parent link="link5" />
-    <child link="link6" />
+    <parent link="${prefix}link5" />
+    <child link="${prefix}link6" />
     <axis xyz="0 0 1" />
     <limit upper="${max_link5_link6}" lower="${min_link5_link6}" effort="100.0" velocity="1300"/>
   </joint>
-  <link name="link7">
+  <link name="${prefix}link7">
     <inertial>
       <origin
@@ -345,13 +345,13 @@
     </collision>
   </link>
-  <joint name="link6-link7" type="continuous">
+  <joint name="${prefix}link6-link7" type="continuous">
     <origin xyz="0 0.12032 0.072384" rpy="0 -1.57 0" />
-    <parent link="link6" />
-    <child link="link7" />
+    <parent link="${prefix}link6" />
+    <child link="${prefix}link7" />
     <axis xyz="0 1 0" />
     <dynamics damping="0.7"/>
     <limit upper="${max_link6_link7}" lower="${min_link6_link7}" effort="100.0" velocity="1300"/>
   </joint>
-  <link  name="link8">
+  <link name="${prefix}link8">
     <inertial>
       <origin
@@ -392,8 +392,8 @@
     </collision>
   </link>
-  <joint name="link7-link8" type="continuous">
+  <joint name="${prefix}link7-link8" type="continuous">
     <origin xyz="0 0.029477 0.15419" rpy="0 0 0" />
-    <parent link="link7" />
-    <child link="link8" />
+    <parent link="${prefix}link7" />
+    <child link="${prefix}link8" />
     <axis xyz="0 0 1" />
     <dynamics damping="0.7"/>
@@ -410,11 +410,11 @@
     rpy="0 ${-pi} ${-pi}" />
     <parent
-      link="link8" />
+    link="${prefix}link8" />
     <child
-      link="gripper2" />
+    link="${prefix}gripper2" />
   </joint>
   <transmission name="link2_trans">
     <type>transmission_interface/SimpleTransmission</type>
-    <joint name="base_link-link2">
+    <joint name="${prefix}base_link-link2">
       <hardwareInterface>hardware_interface/PositionJointInterface</hardwareInterface>
     </joint>
@@ -426,5 +426,5 @@
   <transmission name="link3_trans">
     <type>transmission_interface/SimpleTransmission</type>
-    <joint name="link2-link3">
+    <joint name="${prefix}link2-link3">
       <hardwareInterface>hardware_interface/PositionJointInterface</hardwareInterface>
     </joint>
@@ -436,5 +436,5 @@
   <transmission name="link4_trans">
     <type>transmission_interface/SimpleTransmission</type>
-    <joint name="link3-link4">
+    <joint name="${prefix}link3-link4">
       <hardwareInterface>hardware_interface/PositionJointInterface</hardwareInterface>
     </joint>
@@ -446,5 +446,5 @@
   <transmission name="link5_trans">
     <type>transmission_interface/SimpleTransmission</type>
-    <joint name="link4-link5">
+    <joint name="${prefix}link4-link5">
       <hardwareInterface>hardware_interface/PositionJointInterface</hardwareInterface>
     </joint>
@@ -456,5 +456,5 @@
   <transmission name="link6_trans">
     <type>transmission_interface/SimpleTransmission</type>
-    <joint name="link5-link6">
+    <joint name="${prefix}link5-link6">
       <hardwareInterface>hardware_interface/PositionJointInterface</hardwareInterface>
     </joint>
@@ -466,5 +466,5 @@
   <transmission name="link7_trans">
     <type>transmission_interface/SimpleTransmission</type>
-    <joint name="link6-link7">
+    <joint name="${prefix}link6-link7">
       <hardwareInterface>hardware_interface/PositionJointInterface</hardwareInterface>
     </joint>
@@ -476,5 +476,5 @@
   <transmission name="link_7_trans">
     <type>transmission_interface/SimpleTransmission</type>
-    <joint name="link7-link8">
+    <joint name="${prefix}link7-link8">
       <hardwareInterface>hardware_interface/PositionJointInterface</hardwareInterface>
     </joint>
@@ -507,6 +507,7 @@
     <selfCollide>true</selfCollide>
   </gazebo>
-  <gazebo reference="link8">
-    <selfCollide>true</selfCollide>
-  </gazebo>
+  <gazebo reference="${prefix}link8">
+    <selfCollide>true</selfCollide>
+  </gazebo>
+</xacro:macro>
 </robot>

File: src/urdf_packer/urdf/hero_7dof/hero_dragon.xacro (robot description, xacro)
@@ -1,4 +1,4 @@
 <?xml version="1.0"?>
-<robot xmlns:xacro="http://www.ros.org/wiki/xacro" name="hero_7dofm3">
+<robot xmlns:xacro="http://www.ros.org/wiki/xacro" name="hero_dragon">
 <xacro:property name="ThisPackage" value="urdf_packer" />
 <xacro:property name="Filename" value="hero_7dof" />
@@ -6,8 +6,5 @@
 <xacro:property name="MeshPath" value="package://${ThisPackage}/meshes/${Filename}" />
   <!-- Include the original xacro file -->
-  <link
-  name="base_link">
-  </link>
-<xacro:include filename="hero_7dofm4.xacro"/>
+<link name="base_link" />
 <xacro:include filename="wheel_macro.xacro"/>
 <joint name="bfix" type="fixed">
@@ -16,7 +13,5 @@
 <child link="base_link45"/>
 </joint>
-  <link
-  name="base_link45">
-  </link>
+<link name="base_link45" />
 <joint name="bfixstraight" type="fixed">
 <origin xyz="0 0 0" rpy="-${pi/4} 0 0"/>
@@ -24,4 +19,13 @@
 <child link="wheel1"/>
 </joint>
+<xacro:add_wheel  wheel_number="1" />
+<link name="wheel1c45" />
+<joint name="fix451" type="fixed">
+<origin xyz="0 0 0" rpy="${-pi/4} 0 0"/>
+<parent link="wheel_center_1"/>
+<child link="wheel1c45"/>
+</joint>
+<xacro:include filename="hero_7dofm4.xacro" ns="leg1"/>
+<xacro:leg1.get_hero prefix="" />
 <joint name="fixwheel1" type="fixed">
 <origin xyz="0 0 0" rpy="0 0 0"/>
@@ -41,11 +45,11 @@
 <child link="wheel2c45"/>
 </joint>
-<xacro:add_wheel  wheel_number="1" />
-<link name="wheel1c45" />
-<joint name="fix451" type="fixed">
-<origin xyz="0 0 0" rpy="${-pi/4} 0 0"/>
-<parent link="wheel_center_1"/>
-<child link="wheel1c45"/>
-</joint>
-  <!-- Rest of your new robot description -->
+<!-- <group ns="leg2"> -->
+<!-- <xacro:get_hero prefix="leg2" /> -->
+<!-- <joint name="fixwheel1-2" type="fixed"> -->
+<!-- <origin xyz="0 0 0" rpy="0 0 0"/> -->
+<!-- <parent link="wheel1"/> -->
+<!-- <child link="leg2/gripper1"/> -->
+<!-- </joint> -->
+<!-- </group> -->
 </robot>
