Commit message: dragon test irl

File: src/urdf_packer/urdf/hero_7dof/hero_7dof.xacro (robot description, xacro)
@@ -1,6 +1,3 @@
 <?xml version="1.0" encoding="utf-8"?>
-<!-- This URDF was automatically created by SolidWorks to URDF Exporter! Originally created by Stephen Brawner (brawner@gmail.com)
-     Commit Version: 1.6.0-4-g7f85cfe  Build Version: 1.6.7995.38578
-     For more information, please see http://wiki.ros.org/sw_urdf_exporter -->
 <robot name="hero_7dof" xmlns:xacro="http://www.ros.org/wiki/xacro">
 <xacro:property name="ThisPackage" value="urdf_packer" />
@@ -9,14 +6,14 @@
 <xacro:property name="MeshPath" value="package://${ThisPackage}/meshes/${Filename}" />
 <xacro:property name="mesh_extension" value="dae" />
-<xacro:macro name="get_hero" params="prefix">
+<xacro:macro name="get_hero" params="prefix off_base_link_link2 off_link2_link3 off_link3_link4 off_link4_link5 off_link5_link6 off_link6_link7 off_link7_link8">
 <!-- use this instead for moveit or other stuff -->
 <!-- <xacro:property name="MeshPath" value="package://new_hero/meshes" /> -->
-<xacro:property name="off_base_link_link2" value="-1.5968164926267214" />
-<xacro:property name="off_link2_link3" value="-1.5249186659861529" />
-<xacro:property name="off_link3_link4" value="-1.1246189568997114" />
-<xacro:property name="off_link4_link5" value="-1.2173329162057398" />
-<xacro:property name="off_link5_link6" value="-0.4995871839710359" />
-<xacro:property name="off_link6_link7" value="-1.6035269564465078" />
-<xacro:property name="off_link7_link8" value="-0.8002183286638307" />
+<!-- <xacro:property name="off_base_link_link2" value="-1.5968164926267214" /> -->
+<!-- <xacro:property name="off_link2_link3" value="-1.5249186659861529" /> -->
+<!-- <xacro:property name="off_link3_link4" value="-1.1246189568997114" /> -->
+<!-- <xacro:property name="off_link4_link5" value="-1.2173329162057398" /> -->
+<!-- <xacro:property name="off_link5_link6" value="-0.4995871839710359" /> -->
+<!-- <xacro:property name="off_link6_link7" value="-1.6035269564465078" /> -->
+<!-- <xacro:property name="off_link7_link8" value="-0.8002183286638307" /> -->
 <xacro:property name="max_base_link_link2" value="${-1 * off_base_link_link2}" />
 <xacro:property name="max_link2_link3" value="${-1 * off_link2_link3}" />
@@ -401,8 +398,8 @@
   </joint>
   <link
-  name="gripper2">
+  name="${prefix}gripper2">
   </link>
   <joint
-    name="eefix"
+  name="${prefix}eefix"
     type="fixed">
     <origin
@@ -414,70 +411,70 @@
     link="${prefix}gripper2" />
   </joint>
-  <transmission name="link2_trans">
+  <transmission name="${prefix}link2_trans">
     <type>transmission_interface/SimpleTransmission</type>
     <joint name="${prefix}base_link-link2">
       <hardwareInterface>hardware_interface/PositionJointInterface</hardwareInterface>
     </joint>
-    <actuator name="link2_motor">
-      <hardwareInterface>hardware_interface/PositionJointInterface</hardwareInterface>
-      <mechanicalReduction>1</mechanicalReduction>
-    </actuator>
-  </transmission>
-  <transmission name="link3_trans">
+    <actuator name="${prefix}link2_motor">
+      <hardwareInterface>hardware_interface/PositionJointInterface</hardwareInterface>
+      <mechanicalReduction>1</mechanicalReduction>
+    </actuator>
+  </transmission>
+  <transmission name="${prefix}link3_trans">
     <type>transmission_interface/SimpleTransmission</type>
     <joint name="${prefix}link2-link3">
       <hardwareInterface>hardware_interface/PositionJointInterface</hardwareInterface>
     </joint>
-    <actuator name="link3_motor">
-      <hardwareInterface>hardware_interface/PositionJointInterface</hardwareInterface>
-      <mechanicalReduction>1</mechanicalReduction>
-    </actuator>
-  </transmission>
-  <transmission name="link4_trans">
+    <actuator name="${prefix}link3_motor">
+      <hardwareInterface>hardware_interface/PositionJointInterface</hardwareInterface>
+      <mechanicalReduction>1</mechanicalReduction>
+    </actuator>
+  </transmission>
+  <transmission name="${prefix}link4_trans">
     <type>transmission_interface/SimpleTransmission</type>
     <joint name="${prefix}link3-link4">
       <hardwareInterface>hardware_interface/PositionJointInterface</hardwareInterface>
     </joint>
-    <actuator name="link4_motor">
-      <hardwareInterface>hardware_interface/PositionJointInterface</hardwareInterface>
-      <mechanicalReduction>1</mechanicalReduction>
-    </actuator>
-  </transmission>
-  <transmission name="link5_trans">
+    <actuator name="${prefix}link4_motor">
+      <hardwareInterface>hardware_interface/PositionJointInterface</hardwareInterface>
+      <mechanicalReduction>1</mechanicalReduction>
+    </actuator>
+  </transmission>
+  <transmission name="${prefix}link5_trans">
     <type>transmission_interface/SimpleTransmission</type>
     <joint name="${prefix}link4-link5">
       <hardwareInterface>hardware_interface/PositionJointInterface</hardwareInterface>
     </joint>
-    <actuator name="link5_motor">
-      <hardwareInterface>hardware_interface/PositionJointInterface</hardwareInterface>
-      <mechanicalReduction>1</mechanicalReduction>
-    </actuator>
-  </transmission>
-  <transmission name="link6_trans">
+    <actuator name="${prefix}link5_motor">
+      <hardwareInterface>hardware_interface/PositionJointInterface</hardwareInterface>
+      <mechanicalReduction>1</mechanicalReduction>
+    </actuator>
+  </transmission>
+  <transmission name="${prefix}link6_trans">
     <type>transmission_interface/SimpleTransmission</type>
     <joint name="${prefix}link5-link6">
       <hardwareInterface>hardware_interface/PositionJointInterface</hardwareInterface>
     </joint>
-    <actuator name="link6_motor">
-      <hardwareInterface>hardware_interface/PositionJointInterface</hardwareInterface>
-      <mechanicalReduction>1</mechanicalReduction>
-    </actuator>
-  </transmission>
-  <transmission name="link7_trans">
+    <actuator name="${prefix}link6_motor">
+      <hardwareInterface>hardware_interface/PositionJointInterface</hardwareInterface>
+      <mechanicalReduction>1</mechanicalReduction>
+    </actuator>
+  </transmission>
+  <transmission name="${prefix}link7_trans">
     <type>transmission_interface/SimpleTransmission</type>
     <joint name="${prefix}link6-link7">
       <hardwareInterface>hardware_interface/PositionJointInterface</hardwareInterface>
     </joint>
-    <actuator name="link7_motor">
-      <hardwareInterface>hardware_interface/PositionJointInterface</hardwareInterface>
-      <mechanicalReduction>1</mechanicalReduction>
-    </actuator>
-  </transmission>
-  <transmission name="link_7_trans">
+    <actuator name="${prefix}link7_motor">
+      <hardwareInterface>hardware_interface/PositionJointInterface</hardwareInterface>
+      <mechanicalReduction>1</mechanicalReduction>
+    </actuator>
+  </transmission>
+  <transmission name="${prefix}link_7_trans">
     <type>transmission_interface/SimpleTransmission</type>
     <joint name="${prefix}link7-link8">
       <hardwareInterface>hardware_interface/PositionJointInterface</hardwareInterface>
     </joint>
-    <actuator name="link8_motor">
+    <actuator name="${prefix}link8_motor">
       <hardwareInterface>hardware_interface/PositionJointInterface</hardwareInterface>
       <mechanicalReduction>1</mechanicalReduction>

File: src/urdf_packer/urdf/hero_7dof/hero_7dofm3.xacro (robot description, xacro)
@@ -7,12 +7,19 @@
   <!-- Include the original xacro file -->
 <xacro:include filename="${Filename}.xacro"/>
-  <!-- Override specific properties -->
-<xacro:property name="off_base_link_link2" value="-1.5968164926267214" />
-<xacro:property name="off_link2_link3" value="-1.5249186659861529" />
-<xacro:property name="off_link3_link4" value="-1.1246189568997114" />
-<xacro:property name="off_link4_link5" value="-1.2173329162057398" />
-<xacro:property name="off_link5_link6" value="-0.4995871839710359" />
-<xacro:property name="off_link6_link7" value="-1.6035269564465078" />
-<xacro:property name="off_link7_link8" value="-0.8002183286638307" />
-  <!-- Rest of your new robot description -->
+<xacro:get_hero prefix = "leg3"
+off_base_link_link2 = "-1.5968164926267214"
+off_link2_link3 = "-1.5249186659861529"
+off_link3_link4 = "-1.1246189568997114"
+off_link4_link5 = "-1.2173329162057398"
+off_link5_link6 = "-0.4995871839710359"
+off_link6_link7 = "-1.6035269564465078"
+off_link7_link8 = "-0.8002183286638307"
+/>
+<!-- <xacro:property name="off_base_link_link2" value="-1.5968164926267214" /> -->
+<!-- <xacro:property name="off_link2_link3" value="-1.5249186659861529" /> -->
+<!-- <xacro:property name="off_link3_link4" value="-1.1246189568997114" /> -->
+<!-- <xacro:property name="off_link4_link5" value="-1.2173329162057398" /> -->
+<!-- <xacro:property name="off_link5_link6" value="-0.4995871839710359" /> -->
+<!-- <xacro:property name="off_link6_link7" value="-1.6035269564465078" /> -->
+<!-- <xacro:property name="off_link7_link8" value="-0.8002183286638307" /> -->
 </robot>

File: src/urdf_packer/urdf/hero_7dof/hero_7dofm4.xacro (robot description, xacro)
@@ -1,4 +1,4 @@
 <?xml version="1.0"?>
-<robot xmlns:xacro="http://www.ros.org/wiki/xacro" name="hero_7dofm3">
+<robot xmlns:xacro="http://www.ros.org/wiki/xacro" name="hero_7dofm4">
 <xacro:property name="ThisPackage" value="urdf_packer" />
 <xacro:property name="Filename" value="hero_7dof" />
@@ -7,12 +7,13 @@
   <!-- Include the original xacro file -->
 <xacro:include filename="${Filename}.xacro"/>
-  <!-- Override specific properties -->
-<xacro:property name="off_base_link_link2" value="-1.5968164926267214" />
-<xacro:property name="off_link2_link3" value="-1.5249186659861529" />
-<xacro:property name="off_link3_link4" value="-1.1246189568997114" />
-<xacro:property name="off_link4_link5" value="-1.2173329162057398" />
-<xacro:property name="off_link5_link6" value="-0.4995871839710359" />
-<xacro:property name="off_link6_link7" value="-1.6035269564465078" />
-<xacro:property name="off_link7_link8" value="-0.8002183286638307" />
+<xacro:get_hero prefix = "leg4"
+off_base_link_link2 = "-1.5968164926267214"
+off_link2_link3 = "-1.5249186659861529"
+off_link3_link4 = "-1.1246189568997114"
+off_link4_link5 = "-1.2173329162057398"
+off_link5_link6 = "-0.4995871839710359"
+off_link6_link7 = "-1.6035269564465078"
+off_link7_link8 = "-0.8002183286638307"
+/>
   <!-- Rest of your new robot description -->
 </robot>

File: src/urdf_packer/urdf/hero_7dof/hero_dragon.xacro (robot description, xacro)
@@ -8,4 +8,6 @@
 <link name="base_link" />
 <xacro:include filename="wheel_macro.xacro"/>
+<xacro:include filename="hero_7dofm4.xacro" ns="leg4"/>
+<xacro:include filename="hero_7dofm3.xacro" ns="leg3"/>
 <joint name="bfix" type="fixed">
 <origin xyz="0 0 0.165" rpy="${pi/4} 0 0"/>
@@ -17,39 +19,41 @@
 <origin xyz="0 0 0" rpy="-${pi/4} 0 0"/>
 <parent link="base_link45"/>
-<child link="wheel1"/>
+<child link="1wheel_in"/>
 </joint>
-<xacro:add_wheel  wheel_number="1" />
+<xacro:add_wheel prefix="1" />
 <link name="wheel1c45" />
 <joint name="fix451" type="fixed">
 <origin xyz="0 0 0" rpy="${-pi/4} 0 0"/>
-<parent link="wheel_center_1"/>
+<parent link="1wheel_center"/>
 <child link="wheel1c45"/>
 </joint>
-<xacro:include filename="hero_7dofm4.xacro" ns="leg1"/>
-<xacro:leg1.get_hero prefix="" />
 <joint name="fixwheel1" type="fixed">
 <origin xyz="0 0 0" rpy="0 0 0"/>
-<parent link="wheel1"/>
-<child link="gripper1"/>
+<parent link="1wheel_in"/>
+<child link="leg4gripper1"/>
 </joint>
 <joint name="fixwheel2" type="fixed">
 <origin xyz="0 0 0" rpy="0 0 0"/>
-<parent link="gripper2"/>
-<child link="wheel2"/>
+<parent link="leg4gripper2"/>
+<child link="2wheel_in"/>
 </joint>
-<xacro:add_wheel  wheel_number="2" />
+<xacro:add_wheel  prefix="2" />
 <link name="wheel2c45" />
 <joint name="fix452" type="fixed">
 <origin xyz="0 0 0" rpy="${pi/4} 0 0"/>
-<parent link="wheel_center_2"/>
+<parent link="2wheel_center"/>
 <child link="wheel2c45"/>
 </joint>
-<!-- <group ns="leg2"> -->
-<!-- <xacro:get_hero prefix="leg2" /> -->
-<!-- <joint name="fixwheel1-2" type="fixed"> -->
+<joint name="fixwheel1-2" type="fixed">
+<origin xyz="0 0 0" rpy="0 0 0"/>
+<parent link="1wheel_out"/>
+<child link="leg3gripper1"/>
+</joint>
+<!-- <xacro:add_wheel  prefix="3" /> -->
+<!---->
+<!-- <joint name="fixwheel1-3" type="fixed"> -->
 <!-- <origin xyz="0 0 0" rpy="0 0 0"/> -->
-<!-- <parent link="wheel1"/> -->
-<!-- <child link="leg2/gripper1"/> -->
+<!-- <parent link="leg4gripper2"/> -->
+<!-- <child link="3wheel_in"/> -->
 <!-- </joint> -->
-<!-- </group> -->
 </robot>

File: src/urdf_packer/urdf/hero_7dof/wheel_macro.xacro (robot description, xacro)
@@ -9,6 +9,6 @@
 <color rgba="0 0 0 1.000"/>
 </material>
-<xacro:macro name="add_wheel" params="wheel_number">
-  <link name="wheel_body_${wheel_number}">
+<xacro:macro name="add_wheel" params="prefix">
+  <link name="${prefix}wheel_body">
     <inertial>
       <origin xyz="0.012120027900982211 1.7479052741023483e-05 -0.1932995813581685" rpy="0 0 0"/>
@@ -30,5 +30,5 @@
     </collision>
   </link>
-  <link name="wheel_left_${wheel_number}">
+  <link name="${prefix}wheel_left">
     <inertial>
       <origin xyz="6.05831716671279e-06 -0.079400296699694 3.750658923479255e-05" rpy="0 0 0"/>
@@ -50,5 +50,5 @@
     </collision>
   </link>
-  <link name="wheel_right_${wheel_number}">
+  <link name="${prefix}wheel_right">
     <inertial>
       <origin xyz="-6.058317166268701e-06 0.07940029669969387 3.7506589234403975e-05" rpy="0 0 0"/>
@@ -70,31 +70,34 @@
     </collision>
   </link>
-  <link
-  name="wheel_center_${wheel_number}">
-  </link>
-  <link
-  name="wheel${wheel_number}">
-  </link>
-  <joint name="wheel_fix_${wheel_number}" type="fixed">
+  <link name="${prefix}wheel_in"/>
+  <link name="${prefix}wheel_center"/>
+  <link name="${prefix}wheel_out"/>
+  <joint name="${prefix}wheel_fix" type="fixed">
   <origin xyz="0 0 0.05" rpy="0 0 ${pi/2}"/>
-    <parent link="wheel${wheel_number}"/>
-    <child link="wheel_body_${wheel_number}"/>
+    <parent link="${prefix}wheel_in"/>
+    <child link="${prefix}wheel_body"/>
   </joint>
-  <joint name="wheel_cent_fix${wheel_number}" type="fixed">
+  <joint name="${prefix}wheel_cent_fix" type="fixed">
   <origin xyz="0 0 -0.213" rpy="0 0 -${pi/2}"/>
-    <parent link="wheel_body_${wheel_number}"/>
-    <child link="wheel_center_${wheel_number}"/>
+    <parent link="${prefix}wheel_body"/>
+    <child link="${prefix}wheel_center"/>
   </joint>
-  <joint name="wheel_left_joint_${wheel_number}" type="continuous">
+  <joint name="${prefix}wheel_left_joint" type="continuous">
     <origin xyz="0.004 0.277 -0.213" rpy="0 0 0"/>
-    <parent link="wheel_body_${wheel_number}"/>
-    <child link="wheel_left_${wheel_number}"/>
+    <parent link="${prefix}wheel_body"/>
+    <child link="${prefix}wheel_left"/>
     <axis xyz="0.0 1.0 0.0"/>
   </joint>
-  <joint name="wheel_right_joint_${wheel_number}" type="continuous">
-    <origin xyz="0.004 -0.277 -0.213" rpy="0 0 0"/>
-    <parent link="wheel_body_${wheel_number}"/>
-    <child link="wheel_right_${wheel_number}"/>
+  <joint name="${prefix}wheel_right_joint" type="continuous">
+  <origin xyz="0.004 -0.277 -0.213" rpy="0 0 0"/>
+    <parent link="${prefix}wheel_body"/>
+    <child link="${prefix}wheel_right"/>
     <axis xyz="-0.0 -1.0 -0.0"/>
+  </joint>
+  <joint name="${prefix}wheel_cen2out" type="fixed">
+    <origin xyz="0 0.100 0" rpy="${-pi/2} 0 0"/>
+    <parent link="${prefix}wheel_center"/>
+    <child link="${prefix}wheel_out"/>
+    <axis xyz="0 0 0"/>
   </joint>
 </xacro:macro>

Commit message: relative to ee ik2 option

File: src/urdf_packer/urdf/hero_7dof/hero_7dof.xacro (robot description, xacro)
@@ -411,4 +411,18 @@
     link="${prefix}gripper2" />
   </joint>
+  <link
+  name="${prefix}gripper2_straight">
+  </link>
+  <joint
+  name="${prefix}eestraight"
+    type="fixed">
+    <origin
+      xyz="0 0 0"
+    rpy="0 ${pi/2} 0" />
+    <parent
+    link="${prefix}gripper2" />
+    <child
+    link="${prefix}gripper2_straight" />
+  </joint>
   <transmission name="${prefix}link2_trans">
     <type>transmission_interface/SimpleTransmission</type>
