Commit message: much better launch for MH

File: src/urdf_packer/urdf/hero_7dof/hero_3legwheel.xacro (robot description, xacro)
@@ -4,18 +4,24 @@
 <xacro:include filename="wheel_macro.xacro"/>
 <xacro:add_wheel prefix="11" />
-<joint name="fix11" type="fixed">
-<origin xyz="0 0 0" rpy="0 0 0"/>
+<joint name="fix11"
+type="fixed">
+<origin xyz="0 0 0"
+rpy="0 0 0"/>
 <parent link="leg1gripper2"/>
 <child link="11wheel_in"/>
 </joint>
 <xacro:add_wheel prefix="12" />
-<joint name="fix12" type="fixed">
-<origin xyz="0 0 0" rpy="0 0 0"/>
+<joint name="fix12"
+type="fixed">
+<origin xyz="0 0 0"
+rpy="0 0 0"/>
 <parent link="leg2gripper2"/>
 <child link="12wheel_in"/>
 </joint>
 <xacro:add_wheel prefix="13" />
-<joint name="fix13" type="fixed">
-<origin xyz="0 0 0" rpy="0 0 0"/>
+<joint name="fix13"
+type="fixed">
+<origin xyz="0 0 0"
+rpy="0 0 0"/>
 <parent link="leg3gripper2"/>
 <child link="13wheel_in"/>

File: src/urdf_packer/urdf/hero_7dof/hero_dragon.xacro (robot description, xacro)
@@ -5,4 +5,9 @@
   <xacro:property name="UrdfDataPath" value="package://${ThisPackage}/urdf/${Filename}"></xacro:property>
   <xacro:property name="MeshPath" value="package://${ThisPackage}/meshes/${Filename}"></xacro:property>
+  <!-- change what leg is where -->
+  <!--  -->
+  <!--  -->
+  <xacro:property name="wheelfront" value="11"></xacro:property>
+  <xacro:property name="wheelback" value="12"></xacro:property>
   <xacro:property name="main_leg" value="2"></xacro:property>
   <!-- also change that here !!!!    V   -->
@@ -11,5 +16,7 @@
   <!-- also change that here !!!!    V   -->
   <xacro:include filename="hero_7dofm4.xacro" ns="leg${manip_leg}"></xacro:include>
-  <!-- Include the original xacro file -->
+  <!--  -->
+  <!--  -->
+  <!--  -->
   <link name="base_link"></link>
   <xacro:include filename="wheel_macro.xacro"></xacro:include>
@@ -23,33 +30,37 @@
     <origin rpy="0 0 0" xyz="0 0 0.165"></origin>
     <parent link="base_link45"></parent>
-    <child link="1wheel_in"></child>
+    <child link="${wheelfront}wheel_in"></child>
   </joint>
-  <xacro:add_wheel prefix="1"></xacro:add_wheel>
-  <link name="wheel1c45"></link>
-  <joint name="fix451" type="fixed">
+  <!---->
+  <!---->
+  <xacro:add_wheel prefix="${wheelfront}"></xacro:add_wheel>
+  <link name="wheel${wheelfront}c45"></link>
+  <joint name="fix45${wheelfront}" type="fixed">
     <origin rpy="${-pi/4} 0 0" xyz="0 0 0"></origin>
-    <parent link="1wheel_center"></parent>
-    <child link="wheel1c45"></child>
+    <parent link="${wheelfront}wheel_center"></parent>
+    <child link="wheel${wheelfront}c45"></child>
   </joint>
-  <joint name="fixwheel1" type="fixed">
+  <joint name="fixwheel${wheelfront}" type="fixed">
     <origin rpy="0 0 0" xyz="0 0 0"></origin>
-    <parent link="1wheel_in"></parent>
+    <parent link="${wheelfront}wheel_in"></parent>
     <child link="leg${main_leg}gripper1"></child>
   </joint>
-  <joint name="fixwheel2" type="fixed">
+  <!---->
+  <!---->
+  <joint name="fixwheel${wheelback}" type="fixed">
     <origin rpy="0 0 ${0*pi}" xyz="0 0 0"></origin>
     <parent link="leg${main_leg}gripper2"></parent>
-    <child link="2wheel_in"></child>
+    <child link="${wheelback}wheel_in"></child>
   </joint>
-  <xacro:add_wheel prefix="2"></xacro:add_wheel>
-  <link name="wheel2c45"></link>
-  <joint name="fix452" type="fixed">
+  <xacro:add_wheel prefix="${wheelback}"></xacro:add_wheel>
+  <link name="wheel${wheelback}c45"></link>
+  <joint name="fix45${wheelback}" type="fixed">
     <origin rpy="${pi/4} 0 0" xyz="0 0 0"></origin>
-    <parent link="2wheel_center"></parent>
-    <child link="wheel2c45"></child>
+    <parent link="${wheelback}wheel_center"></parent>
+    <child link="wheel${wheelback}c45"></child>
   </joint>
-  <joint name="fixwheel1-2" type="fixed">
+  <joint name="fixwheel1-${wheelback}" type="fixed">
     <origin rpy="0 0 0" xyz="0 0 0"></origin>
-    <parent link="1wheel_out"></parent>
+    <parent link="${wheelfront}wheel_out"></parent>
     <child link="leg${manip_leg}gripper1"></child>
   </joint>

File: src/urdf_packer/urdf/hero_7dof/hero_vehicle.xacro (robot description, xacro)
@@ -1,8 +1,10 @@
 <?xml version="1.0" encoding="UTF-8"?>
-<robot name="hero_dragon" xmlns:xacro="http://www.ros.org/wiki/xacro">
+<robot name="hero_vehicle" xmlns:xacro="http://www.ros.org/wiki/xacro">
   <xacro:property name="ThisPackage" value="urdf_packer"></xacro:property>
   <xacro:property name="Filename" value="hero_7dof"></xacro:property>
   <xacro:property name="UrdfDataPath" value="package://${ThisPackage}/urdf/${Filename}"></xacro:property>
   <xacro:property name="MeshPath" value="package://${ThisPackage}/meshes/${Filename}"></xacro:property>
+  <xacro:property name="wheelfront" value="11"></xacro:property>
+  <xacro:property name="wheelback" value="12"></xacro:property>
   <xacro:property name="main_leg" value="4"></xacro:property>
   <!-- also change that here !!!!    V   -->
@@ -19,29 +21,29 @@
     <origin rpy="0 0 ${-pi/2}" xyz="0 0 0.165"></origin>
     <parent link="base_link"></parent>
-    <child link="1wheel_in"></child>
+    <child link="${wheelfront}wheel_in"></child>
   </joint>
-  <xacro:add_wheel prefix="1"></xacro:add_wheel>
-  <link name="wheel1c45"></link>
-  <joint name="fix451" type="fixed">
+  <xacro:add_wheel prefix="${wheelfront}"></xacro:add_wheel>
+  <link name="wheel${wheelfront}c45"></link>
+  <joint name="fix45${wheelfront}" type="fixed">
     <origin rpy="${-pi/4} 0 0" xyz="0 0 0"></origin>
-    <parent link="1wheel_center"></parent>
-    <child link="wheel1c45"></child>
+    <parent link="${wheelfront}wheel_center"></parent>
+    <child link="wheel${wheelfront}c45"></child>
   </joint>
-  <joint name="fixwheel1" type="fixed">
+  <joint name="fixwheel${wheelfront}" type="fixed">
     <origin rpy="0 0 0" xyz="0 0 0"></origin>
-    <parent link="1wheel_in"></parent>
+    <parent link="${wheelfront}wheel_in"></parent>
     <child link="leg${main_leg}gripper1"></child>
   </joint>
-  <joint name="fixwheel2" type="fixed">
+  <joint name="fixwheel${wheelback}" type="fixed">
     <origin rpy="0 0 ${0*pi}" xyz="0 0 0"></origin>
     <parent link="leg${main_leg}gripper2"></parent>
-    <child link="2wheel_in"></child>
+    <child link="${wheelback}wheel_in"></child>
   </joint>
-  <xacro:add_wheel prefix="2"></xacro:add_wheel>
-  <link name="wheel2c45"></link>
+  <xacro:add_wheel prefix="${wheelback}"></xacro:add_wheel>
+  <link name="wheel${wheelback}c45"></link>
   <joint name="fix452" type="fixed">
     <origin rpy="${pi/4} 0 0" xyz="0 0 0"></origin>
-    <parent link="2wheel_center"></parent>
-    <child link="wheel2c45"></child>
+    <parent link="${wheelback}wheel_center"></parent>
+    <child link="wheel${wheelback}c45"></child>
   </joint>
 </robot>

Commit message: Fix link name in hero_3legwheel.xacro

File: src/urdf_packer/urdf/hero_7dof/hero_3legwheel.xacro (robot description, xacro)
@@ -24,5 +24,5 @@
 <origin xyz="0 0 0"
 rpy="0 0 0"/>
-<parent link="leg3gripper2"/>
+<parent link="leg4gripper2"/>
 <child link="13wheel_in"/>
 </joint>

Commit message: wheel name fix (oof)

File: src/urdf_packer/urdf/hero_7dof/hero_3legwheel.xacro (robot description, xacro)
@@ -3,5 +3,9 @@
 <xacro:include filename="hero_3leg.xacro"/>
 <xacro:include filename="wheel_macro.xacro"/>
-<xacro:add_wheel prefix="11" />
+<!-- change wheel number here                 VV       -->
+<xacro:property name="wheelfront" value="wheel11_"></xacro:property>
+<xacro:property name="wheelleft" value="wheel12_"></xacro:property>
+<xacro:property name="wheelright" value="wheel13_"></xacro:property>
+<xacro:add_wheel prefix="${wheelfront}" />
 <joint name="fix11"
 type="fixed">
@@ -9,7 +13,7 @@
 rpy="0 0 0"/>
 <parent link="leg1gripper2"/>
-<child link="11wheel_in"/>
+<child link="${wheelfront}in"/>
 </joint>
-<xacro:add_wheel prefix="12" />
+<xacro:add_wheel prefix="${wheelleft}" />
 <joint name="fix12"
 type="fixed">
@@ -17,7 +21,7 @@
 rpy="0 0 0"/>
 <parent link="leg2gripper2"/>
-<child link="12wheel_in"/>
+<child link="${wheelleft}in"/>
 </joint>
-<xacro:add_wheel prefix="13" />
+<xacro:add_wheel prefix="${wheelright}" />
 <joint name="fix13"
 type="fixed">
@@ -25,5 +29,5 @@
 rpy="0 0 0"/>
 <parent link="leg4gripper2"/>
-<child link="13wheel_in"/>
+<child link="${wheelright}in"/>
 </joint>
 </robot>

File: src/urdf_packer/urdf/hero_7dof/hero_7dof_all.xacro (robot description, xacro)
@@ -31,27 +31,27 @@
 <xacro:include filename="hero_7dofm4.xacro"/>
 <xacro:include filename="wheel_macro.xacro"/>
-<xacro:add_wheel prefix="11" />
+<xacro:add_wheel prefix="wheel11_" />
 <joint name="fix11" type="fixed">
 <origin xyz="0.2 2 0" rpy="0 0 ${pi/2}"/>
 <parent link="base_link"/>
-<child link="11wheel_in"/>
+<child link="wheel11_in"/>
 </joint>
-<xacro:add_wheel prefix="12" />
+<xacro:add_wheel prefix="wheel12_" />
 <joint name="fix12" type="fixed">
 <origin xyz="0.6 2 0" rpy="0 0 ${pi/2}"/>
 <parent link="base_link"/>
-<child link="12wheel_in"/>
+<child link="wheel12_in"/>
 </joint>
-<xacro:add_wheel prefix="13" />
+<xacro:add_wheel prefix="wheel13_" />
 <joint name="fix13" type="fixed">
 <origin xyz="1 2 0" rpy="0 0 ${pi/2}"/>
 <parent link="base_link"/>
-<child link="13wheel_in"/>
+<child link="wheel13_in"/>
 </joint>
-<xacro:add_wheel prefix="14" />
+<xacro:add_wheel prefix="wheel14_" />
 <joint name="fix14" type="fixed">
 <origin xyz="1.4 2 0" rpy="0 0 ${pi/2}"/>
 <parent link="base_link"/>
-<child link="14wheel_in"/>
+<child link="wheel14_in"/>
 </joint>
 </robot>

File: src/urdf_packer/urdf/hero_7dof/hero_dragon.xacro (robot description, xacro)
@@ -8,7 +8,7 @@
   <!--  -->
   <!--  -->
-  <xacro:property name="wheelfront" value="14"></xacro:property>
-  <xacro:property name="wheelback" value="12"></xacro:property>
-  <xacro:property name="main_leg" value="2"></xacro:property>
+  <xacro:property name="wheelfront" value="wheel12_"></xacro:property>
+  <xacro:property name="wheelback" value="wheel14_"></xacro:property>
+  <xacro:property name="bridge_leg" value="2"></xacro:property>
   <!-- also change that here !!!!    V   -->
   <xacro:include filename="hero_7dofm2.xacro"></xacro:include>
@@ -30,37 +30,37 @@
     <origin rpy="0 0 0" xyz="0 0 0.165"></origin>
     <parent link="base_link45"></parent>
-    <child link="${wheelfront}wheel_in"></child>
+    <child link="${wheelfront}in"></child>
   </joint>
   <!---->
   <!---->
   <xacro:add_wheel prefix="${wheelfront}"></xacro:add_wheel>
-  <link name="wheel${wheelfront}c45"></link>
-  <joint name="fix45${wheelfront}" type="fixed">
-    <origin rpy="${-pi/4} 0 0" xyz="0 0 0"></origin>
-    <parent link="${wheelfront}wheel_center"></parent>
-    <child link="wheel${wheelfront}c45"></child>
-  </joint>
-  <joint name="fixwheel${wheelfront}" type="fixed">
+  <!-- <link name="${wheelfront}c45"></link> -->
+  <!-- <joint name="${wheelfront}fix45" type="fixed"> -->
+  <!--   <origin rpy="${-pi/4} 0 0" xyz="0 0 0"></origin> -->
+  <!--   <parent link="${wheelfront}center"></parent> -->
+  <!--   <child link="${wheelfront}c45"></child> -->
+  <!-- </joint> -->
+  <joint name="${wheelfront}fixin" type="fixed">
     <origin rpy="0 0 0" xyz="0 0 0"></origin>
-    <parent link="${wheelfront}wheel_in"></parent>
-    <child link="leg${main_leg}gripper1"></child>
+    <parent link="${wheelfront}in"></parent>
+    <child link="leg${bridge_leg}gripper1"></child>
   </joint>
   <!---->
   <!---->
-  <joint name="fixwheel${wheelback}" type="fixed">
+  <joint name="${wheelback}fix1" type="fixed">
     <origin rpy="0 0 ${0*pi}" xyz="0 0 0"></origin>
-    <parent link="leg${main_leg}gripper2"></parent>
-    <child link="${wheelback}wheel_in"></child>
+    <parent link="leg${bridge_leg}gripper2"></parent>
+    <child link="${wheelback}in"></child>
   </joint>
   <xacro:add_wheel prefix="${wheelback}"></xacro:add_wheel>
-  <link name="wheel${wheelback}c45"></link>
+  <link name="${wheelback}c45"></link>
   <joint name="fix45${wheelback}" type="fixed">
     <origin rpy="${pi/4} 0 0" xyz="0 0 0"></origin>
-    <parent link="${wheelback}wheel_center"></parent>
-    <child link="wheel${wheelback}c45"></child>
+    <parent link="${wheelback}center"></parent>
+    <child link="${wheelback}c45"></child>
   </joint>
-  <joint name="fixwheel1-${wheelback}" type="fixed">
+  <joint name="${wheelfront}fix_out" type="fixed">
     <origin rpy="0 0 0" xyz="0 0 0"></origin>
-    <parent link="${wheelfront}wheel_out"></parent>
+    <parent link="${wheelfront}out"></parent>
     <child link="leg${manip_leg}gripper1"></child>
   </joint>

File: src/urdf_packer/urdf/hero_7dof/wheel_macro.xacro (robot description, xacro)
@@ -10,5 +10,5 @@
 </material>
 <xacro:macro name="add_wheel" params="prefix">
-  <link name="${prefix}wheel_body">
+  <link name="${prefix}body">
     <inertial>
       <origin xyz="0.012120027900982211 1.7479052741023483e-05 -0.1932995813581685" rpy="0 0 0"/>
@@ -30,5 +30,5 @@
     </collision>
   </link>
-  <link name="${prefix}wheel_left">
+  <link name="${prefix}left">
     <inertial>
       <origin xyz="6.05831716671279e-06 -0.079400296699694 3.750658923479255e-05" rpy="0 0 0"/>
@@ -50,5 +50,5 @@
     </collision>
   </link>
-  <link name="${prefix}wheel_right">
+  <link name="${prefix}right">
     <inertial>
       <origin xyz="-6.058317166268701e-06 0.07940029669969387 3.7506589234403975e-05" rpy="0 0 0"/>
@@ -70,33 +70,33 @@
     </collision>
   </link>
-  <link name="${prefix}wheel_in"/>
-  <link name="${prefix}wheel_center"/>
-  <link name="${prefix}wheel_out"/>
-  <joint name="${prefix}wheel_fix" type="fixed">
+  <link name="${prefix}in"/>
+  <link name="${prefix}center"/>
+  <link name="${prefix}out"/>
+  <joint name="${prefix}fix" type="fixed">
   <origin xyz="0 0 0.05" rpy="0 0 ${pi/2}"/>
-    <parent link="${prefix}wheel_in"/>
-    <child link="${prefix}wheel_body"/>
+    <parent link="${prefix}in"/>
+    <child link="${prefix}body"/>
   </joint>
-  <joint name="${prefix}wheel_cent_fix" type="fixed">
+  <joint name="${prefix}cent_fix" type="fixed">
   <origin xyz="0 0 -0.213" rpy="0 0 -${pi/2}"/>
-    <parent link="${prefix}wheel_body"/>
-    <child link="${prefix}wheel_center"/>
+    <parent link="${prefix}body"/>
+    <child link="${prefix}center"/>
   </joint>
-  <joint name="${prefix}wheel_left_joint" type="continuous">
+  <joint name="${prefix}left_joint" type="continuous">
     <origin xyz="0.004 0.277 -0.213" rpy="0 0 0"/>
-    <parent link="${prefix}wheel_body"/>
-    <child link="${prefix}wheel_left"/>
+    <parent link="${prefix}body"/>
+    <child link="${prefix}left"/>
     <axis xyz="0 1 0"/>
   </joint>
-  <joint name="${prefix}wheel_right_joint" type="continuous">
+  <joint name="${prefix}right_joint" type="continuous">
   <origin xyz="0.004 -0.277 -0.213" rpy="0 0 0"/>
-    <parent link="${prefix}wheel_body"/>
-    <child link="${prefix}wheel_right"/>
+    <parent link="${prefix}body"/>
+    <child link="${prefix}right"/>
     <axis xyz="0 1 0"/>
   </joint>
-  <joint name="${prefix}wheel_cen2out" type="fixed">
+  <joint name="${prefix}cen2out" type="fixed">
     <origin xyz="0 0.100 0" rpy="${-pi/2} 0 0"/>
-    <parent link="${prefix}wheel_center"/>
-    <child link="${prefix}wheel_out"/>
+    <parent link="${prefix}center"/>
+    <child link="${prefix}out"/>
     <axis xyz="0 0 0"/>
   </joint>
