Commit message: unified launc hfor moonbot

File: src/urdf_packer/urdf/hero_7dof/hero_dragon.xacro (robot description, xacro)
@@ -11,5 +11,5 @@
 <xacro:include filename="hero_7dofm3.xacro" ns="leg3"/>
 <joint name="bfix" type="fixed">
-<origin xyz="0 0 0.165" rpy="${pi/4} 0 0"/>
+<origin xyz="0 0 0" rpy="${1*pi/4} 0 0"/>
 <parent link="base_link"/>
 <child link="base_link45"/>
@@ -17,5 +17,5 @@
 <link name="base_link45" />
 <joint name="bfixstraight" type="fixed">
-<origin xyz="0 0 0" rpy="-${pi/4} 0 0"/>
+<origin xyz="0 0 0.165" rpy="0 0 0"/>
 <parent link="base_link45"/>
 <child link="1wheel_in"/>
@@ -34,5 +34,5 @@
 </joint>
 <joint name="fixwheel2" type="fixed">
-<origin xyz="0 0 0" rpy="0 0 0"/>
+<origin xyz="0 0 0" rpy="0 0 ${0*pi}"/>
 <parent link="leg4gripper2"/>
 <child link="2wheel_in"/>

Commit message: dragon again

File: src/urdf_packer/urdf/hero_7dof/hero_dragon.xacro (robot description, xacro)
@@ -5,9 +5,13 @@
 <xacro:property name="UrdfDataPath" value="package://${ThisPackage}/urdf/${Filename}" />
 <xacro:property name="MeshPath" value="package://${ThisPackage}/meshes/${Filename}" />
+<xacro:property name="main_leg" value="1" />
+<!-- also change that here !!!!    V   -->
+<xacro:include filename="hero_7dofm1.xacro" ns="leg${main_leg}"/>
+<xacro:property name="manip_leg" value="2" />
+<!-- also change that here !!!!    V   -->
+<xacro:include filename="hero_7dofm2.xacro" ns="leg${manip_leg}"/>
   <!-- Include the original xacro file -->
 <link name="base_link" />
 <xacro:include filename="wheel_macro.xacro"/>
-<xacro:include filename="hero_7dofm4.xacro" ns="leg4"/>
-<xacro:include filename="hero_7dofm3.xacro" ns="leg3"/>
 <joint name="bfix" type="fixed">
 <origin xyz="0 0 0" rpy="${1*pi/4} 0 0"/>
@@ -31,9 +35,9 @@
 <origin xyz="0 0 0" rpy="0 0 0"/>
 <parent link="1wheel_in"/>
-<child link="leg4gripper1"/>
+<child link="leg${main_leg}gripper1"/>
 </joint>
 <joint name="fixwheel2" type="fixed">
 <origin xyz="0 0 0" rpy="0 0 ${0*pi}"/>
-<parent link="leg4gripper2"/>
+<parent link="leg${main_leg}gripper2"/>
 <child link="2wheel_in"/>
 </joint>
@@ -48,12 +52,12 @@
 <origin xyz="0 0 0" rpy="0 0 0"/>
 <parent link="1wheel_out"/>
-<child link="leg3gripper1"/>
+<child link="leg${manip_leg}gripper1"/>
 </joint>
-<!-- <xacro:add_wheel  prefix="3" /> -->
+<!-- <xacro:add_wheel  prefix="${manip_leg}" /> -->
 <!---->
-<!-- <joint name="fixwheel1-3" type="fixed"> -->
+<!-- <joint name="fixwheel1-${manip_leg}" type="fixed"> -->
 <!-- <origin xyz="0 0 0" rpy="0 0 0"/> -->
 <!-- <parent link="leg4gripper2"/> -->
-<!-- <child link="3wheel_in"/> -->
+<!-- <child link="${manip_leg}wheel_in"/> -->
 <!-- </joint> -->
 </robot>

Commit message: ready for gragon

File: src/urdf_packer/urdf/hero_7dof/hero_dragon.xacro (robot description, xacro)
@@ -5,7 +5,7 @@
 <xacro:property name="UrdfDataPath" value="package://${ThisPackage}/urdf/${Filename}" />
 <xacro:property name="MeshPath" value="package://${ThisPackage}/meshes/${Filename}" />
-<xacro:property name="main_leg" value="1" />
+<xacro:property name="main_leg" value="4" />
 <!-- also change that here !!!!    V   -->
-<xacro:include filename="hero_7dofm1.xacro" ns="leg${main_leg}"/>
+<xacro:include filename="hero_7dofm4.xacro" ns="leg${main_leg}"/>
 <xacro:property name="manip_leg" value="2" />
 <!-- also change that here !!!!    V   -->

Commit message: dragon fix, not in general settings

File: src/urdf_packer/urdf/hero_7dof/hero_dragon.xacro (robot description, xacro)
@@ -5,10 +5,10 @@
 <xacro:property name="UrdfDataPath" value="package://${ThisPackage}/urdf/${Filename}" />
 <xacro:property name="MeshPath" value="package://${ThisPackage}/meshes/${Filename}" />
-<xacro:property name="main_leg" value="4" />
+<xacro:property name="main_leg" value="2" />
 <!-- also change that here !!!!    V   -->
-<xacro:include filename="hero_7dofm4.xacro" ns="leg${main_leg}"/>
-<xacro:property name="manip_leg" value="2" />
+<xacro:include filename="hero_7dofm2.xacro" ns="leg${main_leg}"/>
+<xacro:property name="manip_leg" value="3" />
 <!-- also change that here !!!!    V   -->
-<xacro:include filename="hero_7dofm2.xacro" ns="leg${manip_leg}"/>
+<xacro:include filename="hero_7dofm3.xacro" ns="leg${manip_leg}"/>
   <!-- Include the original xacro file -->
 <link name="base_link" />

Commit message: updated for drag

File: src/urdf_packer/urdf/hero_7dof/hero_dragon.xacro (robot description, xacro)
@@ -8,12 +8,12 @@
   <!--  -->
   <!--  -->
-  <xacro:property name="wheelfront" value="11"></xacro:property>
+  <xacro:property name="wheelfront" value="14"></xacro:property>
   <xacro:property name="wheelback" value="12"></xacro:property>
   <xacro:property name="main_leg" value="2"></xacro:property>
   <!-- also change that here !!!!    V   -->
-  <xacro:include filename="hero_7dofm2.xacro" ns="leg${main_leg}"></xacro:include>
+  <xacro:include filename="hero_7dofm2.xacro"></xacro:include>
   <xacro:property name="manip_leg" value="4"></xacro:property>
   <!-- also change that here !!!!    V   -->
-  <xacro:include filename="hero_7dofm4.xacro" ns="leg${manip_leg}"></xacro:include>
+  <xacro:include filename="hero_7dofm4.xacro"></xacro:include>
   <!--  -->
   <!--  -->

Commit message: operator unstuck

File: src/urdf_packer/urdf/hero_7dof/hero_dragon.xacro (robot description, xacro)
@@ -10,10 +10,10 @@
   <xacro:property name="wheelfront" value="wheel12_"></xacro:property>
   <xacro:property name="wheelback" value="wheel14_"></xacro:property>
-  <xacro:property name="bridge_leg" value="2"></xacro:property>
-  <!-- also change that here !!!!    V   -->
-  <xacro:include filename="hero_7dofm2.xacro"></xacro:include>
-  <xacro:property name="manip_leg" value="4"></xacro:property>
+  <xacro:property name="bridge_leg" value="4"></xacro:property>
   <!-- also change that here !!!!    V   -->
   <xacro:include filename="hero_7dofm4.xacro"></xacro:include>
+  <xacro:property name="manip_leg" value="3"></xacro:property>
+  <!-- also change that here !!!!    V   -->
+  <xacro:include filename="hero_7dofm3.xacro"></xacro:include>
   <!--  -->
   <!--  -->
