Commit message: in progress broken

File: src/urdf_packer/urdf/moonbot_7/moonbot_7.xacro (robot description, xacro)
@@ -22,5 +22,5 @@
     <parent link="base_link"/>
     <child link="body"/>
-    <origin rpy="0 0 2.35619449" xyz="0 0 0"/>
+    <origin rpy="0 0 ${-pi/4}" xyz="0 0 0"/>
   </joint>
   <link
