Commit message: fix end eff name to 0 by default

File: src/urdf_packer/urdf/ur16_3f/ur16_3f_old.xacro (robot description, xacro)
@@ -46,5 +46,5 @@
   </link>
   <link
-    name="forearm_link">
+    name="link1">
     <inertial>
       <origin
@@ -86,5 +86,5 @@
   </link>
   <joint
-    name="shoulder_lift_joint"
+    name="joint1"
     type="revolute">
     <origin
@@ -94,5 +94,5 @@
       link="base_link" />
     <child
-      link="forearm_link" />
+      link="link1" />
     <axis
       xyz="0 0 1" />
@@ -104,5 +104,5 @@
   </joint>
   <link
-    name="shoulder_link">
+    name="link2">
     <inertial>
       <origin
@@ -144,5 +144,5 @@
   </link>
   <joint
-    name="elbow_joint"
+    name="joint2"
     type="revolute">
     <origin
@@ -150,7 +150,7 @@
       rpy="1.5708 0 0" />
     <parent
-      link="forearm_link" />
+      link="link1" />
     <child
-      link="shoulder_link" />
+      link="link2" />
     <axis
       xyz="-0.3796 0 0.92515" />
@@ -162,5 +162,5 @@
   </joint>
   <link
-    name="upper_arm_link">
+    name="link3">
     <inertial>
       <origin
@@ -202,5 +202,5 @@
   </link>
   <joint
-    name="wrist_1_joint"
+    name="joint3"
     type="revolute">
     <origin
@@ -208,7 +208,7 @@
       rpy="0 -0.38936 0" />
     <parent
-      link="forearm_link" />
+      link="link2" />
     <child
-      link="upper_arm_link" />
+      link="link3" />
     <axis
       xyz="0 0 -1" />
@@ -220,5 +220,5 @@
   </joint>
   <link
-    name="wrist_1_link">
+    name="link4">
     <inertial>
       <origin
@@ -260,5 +260,5 @@
   </link>
   <joint
-    name="wrist_2_joint"
+    name="joint4"
     type="revolute">
     <origin
@@ -266,7 +266,7 @@
       rpy="0 0.38936 0" />
     <parent
-      link="upper_arm_link" />
+      link="link3" />
     <child
-      link="wrist_1_link" />
+      link="link4" />
     <axis
       xyz="-0.3796 0 0.92515" />
@@ -278,5 +278,5 @@
   </joint>
   <link
-    name="wrist_2_link">
+    name="link5">
     <inertial>
       <origin
@@ -318,5 +318,5 @@
   </link>
   <joint
-    name="wrist_3_joint"
+    name="joint5"
     type="revolute">
     <origin
@@ -324,7 +324,7 @@
       rpy="-1.5924 0.0011384 0.052648" />
     <parent
-      link="wrist_1_link" />
+      link="link4" />
     <child
-      link="wrist_2_link" />
+      link="link5" />
     <axis
       xyz="0 0 1" />
@@ -336,5 +336,5 @@
   </joint>
   <link
-    name="wrist_3_link">
+    name="link6">
     <inertial>
       <origin
@@ -376,5 +376,5 @@
   </link>
   <joint
-    name="shoudler_pan_joint"
+    name="joint6"
     type="revolute">
     <origin
@@ -382,7 +382,7 @@
       rpy="-1.5708 0.33462 1.4186" />
     <parent
-      link="wrist_2_link" />
+      link="link5" />
     <child
-      link="wrist_3_link" />
+      link="link6" />
     <axis
       xyz="0 0 1" />
@@ -400,5 +400,5 @@
       xyz="0 0 0.132"
       rpy="1.57 0 0" />
-    <parent link="wrist_3_link" />
+    <parent link="link6" />
     <child link="palm" />
     <axis
