Commit message: updated ur16e with real one

File: src/urdf_packer/urdf/ur16_3f/ur16_3f.xacro (robot description, xacro)
@@ -1,501 +1,307 @@
-<?xml version="1.0" ?>
+<?xml version="1.0" encoding="UTF-8"?>
 <robot name="ur16_3f" xmlns:xacro="http://www.ros.org/wiki/xacro">
-<xacro:property name="ThisPackage" value="urdf_packer" />
-<xacro:property name="Filename" value="ur16_3f" />
-<xacro:property name="UrdfDataPath" value="package://${ThisPackage}/urdf/${Filename}" />
-<xacro:property name="MeshPath" value="package://${ThisPackage}/meshes/${Filename}" />
-  <link
-    name="base_link">
-    <inertial>
-      <origin
-        xyz="7.5641E-05 0.022175 0.056242"
-        rpy="0 0 0" />
-      <mass
-        value="1.3189" />
-      <inertia
-        ixx="0.013561"
-        ixy="1.2819E-06"
-        ixz="2.3471E-06"
-        iyy="0.003855"
-        iyz="0.0014126"
-        izz="0.015106" />
-    </inertial>
-    <visual>
-      <origin
-        xyz="0 0 0"
-        rpy="0 0 0" />
-      <geometry>
-        <mesh
-        filename="${MeshPath}/base_link.STL" />
-      </geometry>
-      <material
-        name="">
-        <color
-          rgba="0.79216 0.81961 0.93333 1" />
-      </material>
-    </visual>
-    <collision>
-      <origin
-        xyz="0 0 0"
-        rpy="0 0 0" />
-      <geometry>
-        <mesh
-        filename="${MeshPath}/base_link.STL" />
-      </geometry>
-    </collision>
-  </link>
-  <link
-    name="forearm_link">
-    <inertial>
-      <origin
-        xyz="-0.0049712 -0.012113 0.083255"
-        rpy="0 0 0" />
-      <mass
-        value="3.4563" />
-      <inertia
-        ixx="0.013809"
-        ixy="-0.0005603"
-        ixz="8.6356E-05"
-        iyy="0.012674"
-        iyz="0.00021045"
-        izz="0.011893" />
-    </inertial>
-    <visual>
-      <origin
-        xyz="0 0 0"
-        rpy="0 0 0" />
-      <geometry>
-        <mesh
-        filename="${MeshPath}/link1.STL" />
-      </geometry>
-      <material
-        name="">
-        <color
-          rgba="0.79216 0.81961 0.93333 1" />
-      </material>
-    </visual>
-    <collision>
-      <origin
-        xyz="0 0 0"
-        rpy="0 0 0" />
-      <geometry>
-        <mesh
-        filename="${MeshPath}/link1.STL" />
-      </geometry>
-    </collision>
-  </link>
-  <joint
-    name="shoulder_lift_joint"
-    type="revolute">
-    <origin
-      xyz="0 0 0.0983"
-      rpy="0 0 0" />
-    <parent
-      link="base_link" />
-    <child
-      link="forearm_link" />
-    <axis
-      xyz="0 0 1" />
-    <limit
-      lower="-6.28"
-      upper="6.28"
-      effort="10.0"
-      velocity="6.28" />
-  </joint>
-  <link
-    name="shoulder_link">
-    <inertial>
-      <origin
-        xyz="-0.16137 0.12752 0.023124"
-        rpy="0 0 0" />
-      <mass
-        value="8.0873" />
-      <inertia
-        ixx="0.16123"
-        ixy="0.12191"
-        ixz="-0.050418"
-        iyy="0.166"
-        iyz="0.050437"
-        izz="0.2622" />
-    </inertial>
-    <visual>
-      <origin
-        xyz="0 0 0"
-        rpy="0 0 0" />
-      <geometry>
-        <mesh
-        filename="${MeshPath}/link2.STL" />
-      </geometry>
-      <material
-        name="">
-        <color
-          rgba="0.79216 0.81961 0.93333 1" />
-      </material>
-    </visual>
-    <collision>
-      <origin
-        xyz="0 0 0"
-        rpy="0 0 0" />
-      <geometry>
-        <mesh
-        filename="${MeshPath}/link2.STL" />
-      </geometry>
-    </collision>
-  </link>
-  <joint
-    name="elbow_joint"
-    type="revolute">
-    <origin
-      xyz="-0.035531 -0.086594 0.0824"
-      rpy="1.5708 0 0" />
-    <parent
-      link="forearm_link" />
-    <child
-      link="shoulder_link" />
-    <axis
-      xyz="-0.3796 0 0.92515" />
-    <limit
-      lower="-6.28"
-      upper="6.28"
-      effort="10.0"
-      velocity="6.28" />
-  </joint>
-  <link
-    name="upper_arm_link">
-    <inertial>
-      <origin
-        xyz="-0.08685 0.13999 -0.053044"
-        rpy="0 0 0" />
-      <mass
-        value="3.4237" />
-      <inertia
-        ixx="0.049767"
-        ixy="0.027689"
-        ixz="-0.001931"
-        iyy="0.022313"
-        iyz="0.0031129"
-        izz="0.066106" />
-    </inertial>
-    <visual>
-      <origin
-        xyz="0 0 0"
-        rpy="0 0 0" />
-      <geometry>
-        <mesh
-        filename="${MeshPath}/link3.STL" />
-      </geometry>
-      <material
-        name="">
-        <color
-          rgba="0.79216 0.81961 0.93333 1" />
-      </material>
-    </visual>
-    <collision>
-      <origin
-        xyz="0 0 0"
-        rpy="0 0 0" />
-      <geometry>
-        <mesh
-        filename="${MeshPath}/link3.STL" />
-      </geometry>
-    </collision>
-  </link>
-  <joint
-    name="wrist_1_joint"
-    type="revolute">
-    <origin
-      xyz="-0.32986 0.32151 -0.12931"
-      rpy="0 -0.38936 0" />
-    <parent
-      link="forearm_link" />
-    <child
-      link="upper_arm_link" />
-    <axis
-      xyz="0 0 -1" />
-    <limit
-      lower="-6.28"
-      upper="6.28"
-      effort="10.0"
-      velocity="6.28" />
-  </joint>
-  <link
-    name="wrist_1_link">
-    <inertial>
-      <origin
-        xyz="-0.020167 0.0015485 0.048913"
-        rpy="0 0 0" />
-      <mass
-        value="0.9534" />
-      <inertia
-        ixx="0.0017484"
-        ixy="3.4168E-05"
-        ixz="0.00017539"
-        iyy="0.0015085"
-        iyz="-3.6139E-05"
-        izz="0.0014004" />
-    </inertial>
-    <visual>
-      <origin
-        xyz="0 0 0"
-        rpy="0 0 0" />
-      <geometry>
-        <mesh
-        filename="${MeshPath}/link4.STL" />
-      </geometry>
-      <material
-        name="">
-        <color
-          rgba="0.79216 0.81961 0.93333 1" />
-      </material>
-    </visual>
-    <collision>
-      <origin
-        xyz="0 0 0"
-        rpy="0 0 0" />
-      <geometry>
-        <mesh
-        filename="${MeshPath}/link4.STL" />
-      </geometry>
-    </collision>
-  </link>
-  <joint
-    name="wrist_2_joint"
-    type="revolute">
-    <origin
-      xyz="-0.18979 0.30591 0.006123"
-      rpy="0 0.38936 0" />
-    <parent
-      link="upper_arm_link" />
-    <child
-      link="wrist_1_link" />
-    <axis
-      xyz="-0.3796 0 0.92515" />
-    <limit
-      lower="-6.28"
-      upper="6.28"
-      effort="10.0"
-      velocity="6.28" />
-  </joint>
-  <link
-    name="wrist_2_link">
-    <inertial>
-      <origin
-        xyz="-0.0017178 0.0002635 0.043297"
-        rpy="0 0 0" />
-      <mass
-        value="0.85443" />
-      <inertia
-        ixx="0.001132"
-        ixy="4.7099E-05"
-        ixz="3.6665E-05"
-        iyy="0.0014318"
-        iyz="-5.6254E-06"
-        izz="0.0012261" />
-    </inertial>
-    <visual>
-      <origin
-        xyz="0 0 0"
-        rpy="0 0 0" />
-      <geometry>
-        <mesh
-        filename="${MeshPath}/link5.STL" />
-      </geometry>
-      <material
-        name="">
-        <color
-          rgba="0.79216 0.81961 0.93333 1" />
-      </material>
-    </visual>
-    <collision>
-      <origin
-        xyz="0 0 0"
-        rpy="0 0 0" />
-      <geometry>
-        <mesh
-        filename="${MeshPath}/link5.STL" />
-      </geometry>
-    </collision>
-  </link>
-  <joint
-    name="wrist_3_joint"
-    type="revolute">
-    <origin
-      xyz="-0.029657 0.066842 0.062244"
-      rpy="-1.5924 0.0011384 0.052648" />
-    <parent
-      link="wrist_1_link" />
-    <child
-      link="wrist_2_link" />
-    <axis
-      xyz="0 0 1" />
-    <limit
-      lower="-6.28"
-      upper="6.28"
-      effort="10.0"
-      velocity="6.28" />
-  </joint>
-  <link
-    name="wrist_3_link">
-    <inertial>
-      <origin
-        xyz="-5.5756E-05 -5.5473E-05 0.027963"
-        rpy="0 0 0" />
-      <mass
-        value="0.35054" />
-      <inertia
-        ixx="0.00026479"
-        ixy="4.7422E-07"
-        ixz="3.6655E-08"
-        iyy="0.00026479"
-        iyz="3.6336E-08"
-        izz="0.00034748" />
-    </inertial>
-    <visual>
-      <origin
-        xyz="0 0 0"
-        rpy="0 0 0" />
-      <geometry>
-        <mesh
-        filename="${MeshPath}/link6.STL" />
-      </geometry>
-      <material
-        name="">
-        <color
-          rgba="0.79216 0.81961 0.93333 1" />
-      </material>
-    </visual>
-    <collision>
-      <origin
-        xyz="0 0 0"
-        rpy="0 0 0" />
-      <geometry>
-        <mesh
-        filename="${MeshPath}/link6.STL" />
-      </geometry>
-    </collision>
-  </link>
-  <joint
-    name="shoudler_pan_joint"
-    type="revolute">
-    <origin
-      xyz="-0.056045 0.0085955 0.0529"
-      rpy="-1.5708 0.33462 1.4186" />
-    <parent
-      link="wrist_2_link" />
-    <child
-      link="wrist_3_link" />
-    <axis
-      xyz="0 0 1" />
-    <limit
-      lower="-6.28"
-      upper="6.28"
-      effort="10.0"
-      velocity="6.28" />
+  <xacro:property name="ThisPackage" value="urdf_packer"></xacro:property>
+  <xacro:property name="Filename" value="ur16_3f"></xacro:property>
+  <xacro:property name="UrdfDataPath" value="package://${ThisPackage}/urdf/${Filename}"></xacro:property>
+  <xacro:property name="MeshPath" value="package://${ThisPackage}/meshes/${Filename}"></xacro:property>
+  <link name="world"></link>
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