Commit message: ALL handles all joint in urdf fixed

File: src/urdf_packer/urdf/ur16_3f/ur16_3f.xacro (robot description, xacro)
@@ -209,99 +209,108 @@
   </joint>
   <!--Start of 3f gripper joint and linkages-->
-  <joint name="joint7" type="revolute">
-    <origin rpy="1.57 0 0" xyz="0 0 0.132"></origin>
-    <parent link="wrist_3_link"></parent>
-    <child link="palm"></child>
-    <axis xyz="0 0 1"></axis>
-    <limit effort="0" lower="0" upper="0" velocity="0"></limit>
-  </joint>
-  <!--Palm link-->
+ <joint
+    name="tool_joint"
+    type="revolute">
+    <origin
+      xyz="0 0 0.132"
+      rpy="1.57 0 0" />
+    <parent link="wrist_3_link" />
+    <child link="palm" />
+    <axis
+      xyz="0 0 1" />
+    <limit
+      lower="0"
+      upper="0"
+      effort="0"
+      velocity="0" />
+  </joint>
+<!--Palm link-->
   <link name="palm">
     <visual>
       <geometry>
-        <mesh filename="${MeshPath}/robotiq-3f-gripper_articulated/visual/palm_new.stl"></mesh>
+      <mesh filename="${MeshPath}/robotiq-3f-gripper_articulated/visual/palm_new.stl"/>
       </geometry>
       <material name="green">
-        <color rgba="0 1 0 1"></color>
-      </material>
-    </visual>
-    <collision>
-      <geometry>
-        <mesh filename="${MeshPath}/robotiq-3f-gripper_articulated/collision/palm_new.stl"></mesh>
+        <color rgba="0 1 0 1"/>
+      </material>
+    </visual>
+    <collision>
+      <geometry>
+      <mesh filename="${MeshPath}/robotiq-3f-gripper_articulated/collision/palm_new.stl"/>
       </geometry>
       <material name="yellow">
-        <color rgba="0 1 1 1"></color>
+        <color rgba="0 1 1 1"/>
       </material>
     </collision>
   </link>
   <inertial>
-    <origin rpy="1.57 0 0" xyz="0 0 0.132"></origin>
-    <mass value="1.3"></mass>
-    <inertia ixx="0.078" ixy="-6.419E-07" ixz="0" iyy="1.909E-08" iyz="5.645E-07" izz="0.078"></inertia>
+    <origin rpy="1.57 0 0" xyz="0 0 0.132"/>
+    <mass value="1.3"/>
+    <inertia ixx="0.078" ixy="-6.419E-07" ixz="0" iyy="1.909E-08" iyz="5.645E-07" izz="0.078"/>
   </inertial>
   <joint name="palm_finger_1_joint" type="revolute">
-    <parent link="palm"></parent>
-    <child link="finger_1_link_0"></child>
-    <axis xyz="0 1 0"></axis>
-    <origin rpy="0 3.1416 -1.57" xyz="-0.0455 0.0214 0.036"></origin>
-    <limit effort="100" lower="-0.16" upper="0.25" velocity="100"></limit>
+    <parent link="palm"/>
+    <child link="finger_1_link_0"/>
+    <axis xyz="0 1 0"/>
+    <origin rpy="0 3.1416 -1.57" xyz="-0.0455 0.0214 0.036"/>
+    <limit effort="100" lower="-0.16" upper="0.25" velocity="100"/>
   </joint>
   <joint name="palm_finger_2_joint" type="revolute">
-    <parent link="palm"></parent>
-    <child link="finger_2_link_0"></child>
-    <axis xyz="0 1 0"></axis>
-    <origin rpy="0 3.1416 -1.57" xyz="-0.0455 0.0214 -0.036"></origin>
-    <limit effort="100" lower="-0.25" upper="0.16" velocity="100"></limit>
+    <parent link="palm"/>
+    <child link="finger_2_link_0"/>
+    <axis xyz="0 1 0"/>
+    <origin rpy="0 3.1416 -1.57" xyz="-0.0455 0.0214 -0.036"/>
+    <limit effort="100" lower="-0.25" upper="0.16" velocity="100"/>
   </joint>
   <joint name="palm_finger_middle_joint" type="fixed">
-    <parent link="palm"></parent>
-    <child link="finger_middle_link_0"></child>
-    <axis xyz="0 0 1"></axis>
-    <origin rpy="0 0 1.57" xyz="0.0455 0.0214 0"></origin>
+    <parent link="palm"/>
+    <child link="finger_middle_link_0"/>
+    <axis xyz="0 0 1"/>
+    <origin rpy="0 0 1.57" xyz="0.0455 0.0214 0"/>
   </joint>
   <link name="finger_1_link_0">
     <visual>
-      <origin rpy="0 0 0" xyz="0.020 0 0"></origin>
-      <geometry>
-        <mesh filename="${MeshPath}/robotiq-3f-gripper_articulated/visual/link_0.STL"></mesh>
+      <origin rpy="0 0 0" xyz="0.020 0 0"/>
+      <geometry>
+      <mesh filename="${MeshPath}/robotiq-3f-gripper_articulated/visual/link_0.STL"/>
       </geometry>
       <material name="green">
-        <color rgba="0 1 0 1"></color>
-      </material>
-    </visual>
-    <collision>
-      <origin rpy="0 3.1416 -1.57" xyz="-0.0455 0.0414 0.036"></origin>
-      <geometry>
-        <mesh filename="${MeshPath}/robotiq-3f-gripper_articulated/collision/link_0.STL"></mesh>
+        <color rgba="0 1 0 1"/>
+      </material>
+    </visual>
+    <collision>
+      <origin rpy="0 3.1416 -1.57" xyz="-0.0455 0.0414 0.036"/>
+      <geometry>
+      <mesh filename="${MeshPath}/robotiq-3f-gripper_articulated/collision/link_0.STL"/>
       </geometry>
       <material name="yellow">
-        <color rgba="0 1 1 1"></color>
-      </material>
-    </collision>
-    <inertial>
-      <origin rpy="0 0 0" xyz="0 0 0"></origin>
-      <mass value="0.05"></mass>
-      <inertia ixx="0.01" ixy="-0.00002" ixz="0.00001" iyy="0.0008" iyz="0" izz="0.001"></inertia>
+        <color rgba="0 1 1 1"/>
+      </material>
+    </collision>
+    <inertial>
+      <origin rpy="0 0 0" xyz="0 0 0"/>
+      <mass value="0.05"/>
+      <inertia ixx="0.01" ixy="-0.00002" ixz="0.00001" iyy="0.0008" iyz="0" izz="0.001"/>
     </inertial>
   </link>
   <link name="finger_1_link_1">
     <visual>
-      <origin rpy="0 0 -0.52" xyz="0.050 -.028 0"></origin>
-      <geometry>
-        <mesh filename="${MeshPath}/robotiq-3f-gripper_articulated/visual/link_1.STL"></mesh>
-      </geometry>
-      <material name="green"></material>
-    </visual>
-    <collision>
-      <origin rpy="0 0 -0.52" xyz="0.050 -.028 0"></origin>
-      <geometry>
-        <mesh filename="${MeshPath}/robotiq-3f-gripper_articulated/collision/link_1.STL"></mesh>
-      </geometry>
-      <material name="yellow"></material>
-    </collision>
-    <inertial>
-      <origin rpy="0 0 0" xyz="0 0 0"></origin>
-      <mass value="0.15"></mass>
-      <inertia ixx="0.001859" ixy="-0.000376" ixz="0.000028" iyy="0.012756" iyz="0" izz="0.0024"></inertia>
+      <origin rpy="0 0 -0.52" xyz="0.050 -.028 0"/>
+      <geometry>
+      <mesh filename="${MeshPath}/robotiq-3f-gripper_articulated/visual/link_1.STL"/>
+      </geometry>
+      <material name="green"/>
+    </visual>
+    <collision>
+      <origin rpy="0 0 -0.52" xyz="0.050 -.028 0"/>
+      <geometry>
+      <mesh filename="${MeshPath}/robotiq-3f-gripper_articulated/collision/link_1.STL"/>
+      </geometry>
+      <material name="yellow"/>
+    </collision>
+    <inertial>
+      <origin rpy="0 0 0" xyz="0 0 0"/>
+      <mass value="0.15"/>
+      <inertia ixx="0.001859" ixy="-0.000376" ixz="0.000028" iyy="0.012756" iyz="0" izz="0.0024"/>
     </inertial>
   </link>
@@ -313,109 +322,109 @@
 			-->
     <visual>
-      <origin rpy="0 0 0" xyz="0.039 0 0.0075"></origin>
-      <geometry>
-        <mesh filename="${MeshPath}/robotiq-3f-gripper_articulated/visual/link_2.STL"></mesh>
-      </geometry>
-      <material name="green"></material>
-    </visual>
-    <collision>
-      <origin rpy="0 0 0" xyz="0.039 0 0.0075"></origin>
-      <geometry>
-        <mesh filename="${MeshPath}/robotiq-3f-gripper_articulated/collision/link_2.STL"></mesh>
-      </geometry>
-      <material name="yellow"></material>
-    </collision>
-    <inertial>
-      <origin rpy="0 0 0" xyz="0 0 0"></origin>
-      <mass value="0.15"></mass>
-      <inertia ixx="0.001859" ixy="-0.000376" ixz="0.000028" iyy="0.012756" iyz="0" izz="0.0024"></inertia>
+      <origin rpy="0 0 0" xyz="0.039 0 0.0075"/>
+      <geometry>
+      <mesh filename="${MeshPath}/robotiq-3f-gripper_articulated/visual/link_2.STL"/>
+      </geometry>
+      <material name="green"/>
+    </visual>
+    <collision>
+      <origin rpy="0 0 0" xyz="0.039 0 0.0075"/>
+      <geometry>
+      <mesh filename="${MeshPath}/robotiq-3f-gripper_articulated/collision/link_2.STL"/>
+      </geometry>
+      <material name="yellow"/>
+    </collision>
+    <inertial>
+      <origin rpy="0 0 0" xyz="0 0 0"/>
+      <mass value="0.15"/>
+      <inertia ixx="0.001859" ixy="-0.000376" ixz="0.000028" iyy="0.012756" iyz="0" izz="0.0024"/>
     </inertial>
   </link>
   <link name="finger_1_link_3">
     <visual>
-      <origin rpy="0 0 0.52" xyz="0 0 0"></origin>
-      <geometry>
-        <mesh filename="${MeshPath}/robotiq-3f-gripper_articulated/visual/link_3.STL"></mesh>
-      </geometry>
-      <material name="green"></material>
-    </visual>
-    <collision>
-      <origin rpy="0 0 0.52" xyz="0 0 0"></origin>
-      <geometry>
-        <mesh filename="${MeshPath}/robotiq-3f-gripper_articulated/collision/link_3.STL"></mesh>
-      </geometry>
-      <material name="yellow"></material>
-    </collision>
-    <inertial>
-      <origin rpy="0 0 0" xyz="0 0 0"></origin>
-      <mass value="0.05"></mass>
-      <inertia ixx="0.001239" ixy="-0.000251" ixz="0.000019" iyy="0.00085" iyz="0" izz="0.001632"></inertia>
+      <origin rpy="0 0 0.52" xyz="0 0 0"/>
+      <geometry>
+      <mesh filename="${MeshPath}/robotiq-3f-gripper_articulated/visual/link_3.STL"/>
+      </geometry>
+      <material name="green"/>
+    </visual>
+    <collision>
+      <origin rpy="0 0 0.52" xyz="0 0 0"/>
+      <geometry>
+      <mesh filename="${MeshPath}/robotiq-3f-gripper_articulated/collision/link_3.STL"/>
+      </geometry>
+      <material name="yellow"/>
+    </collision>
+    <inertial>
+      <origin rpy="0 0 0" xyz="0 0 0"/>
+      <mass value="0.05"/>
+      <inertia ixx="0.001239" ixy="-0.000251" ixz="0.000019" iyy="0.00085" iyz="0" izz="0.001632"/>
     </inertial>
   </link>
   <joint name="finger_1_joint_1" type="revolute">
-    <parent link="finger_1_link_0"></parent>
-    <child link="finger_1_link_1"></child>
-    <axis xyz="0 0 1"></axis>
-    <origin rpy="0 0 0" xyz="0.020 0 0"></origin>
-    <limit effort="100" lower="0" upper="3.1416" velocity="100"></limit>
+    <parent link="finger_1_link_0"/>
+    <child link="finger_1_link_1"/>
+    <axis xyz="0 0 1"/>
+    <origin rpy="0 0 0" xyz="0.020 0 0"/>
+    <limit effort="100" lower="0" upper="3.1416" velocity="100"/>
   </joint>
   <joint name="finger_1_joint_2" type="revolute">
-    <parent link="finger_1_link_1"></parent>
-    <child link="finger_1_link_2"></child>
-    <axis xyz="0 0 1"></axis>
-    <origin rpy="0 0 -0.52" xyz="0.050 -.028 0"></origin>
-    <limit effort="100" lower="0" upper="3.1416" velocity="100"></limit>
+    <parent link="finger_1_link_1"/>
+    <child link="finger_1_link_2"/>
+    <axis xyz="0 0 1"/>
+    <origin rpy="0 0 -0.52" xyz="0.050 -.028 0"/>
+    <limit effort="100" lower="0" upper="3.1416" velocity="100"/>
   </joint>
   <joint name="finger_1_joint_3" type="revolute">
-    <parent link="finger_1_link_2"></parent>
-    <child link="finger_1_link_3"></child>
-    <axis xyz="0 0 1"></axis>
-    <origin rpy="0 0 0" xyz="0.039 0 0"></origin>
-    <limit effort="100" lower="0" upper="3.1416" velocity="100"></limit>
+    <parent link="finger_1_link_2"/>
+    <child link="finger_1_link_3"/>
+    <axis xyz="0 0 1"/>
+    <origin rpy="0 0 0" xyz="0.039 0 0"/>
+    <limit effort="100" lower="0" upper="3.1416" velocity="100"/>
   </joint>
   <link name="finger_2_link_0">
     <visual>
-      <origin rpy="0 0 0" xyz="0.020 0 0"></origin>
-      <geometry>
-        <mesh filename="${MeshPath}/robotiq-3f-gripper_articulated/visual/link_0.STL"></mesh>
+      <origin rpy="0 0 0" xyz="0.020 0 0"/>
+      <geometry>
+      <mesh filename="${MeshPath}/robotiq-3f-gripper_articulated/visual/link_0.STL"/>
       </geometry>
       <material name="green">
-        <color rgba="0 1 0 1"></color>
-      </material>
-    </visual>
-    <collision>
-      <origin rpy="0 3.1416 -1.57" xyz="-0.0455 0.0414 0.036"></origin>
-      <geometry>
-        <mesh filename="${MeshPath}/robotiq-3f-gripper_articulated/collision/link_0.STL"></mesh>
+        <color rgba="0 1 0 1"/>
+      </material>
+    </visual>
+    <collision>
+      <origin rpy="0 3.1416 -1.57" xyz="-0.0455 0.0414 0.036"/>
+      <geometry>
+      <mesh filename="${MeshPath}/robotiq-3f-gripper_articulated/collision/link_0.STL"/>
       </geometry>
       <material name="yellow">
-        <color rgba="0 1 1 1"></color>
-      </material>
-    </collision>
-    <inertial>
-      <origin rpy="0 0 0" xyz="0 0 0"></origin>
-      <mass value="0.05"></mass>
-      <inertia ixx="0.01" ixy="-0.00002" ixz="0.00001" iyy="0.0008" iyz="0" izz="0.001"></inertia>
+        <color rgba="0 1 1 1"/>
+      </material>
+    </collision>
+    <inertial>
+      <origin rpy="0 0 0" xyz="0 0 0"/>
+      <mass value="0.05"/>
+      <inertia ixx="0.01" ixy="-0.00002" ixz="0.00001" iyy="0.0008" iyz="0" izz="0.001"/>
     </inertial>
   </link>
   <link name="finger_2_link_1">
     <visual>
-      <origin rpy="0 0 -0.52" xyz="0.050 -.028 0"></origin>
-      <geometry>
-        <mesh filename="${MeshPath}/robotiq-3f-gripper_articulated/visual/link_1.STL"></mesh>
-      </geometry>
-      <material name="green"></material>
-    </visual>
-    <collision>
-      <origin rpy="0 0 -0.52" xyz="0.050 -.028 0"></origin>
-      <geometry>
-        <mesh filename="${MeshPath}/robotiq-3f-gripper_articulated/collision/link_1.STL"></mesh>
-      </geometry>
-      <material name="yellow"></material>
-    </collision>
-    <inertial>
-      <origin rpy="0 0 0" xyz="0 0 0"></origin>
-      <mass value="0.15"></mass>
-      <inertia ixx="0.001859" ixy="-0.000376" ixz="0.000028" iyy="0.012756" iyz="0" izz="0.0024"></inertia>
+      <origin rpy="0 0 -0.52" xyz="0.050 -.028 0"/>
+      <geometry>
+      <mesh filename="${MeshPath}/robotiq-3f-gripper_articulated/visual/link_1.STL"/>
+      </geometry>
+      <material name="green"/>
+    </visual>
+    <collision>
+      <origin rpy="0 0 -0.52" xyz="0.050 -.028 0"/>
+      <geometry>
+      <mesh filename="${MeshPath}/robotiq-3f-gripper_articulated/collision/link_1.STL"/>
+      </geometry>
+      <material name="yellow"/>
+    </collision>
+    <inertial>
+      <origin rpy="0 0 0" xyz="0 0 0"/>
+      <mass value="0.15"/>
+      <inertia ixx="0.001859" ixy="-0.000376" ixz="0.000028" iyy="0.012756" iyz="0" izz="0.0024"/>
     </inertial>
   </link>
@@ -427,109 +436,109 @@
 			-->
     <visual>
-      <origin rpy="0 0 0" xyz="0.039 0 0.0075"></origin>
-      <geometry>
-        <mesh filename="${MeshPath}/robotiq-3f-gripper_articulated/visual/link_2.STL"></mesh>
-      </geometry>
-      <material name="green"></material>
-    </visual>
-    <collision>
-      <origin rpy="0 0 0" xyz="0.039 0 0.0075"></origin>
-      <geometry>
-        <mesh filename="${MeshPath}/robotiq-3f-gripper_articulated/collision/link_2.STL"></mesh>
-      </geometry>
-      <material name="yellow"></material>
-    </collision>
-    <inertial>
-      <origin rpy="0 0 0" xyz="0 0 0"></origin>
-      <mass value="0.15"></mass>
-      <inertia ixx="0.001859" ixy="-0.000376" ixz="0.000028" iyy="0.012756" iyz="0" izz="0.0024"></inertia>
+      <origin rpy="0 0 0" xyz="0.039 0 0.0075"/>
+      <geometry>
+      <mesh filename="${MeshPath}/robotiq-3f-gripper_articulated/visual/link_2.STL"/>
+      </geometry>
+      <material name="green"/>
+    </visual>
+    <collision>
+      <origin rpy="0 0 0" xyz="0.039 0 0.0075"/>
+      <geometry>
+      <mesh filename="${MeshPath}/robotiq-3f-gripper_articulated/collision/link_2.STL"/>
+      </geometry>
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
Commit message: ee fix ur16

File: src/urdf_packer/urdf/ur16_3f/ur16_3f.xacro (robot description, xacro)
@@ -211,5 +211,5 @@
  <joint
     name="tool_joint"
-    type="revolute">
+    type="fixed">
     <origin
       xyz="0 0 0.132"
@@ -244,4 +244,14 @@
     </collision>
   </link>
+  <link name="palm_straight"/>
+ <joint
+    name="palm_str_fix"
+    type="fixed">
+    <origin
+      xyz="0 0 0"
+      rpy="1.57 0 1.57" />
+    <parent link="palm" />
+    <child link="palm_straight" />
+  </joint>
   <inertial>
     <origin rpy="1.57 0 0" xyz="0 0 0.132"/>

Commit message: more launchers

File: src/urdf_packer/urdf/ur16_3f/ur16_3f.xacro (robot description, xacro)
@@ -5,5 +5,4 @@
   <xacro:property name="UrdfDataPath" value="package://${ThisPackage}/urdf/${Filename}"></xacro:property>
   <xacro:property name="MeshPath" value="package://${ThisPackage}/meshes/${Filename}"></xacro:property>
-  <link name="world"></link>
   <!-- links -  main serial chain -->
   <link name="base_link"></link>
@@ -142,9 +141,4 @@
   </link>
   <!-- base_joint fixes base_link to the environment -->
-  <joint name="base_joint" type="fixed">
-    <origin rpy="0 0 0" xyz="0 0 0"></origin>
-    <parent link="world"></parent>
-    <child link="base_link"></child>
-  </joint>
   <!-- joints - main serial chain -->
   <joint name="base_link-base_link_inertia" type="fixed">
