Commit message: meshes repaired and urdf realigned

File: src/ros2_m_hero_pkg/urdf/hero_7dof_arm.xacro (robot description, xacro)
@@ -27,5 +27,5 @@
     </link>
     <joint name="${prefix}gripper1_fixed_joint" type="fixed">
-        <origin xyz="0 0 -0.075" rpy="0 0 0" />
+    <origin xyz="0 0 0.075" rpy="${pi} 0 ${+pi/2}" />
         <parent link="${prefix}gripper1" />
         <child link="${prefix}gripper1_base"/>
@@ -134,5 +134,5 @@
     </link>
     <joint name="${prefix}joint1" type="continuous">
-        <origin xyz="0 0 0.011" rpy="${pi} 0 0" />
+    <origin xyz="0 0 0.011" rpy="${pi} 0 ${pi/2}" />
         <parent link="${prefix}gripper1_base" />
         <child link="${prefix}link1" />
@@ -314,5 +314,5 @@
     </link>
     <joint name="${prefix}joint7" type="continuous">
-        <origin xyz="0.1646 0 0.072902" rpy="${-pi/2} ${pi} ${-pi/2}" />
+    <origin xyz="0.1646 0 0.072902" rpy="0 ${pi/2} 0" />
         <parent link="${prefix}link6" />
         <child link="${prefix}gripper2_base" />
@@ -382,8 +382,15 @@
     </link>
     <joint name="${prefix}gripper2_fixed_joint" type="fixed">
-        <origin xyz="0 0 0.065" rpy="0 0 0" />
+    <origin xyz="0 0 0.065" rpy="0 ${pi} ${-pi/2}" />
         <parent link="${prefix}gripper2_base" />
         <child link="${prefix}gripper2" />
     </joint>
+    <link name="${prefix}gripper2_straight">
+    </link>
+    <joint name="${prefix}gripper2_fix_to_straight" type="fixed">
+    <origin xyz="0 0 0" rpy="0 ${pi/2} 0" />
+        <parent link="${prefix}gripper2" />
+        <child link="${prefix}gripper2_straight" />
+    </joint>
     </xacro:macro>
 </robot>

Commit message: optimised mesh

File: src/ros2_m_hero_pkg/urdf/hero_7dof_arm.xacro (robot description, xacro)
@@ -5,5 +5,5 @@
 <robot xmlns:xacro="http://www.ros.org/wiki/xacro" name="hero_7dof_arm">
     <xacro:property name="ThisPackage" value="ros2_m_hero_pkg" />
-    <xacro:property name="MeshPath" value="package://${ThisPackage}/meshes/hero_7dof_arm" />
+    <xacro:property name="MeshPath" value="package://${ThisPackage}/meshes/hero_7dof_arm/optimised" />
     <xacro:property name="mesh_extension" value="STL" />
     <xacro:macro name="get_hero" params="prefix off_base_link_link2 off_link2_link3 off_link3_link4 off_link4_link5 off_link5_link6 off_link6_link7 off_link7_link8">

File: src/ros2_m_hero_pkg/urdf/hero_wheel_module.xacro (robot description, xacro)
@@ -5,5 +5,5 @@
 <robot xmlns:xacro="http://www.ros.org/wiki/xacro" name="hero_wheel_module">
   <xacro:property name="ThisPackage" value="ros2_m_hero_pkg" />
-  <xacro:property name="MeshPath" value="package://${ThisPackage}/meshes/hero_wheel_module" />
+  <xacro:property name="MeshPath" value="package://${ThisPackage}/meshes/hero_wheel_module/optimised" />
   <xacro:property name="mesh_extension" value="STL" />
   <xacro:macro name="add_wheel" params="prefix">

Commit message: offset and names for new urdf

File: src/ros2_m_hero_pkg/urdf/hero_7dof_arm.xacro (robot description, xacro)
@@ -75,5 +75,5 @@
         </collision>
     </link>
-    <joint name="${prefix}gripper1_jaw_left_joint" type="prismatic">
+    <joint name="${prefix}grip1" type="prismatic">
         <origin xyz="0 -0.025 0.075" rpy="${-pi/2} ${-pi/2} ${-pi/2}" />
         <parent link="${prefix}gripper1_base" />
@@ -104,5 +104,5 @@
         </collision>
     </link>
-    <joint name="${prefix}gripper1_jaw_right_joint" type="prismatic">
+    <joint name="${prefix}grip1bis" type="prismatic">
         <origin xyz="0 0.025 0.075" rpy="${pi/2} ${-pi/2} ${-pi/2}" />
         <parent link="${prefix}gripper1_base" />
@@ -343,5 +343,5 @@
         </collision>
     </link>
-    <joint name="${prefix}gripper2_jaw_left_joint" type="prismatic">
+    <joint name="${prefix}grip2" type="prismatic">
         <origin xyz="0 -0.025 0.065" rpy="${-pi/2} ${-pi/2} ${-pi/2}" />
         <parent link="${prefix}gripper2_base" />
@@ -372,5 +372,5 @@
         </collision>
     </link>
-    <joint name="${prefix}gripper2_jaw_right_joint" type="prismatic">
+    <joint name="${prefix}grip2bis" type="prismatic">
         <origin xyz="0 0.025 0.065" rpy="${pi/2} ${-pi/2} ${-pi/2}" />
         <parent link="${prefix}gripper2_base" />

Commit message: working irl, reampping done, urdf corrected

File: src/ros2_m_hero_pkg/urdf/hero_7dof_arm.xacro (robot description, xacro)
@@ -137,5 +137,5 @@
         <parent link="${prefix}gripper1_base" />
         <child link="${prefix}link1" />
-        <axis xyz="0 0 -1" />
+        <axis xyz="0 0 1" />
         <limit upper="${max_base_link_link2}" lower="${min_base_link_link2}" effort="100.0"
                 velocity="1300" />
@@ -167,5 +167,5 @@
         <parent link="${prefix}link1" />
         <child link="${prefix}link2" />
-        <axis xyz="0 0 -1" />
+        <axis xyz="0 0 1" />
         <limit upper="${max_link2_link3}" lower="${min_link2_link3}" effort="100.0"
                 velocity="1300" />
@@ -197,5 +197,5 @@
         <parent link="${prefix}link2" />
         <child link="${prefix}link3" />
-        <axis xyz="0 0 -1" />
+        <axis xyz="0 0 1" />
         <limit upper="${max_link3_link4}" lower="${min_link3_link4}" effort="100.0"
                 velocity="1300" />
@@ -227,5 +227,5 @@
         <parent link="${prefix}link3" />
         <child link="${prefix}link4" />
-        <axis xyz="0 0 1" />
+        <axis xyz="0 0 -1" />
         <limit upper="${max_link4_link5}" lower="${min_link4_link5}" effort="100.0"
                 velocity="1300" />
@@ -257,5 +257,5 @@
         <parent link="${prefix}link4" />
         <child link="${prefix}link5" />
-        <axis xyz="0 0 -1" />
+        <axis xyz="0 0 1" />
         <limit upper="${max_link5_link6}" lower="${min_link5_link6}" effort="100.0"
                 velocity="1300" />
@@ -287,5 +287,5 @@
         <parent link="${prefix}link5" />
         <child link="${prefix}link6" />
-        <axis xyz="0 0 -1" />
+        <axis xyz="0 0 1" />
         <limit upper="${max_link6_link7}" lower="${min_link6_link7}" effort="100.0"
                 velocity="1300" />

Commit message: updated urdf with mimic joints

File: src/ros2_m_hero_pkg/urdf/hero_7dof_arm.xacro (robot description, xacro)
@@ -22,4 +22,5 @@
     <xacro:property name="min_link6_link7" value="${-1 * off_link6_link7 - pi}" />
     <xacro:property name="min_link7_link8" value="${-1 * off_link7_link8 - pi}" />
+    <xacro:property name="max_vel" value="0.15" />
     <!-- PREFIX BELOW IS FOR TESTING. TODO: REMOVE -->
     <!-- <xacro:property name="prefix" value = "arm1"/> -->
@@ -80,5 +81,5 @@
         <child link="${prefix}gripper1_jaw_left" />
         <axis xyz="0 0 -1" />
-        <limit lower="0" upper="0" effort="400.0" velocity="100.0" />
+        <limit lower="-9999" upper="9999" effort="9999" velocity="${max_vel}" />
     </joint>
     <link name="${prefix}gripper1_jaw_right">
@@ -109,5 +110,6 @@
         <child link="${prefix}gripper1_jaw_right" />
         <axis xyz="0 0 -1" />
-        <limit lower="0" upper="0" effort="400.0" velocity="100.0" />
+        <limit lower="-9999" upper="9999" effort="9999" velocity="${max_vel}" />
+        <mimic joint="${prefix}grip1" multiplier="1" offset="0" />
     </joint>
     <link name="${prefix}link1">
@@ -138,6 +140,5 @@
         <child link="${prefix}link1" />
         <axis xyz="0 0 1" />
-        <limit upper="${max_base_link_link2}" lower="${min_base_link_link2}" effort="100.0"
-                velocity="1300" />
+        <limit lower="-9999" upper="9999" effort="9999" velocity="${max_vel}" />
     </joint>
     <link name="${prefix}link2">
@@ -168,6 +169,5 @@
         <child link="${prefix}link2" />
         <axis xyz="0 0 1" />
-        <limit upper="${max_link2_link3}" lower="${min_link2_link3}" effort="100.0"
-                velocity="1300" />
+        <limit lower="-9999" upper="9999" effort="9999" velocity="${max_vel}" />
     </joint>
     <link name="${prefix}link3">
@@ -198,6 +198,5 @@
         <child link="${prefix}link3" />
         <axis xyz="0 0 1" />
-        <limit upper="${max_link3_link4}" lower="${min_link3_link4}" effort="100.0"
-                velocity="1300" />
+        <limit lower="-9999" upper="9999" effort="9999" velocity="${max_vel}" />
     </joint>
     <link name="${prefix}link4">
@@ -228,6 +227,5 @@
         <child link="${prefix}link4" />
         <axis xyz="0 0 -1" />
-        <limit upper="${max_link4_link5}" lower="${min_link4_link5}" effort="100.0"
-                velocity="1300" />
+        <limit lower="-9999" upper="9999" effort="9999" velocity="${max_vel}" />
     </joint>
     <link name="${prefix}link5">
@@ -258,6 +256,5 @@
         <child link="${prefix}link5" />
         <axis xyz="0 0 1" />
-        <limit upper="${max_link5_link6}" lower="${min_link5_link6}" effort="100.0"
-                velocity="1300" />
+        <limit lower="-9999" upper="9999" effort="9999" velocity="${max_vel}" />
     </joint>
     <link name="${prefix}link6">
@@ -288,6 +285,5 @@
         <child link="${prefix}link6" />
         <axis xyz="0 0 1" />
-        <limit upper="${max_link6_link7}" lower="${min_link6_link7}" effort="100.0"
-                velocity="1300" />
+        <limit lower="-9999" upper="9999" effort="9999" velocity="${max_vel}" />
     </joint>
     <link name="${prefix}gripper2_base">
@@ -318,6 +314,5 @@
         <child link="${prefix}gripper2_base" />
         <axis xyz="0 0 1" />
-        <limit upper="${max_link7_link8}" lower="${min_link7_link8}" effort="100.0"
-                velocity="1300" />
+        <limit lower="-9999" upper="9999" effort="9999" velocity="${max_vel}" />
     </joint>
     <link name="${prefix}gripper2_jaw_left">
@@ -348,5 +343,5 @@
         <child link="${prefix}gripper2_jaw_left" />
         <axis xyz="0 0 -1" />
-        <limit upper="0" lower="0" effort="100.0" velocity="1300" />
+        <limit lower="-9999" upper="9999" effort="9999" velocity="${max_vel}" />
     </joint>
     <link name="${prefix}gripper2_jaw_right">
@@ -377,5 +372,6 @@
         <child link="${prefix}gripper2_jaw_right" />
         <axis xyz="0 0 -1" />
-        <limit upper="0" lower="0" effort="100.0" velocity="1300" />
+        <limit lower="-9999" upper="9999" effort="9999" velocity="${max_vel}" />
+        <mimic joint="${prefix}grip2" multiplier="1" offset="0" />
     </joint>
     <link name="${prefix}gripper2">
