Commit message: realigned

File: src/ros2_m_hero_pkg/urdf/hero_3leg.xacro (robot description, xacro)
@@ -77,5 +77,5 @@
 <!---->
 <!---->
-<!-- <xacro:include filename="wheel_macro.xacro"/> -->
+<!-- <xacro:include filename="hero_wheel_module.xacro"/> -->
 <!---->
 <!-- <xacro:add_wheel prefix="11" /> -->

File: src/ros2_m_hero_pkg/urdf/hero_3legwheel.xacro (robot description, xacro)
@@ -2,5 +2,5 @@
 <robot xmlns:xacro="http://www.ros.org/wiki/xacro" name="hero_dragon">
 <xacro:include filename="hero_3leg.xacro"/>
-<xacro:include filename="wheel_macro.xacro"/>
+<xacro:include filename="hero_wheel_module.xacro"/>
 <!-- change wheel number here                 VV       -->
 <xacro:property name="wheelfront" value="wheel11_"></xacro:property>

File: src/ros2_m_hero_pkg/urdf/hero_7dof_all.xacro (robot description, xacro)
@@ -32,5 +32,5 @@
 <xacro:add_wheel prefix="wheel11_" />
 <joint name="fix11" type="fixed">
-<origin xyz="0.2 2 0" rpy="0 0 ${pi/2}"/>
+<origin xyz="0 2 0" rpy="0 0 0"/>
 <parent link="base_link"/>
 <child link="wheel11_in"/>
@@ -38,5 +38,5 @@
 <xacro:add_wheel prefix="wheel12_" />
 <joint name="fix12" type="fixed">
-<origin xyz="0.6 2 0" rpy="0 0 ${pi/2}"/>
+<origin xyz="0.6 2 0" rpy="0 0 0"/>
 <parent link="base_link"/>
 <child link="wheel12_in"/>
@@ -44,5 +44,5 @@
 <xacro:add_wheel prefix="wheel13_" />
 <joint name="fix13" type="fixed">
-<origin xyz="1 2 0" rpy="0 0 ${pi/2}"/>
+<origin xyz="1.2 2 0" rpy="0 0 0"/>
 <parent link="base_link"/>
 <child link="wheel13_in"/>
@@ -50,5 +50,5 @@
 <xacro:add_wheel prefix="wheel14_" />
 <joint name="fix14" type="fixed">
-<origin xyz="1.4 2 0" rpy="0 0 ${pi/2}"/>
+<origin xyz="1.8 2 0" rpy="0 0 0"/>
 <parent link="base_link"/>
 <child link="wheel14_in"/>

File: src/ros2_m_hero_pkg/urdf/hero_7dof_arm.xacro (robot description, xacro)
@@ -27,5 +27,5 @@
     </link>
     <joint name="${prefix}gripper1_fixed_joint" type="fixed">
-    <origin xyz="0 0 0.075" rpy="${pi} 0 ${+pi/2}" />
+    <origin xyz="0 0 0.075" rpy="${pi} 0 ${0}" />
         <parent link="${prefix}gripper1" />
         <child link="${prefix}gripper1_base"/>
@@ -134,5 +134,5 @@
     </link>
     <joint name="${prefix}joint1" type="continuous">
-    <origin xyz="0 0 0.011" rpy="${pi} 0 ${pi/2}" />
+    <origin xyz="0 0 0.011" rpy="${pi} 0 ${0}" />
         <parent link="${prefix}gripper1_base" />
         <child link="${prefix}link1" />
@@ -314,5 +314,5 @@
     </link>
     <joint name="${prefix}joint7" type="continuous">
-    <origin xyz="0.1646 0 0.072902" rpy="0 ${pi/2} 0" />
+    <origin xyz="0.1646 0 0.072902" rpy="${-pi/2} 0 ${-pi/2}" />
         <parent link="${prefix}link6" />
         <child link="${prefix}gripper2_base" />
@@ -382,5 +382,5 @@
     </link>
     <joint name="${prefix}gripper2_fixed_joint" type="fixed">
-    <origin xyz="0 0 0.065" rpy="0 ${pi} ${-pi/2}" />
+    <origin xyz="0 0 0.065" rpy="0 ${pi} ${0}" />
         <parent link="${prefix}gripper2_base" />
         <child link="${prefix}gripper2" />

File: src/ros2_m_hero_pkg/urdf/hero_dragon.xacro (robot description, xacro)
@@ -20,7 +20,7 @@
   <!--  -->
   <link name="base_link"></link>
-  <xacro:include filename="wheel_macro.xacro"></xacro:include>
+  <xacro:include filename="hero_wheel_module.xacro"></xacro:include>
   <joint name="bfix" type="fixed">
-    <origin rpy="${1*pi/4} 0 ${-pi/2}" xyz="0 0 0"></origin>
+  <origin rpy="0 ${pi/4 - pi/2} ${pi}" xyz="0 0 0"></origin>
     <parent link="base_link"></parent>
     <child link="base_link45"></child>
@@ -28,5 +28,5 @@
   <link name="base_link45"></link>
   <joint name="bfixstraight" type="fixed">
-    <origin rpy="0 0 0" xyz="0 0 0.165"></origin>
+    <origin rpy="0 0 0" xyz="0 0 0.160"></origin>
     <parent link="base_link45"></parent>
     <child link="${wheelfront}in"></child>
@@ -44,5 +44,5 @@
     <origin rpy="0 0 0" xyz="0 0 0"></origin>
     <parent link="${wheelfront}in"></parent>
-    <child link="leg${bridge_leg}gripper1"></child>
+    <child link="leg${manip_leg}gripper1"></child>
   </joint>
   <!---->
@@ -63,5 +63,5 @@
     <origin rpy="0 0 0" xyz="0 0 0"></origin>
     <parent link="${wheelfront}out"></parent>
-    <child link="leg${manip_leg}gripper1"></child>
+    <child link="leg${bridge_leg}gripper1"></child>
   </joint>
   <!-- <xacro:add_wheel  prefix="${manip_leg}" /> -->

File: src/ros2_m_hero_pkg/urdf/hero_vehicle.xacro (robot description, xacro)
@@ -11,5 +11,5 @@
   <xacro:include filename="hero_7dofm4.xacro" ns="leg${main_leg}"></xacro:include>
   <link name="base_link"></link>
-  <xacro:include filename="wheel_macro.xacro"></xacro:include>
+  <xacro:include filename="hero_wheel_module.xacro"></xacro:include>
   <joint name="bfix" type="fixed">
     <origin rpy="${1*pi/4} 0 ${-pi/2}" xyz="0 0 0"></origin>

File: src/ros2_m_hero_pkg/urdf/hero_wheel_module.xacro (robot description, xacro)
@@ -55,5 +55,5 @@
   </link>
   <joint name="${prefix}left_joint" type="continuous">
-    <origin xyz="0 -0.286 0" rpy="${pi/2} 0 0" />
+  <origin xyz="0 -0.286 0" rpy="${pi/2} 0 0" />
     <parent link="${prefix}body" />
     <child link="${prefix}left" />
@@ -94,15 +94,15 @@
   <link name="${prefix}out"/>
   <joint name="${prefix}fix" type="fixed">
-  <origin xyz="0 0 0.05" rpy="0 0 ${pi/2}"/>
+  <origin xyz="0 0 -0.16" rpy="0 ${pi/4} ${0}"/>
     <parent link="${prefix}in"/>
     <child link="${prefix}body"/>
   </joint>
   <joint name="${prefix}cent_fix" type="fixed">
-  <origin xyz="0 0 -0.213" rpy="0 0 -${pi/2}"/>
-    <parent link="${prefix}body"/>
+  <origin xyz="0 0 -0.16" rpy="0 0 0"/>
+    <parent link="${prefix}in"/>
     <child link="${prefix}center"/>
   </joint>
   <joint name="${prefix}cen2out" type="fixed">
-    <origin xyz="0 0.100 0" rpy="${-pi/2} 0 0"/>
+  <origin xyz="0.15 0 0" rpy="0 ${pi/2} 0"/>
     <parent link="${prefix}center"/>
     <child link="${prefix}out"/>

Commit message: 3 leg and vehicle xacro ok

File: src/ros2_m_hero_pkg/urdf/hero_3leg.xacro (robot description, xacro)
@@ -1,8 +1,6 @@
 <?xml version="1.0"?>
 <robot xmlns:xacro="http://www.ros.org/wiki/xacro" name="hero_dragon">
-<xacro:property name="ThisPackage" value="urdf_packer" />
-<xacro:property name="Filename" value="hero_7dof" />
-<xacro:property name="UrdfDataPath" value="package://${ThisPackage}/urdf/${Filename}" />
-<xacro:property name="MeshPath" value="package://${ThisPackage}/meshes/${Filename}" />
+<xacro:property name="ThisPackage" value="ros2_m_hero_pkg" />
+<xacro:property name="MeshPath" value="package://${ThisPackage}/meshes" />
 <xacro:property name="R" value="0.200" />
 <link name="base_link">
@@ -10,5 +8,5 @@
 	<origin xyz="0 0 0" rpy="0 0 1.04" />
       <geometry>
-        <mesh filename="${MeshPath}/hero_hub_unit.stl" scale="0.001 0.001 0.001">
+        <mesh filename="${MeshPath}/hero_hub_unit_opti.stl" scale="0.001 0.001 0.001">
 	</mesh>
       </geometry>
@@ -24,5 +22,5 @@
 <link name="d1" />
 <joint name="orient1" type="fixed">
-<origin xyz="0 0 0" rpy="${pi} 0 0"/>
+<origin xyz="0 0 0" rpy="${pi/2} 0 0"/>
 <parent link="base_link"/>
 <child link="d1"/>
@@ -36,5 +34,5 @@
 <link name="d2" />
 <joint name="orient2" type="fixed">
-<origin xyz="0 0 0" rpy="${pi} 0 ${2*pi/3}"/>
+<origin xyz="0 0 0" rpy="${pi/2} 0 ${2*pi/3}"/>
 <parent link="base_link"/>
 <child link="d2"/>
@@ -42,5 +40,5 @@
 <link name="d3" />
 <joint name="orient3" type="fixed">
-<origin xyz="0 0 0" rpy="${pi} 0 ${2*2*pi/3}"/>
+<origin xyz="0 0 0" rpy="${pi/2} 0 ${2*2*pi/3}"/>
 <parent link="base_link"/>
 <child link="d3"/>

File: src/ros2_m_hero_pkg/urdf/hero_dragon.xacro (robot description, xacro)
@@ -1,8 +1,4 @@
 <?xml version="1.0" encoding="UTF-8"?>
 <robot name="hero_dragon" xmlns:xacro="http://www.ros.org/wiki/xacro">
-  <xacro:property name="ThisPackage" value="urdf_packer"></xacro:property>
-  <xacro:property name="Filename" value="hero_7dof"></xacro:property>
-  <xacro:property name="UrdfDataPath" value="package://${ThisPackage}/urdf/${Filename}"></xacro:property>
-  <xacro:property name="MeshPath" value="package://${ThisPackage}/meshes/${Filename}"></xacro:property>
   <!-- change what leg is where -->
   <!--  -->

File: src/ros2_m_hero_pkg/urdf/hero_vehicle.xacro (robot description, xacro)
@@ -1,17 +1,19 @@
 <?xml version="1.0" encoding="UTF-8"?>
 <robot name="hero_vehicle" xmlns:xacro="http://www.ros.org/wiki/xacro">
-  <xacro:property name="ThisPackage" value="urdf_packer"></xacro:property>
-  <xacro:property name="Filename" value="hero_7dof"></xacro:property>
-  <xacro:property name="UrdfDataPath" value="package://${ThisPackage}/urdf/${Filename}"></xacro:property>
-  <xacro:property name="MeshPath" value="package://${ThisPackage}/meshes/${Filename}"></xacro:property>
-  <xacro:property name="wheelfront" value="11"></xacro:property>
-  <xacro:property name="wheelback" value="12"></xacro:property>
-  <xacro:property name="main_leg" value="4"></xacro:property>
+  <!-- change what leg is where -->
+  <!--  -->
+  <!--  -->
+  <xacro:property name="wheelfront" value="wheel11_"></xacro:property>
+  <xacro:property name="wheelback" value="wheel12_"></xacro:property>
+  <xacro:property name="bridge_leg" value="1"></xacro:property>
   <!-- also change that here !!!!    V   -->
-  <xacro:include filename="hero_7dofm4.xacro" ns="leg${main_leg}"></xacro:include>
+  <xacro:include filename="hero_7dofm1.xacro"></xacro:include>
+  <!--  -->
+  <!--  -->
+  <!--  -->
   <link name="base_link"></link>
   <xacro:include filename="hero_wheel_module.xacro"></xacro:include>
   <joint name="bfix" type="fixed">
-    <origin rpy="${1*pi/4} 0 ${-pi/2}" xyz="0 0 0"></origin>
+  <origin rpy="0 ${- pi/2} ${pi}" xyz="0 0 0"></origin>
     <parent link="base_link"></parent>
     <child link="base_link45"></child>
@@ -19,31 +21,34 @@
   <link name="base_link45"></link>
   <joint name="bfixstraight" type="fixed">
-    <origin rpy="0 0 ${-pi/2}" xyz="0 0 0.165"></origin>
-    <parent link="base_link"></parent>
-    <child link="${wheelfront}wheel_in"></child>
+    <origin rpy="0 0 0" xyz="0 0 0.160"></origin>
+    <parent link="base_link45"></parent>
+    <child link="${wheelfront}in"></child>
   </joint>
+  <!---->
+  <!---->
   <xacro:add_wheel prefix="${wheelfront}"></xacro:add_wheel>
-  <link name="wheel${wheelfront}c45"></link>
-  <joint name="fix45${wheelfront}" type="fixed">
-    <origin rpy="${-pi/4} 0 0" xyz="0 0 0"></origin>
-    <parent link="${wheelfront}wheel_center"></parent>
-    <child link="wheel${wheelfront}c45"></child>
-  </joint>
-  <joint name="fixwheel${wheelfront}" type="fixed">
-    <origin rpy="0 0 0" xyz="0 0 0"></origin>
-    <parent link="${wheelfront}wheel_in"></parent>
-    <child link="leg${main_leg}gripper1"></child>
-  </joint>
-  <joint name="fixwheel${wheelback}" type="fixed">
+  <joint name="${wheelback}fix1" type="fixed">
     <origin rpy="0 0 ${0*pi}" xyz="0 0 0"></origin>
-    <parent link="leg${main_leg}gripper2"></parent>
-    <child link="${wheelback}wheel_in"></child>
+    <parent link="leg${bridge_leg}gripper2"></parent>
+    <child link="${wheelback}in"></child>
   </joint>
   <xacro:add_wheel prefix="${wheelback}"></xacro:add_wheel>
-  <link name="wheel${wheelback}c45"></link>
-  <joint name="fix452" type="fixed">
-    <origin rpy="${pi/4} 0 0" xyz="0 0 0"></origin>
-    <parent link="${wheelback}wheel_center"></parent>
-    <child link="wheel${wheelback}c45"></child>
+  <link name="${wheelback}c45"></link>
+  <joint name="fix45${wheelback}" type="fixed">
+    <origin rpy="${0} 0 0" xyz="0 0 0"></origin>
+    <parent link="${wheelback}center"></parent>
+    <child link="${wheelback}c45"></child>
   </joint>
+  <joint name="${wheelfront}fix_out" type="fixed">
+    <origin rpy="0 0 0" xyz="0 0 0"></origin>
+    <parent link="${wheelfront}out"></parent>
+    <child link="leg${bridge_leg}gripper1"></child>
+  </joint>
+  <!-- <xacro:add_wheel  prefix="${manip_leg}" /> -->
+  <!---->
+  <!-- <joint name="fixwheel1-${manip_leg}" type="fixed"> -->
+  <!-- <origin xyz="0 0 0" rpy="0 0 0"/> -->
+  <!-- <parent link="leg4gripper2"/> -->
+  <!-- <child link="${manip_leg}wheel_in"/> -->
+  <!-- </joint> -->
 </robot>
