Commit message: xacro improved untested

File: src/ros2_m_hero_pkg/urdf/hero_3leg.xacro (robot description, xacro)
@@ -1,106 +1,70 @@
-<?xml version="1.0"?>
-<robot xmlns:xacro="http://www.ros.org/wiki/xacro" name="hero_dragon">
-<xacro:property name="ThisPackage" value="ros2_m_hero_pkg" />
-<xacro:property name="MeshPath" value="package://${ThisPackage}/meshes" />
-<xacro:property name="R" value="0.200" />
-<link name="base_link">
+<?xml version="1.0" encoding="UTF-8"?>
+<robot name="hero_dragon" xmlns:xacro="http://www.ros.org/wiki/xacro">
+  <xacro:property name="ThisPackage" value="ros2_m_hero_pkg"></xacro:property>
+  <xacro:property name="MeshPath" value="package://${ThisPackage}/meshes"></xacro:property>
+  <xacro:property name="body_radius" value="0.200"></xacro:property>
+    <xacro:property name="limbfront" value="1"></xacro:property>
+    <xacro:property name="limbleft" value="2"></xacro:property>
+    <xacro:property name="limbright" value="4"></xacro:property>
+  <link name="base_link">
     <visual>
-	<origin xyz="0 0 0" rpy="0 0 1.04" />
+      <origin rpy="0 0 1.04" xyz="0 0 0"></origin>
       <geometry>
-        <mesh filename="${MeshPath}/hero_hub_unit_opti.stl" scale="0.001 0.001 0.001">
-	</mesh>
+        <mesh filename="${MeshPath}/hero_hub_unit_opti.stl" scale="0.001 0.001 0.001"></mesh>
       </geometry>
-	<material
-        name="">
-        <color
-          rgba="0.627450980392157 0.627450980392157 0.627450980392157 1" />
+      <material name="">
+        <color rgba="0.627450980392157 0.627450980392157 0.627450980392157 1"></color>
       </material>
     </visual>
-</link>
-<link name="base_linkp" />
-<!-- fake end of gripper 3-2 -->
-<link name="d1" />
-<joint name="orient1" type="fixed">
-<origin xyz="0 0 0" rpy="${pi/2} 0 0"/>
-<parent link="base_link"/>
-<child link="d1"/>
-</joint>
-<link name="d1p" />
-<joint name="orient1p" type="fixed">
-<origin xyz="0 0 0" rpy="0 0 0"/>
-<parent link="d1p"/>
-<child link="base_linkp"/>
-</joint>
-<link name="d2" />
-<joint name="orient2" type="fixed">
-<origin xyz="0 0 0" rpy="${pi/2} 0 ${2*pi/3}"/>
-<parent link="base_link"/>
-<child link="d2"/>
-</joint>
-<link name="d3" />
-<joint name="orient3" type="fixed">
-<origin xyz="0 0 0" rpy="${pi/2} 0 ${2*2*pi/3}"/>
-<parent link="base_link"/>
-<child link="d3"/>
-</joint>
-<joint name="fix1" type="fixed">
-<origin xyz="${R} 0 0" rpy="0 ${pi/2} 0"/>
-<parent link="d1"/>
-<child link="leg1gripper1"/>
-</joint>
-<joint name="fix1p" type="fixed">
-<origin xyz="${R} 0 0" rpy="${pi} 0 ${pi}"/>
-<parent link="leg1gripper2_straight"/>
-<child link="d1p"/>
-</joint>
-<joint name="fix2" type="fixed">
-<origin xyz="${R} 0 0" rpy="0 ${pi/2} 0"/>
-<parent link="d3"/>
-<child link="leg4gripper1"/>
-</joint>
-<joint name="fix3" type="fixed">
-<origin xyz="${R} 0 0" rpy="0 ${pi/2} 0"/>
-<parent link="d2"/>
-<child link="leg2gripper1"/>
-</joint>
-<xacro:include filename="hero_7dofm4.xacro"/>
-<xacro:include filename="hero_7dofm2.xacro"/>
-<xacro:include filename="hero_7dofm1.xacro"/>
-<!-- <xacro:include filename="hero_7dofm4.xacro"/> -->
-<!-- <joint name="fix4" type="fixed"> -->
-<!-- <origin xyz="1 0 0.12" rpy="0 0 0"/> -->
-<!-- <parent link="base_link"/> -->
-<!-- <child link="leg4gripper1"/> -->
-<!-- </joint> -->
-<!---->
-<!---->
-<!-- <xacro:include filename="hero_wheel_module.xacro"/> -->
-<!---->
-<!-- <xacro:add_wheel prefix="11" /> -->
-<!-- <joint name="fix11" type="fixed"> -->
-<!-- <origin xyz="0 0 0" rpy="0 0 0"/> -->
-<!-- <parent link="base_link"/> -->
-<!-- <child link="11wheel_in"/> -->
-<!-- </joint> -->
-<!---->
-<!-- <xacro:add_wheel prefix="12" /> -->
-<!-- <joint name="fix12" type="fixed"> -->
-<!-- <origin xyz="0 0 0" rpy="0 0 0"/> -->
-<!-- <parent link="base_link"/> -->
-<!-- <child link="12wheel_in"/> -->
-<!-- </joint> -->
-<!---->
-<!-- <xacro:add_wheel prefix="13" /> -->
-<!-- <joint name="fix13" type="fixed"> -->
-<!-- <origin xyz="0 0 0" rpy="0 0 0"/> -->
-<!-- <parent link="base_link"/> -->
-<!-- <child link="13wheel_in"/> -->
-<!-- </joint> -->
-<!---->
-<!-- <xacro:add_wheel prefix="14" /> -->
-<!-- <joint name="fix14" type="fixed"> -->
-<!-- <origin xyz="0 0 0" rpy="0 0 0"/> -->
-<!-- <parent link="base_link"/> -->
-<!-- <child link="14wheel_in"/> -->
-<!-- </joint> -->
+  </link>
+  <link name="base_linkp"></link>
+  <!-- fake end of gripper 3-2 -->
+  <link name="d1"></link>
+  <joint name="orient1" type="fixed">
+    <origin rpy="${pi/2} 0 0" xyz="0 0 0"></origin>
+    <parent link="base_link"></parent>
+    <child link="d1"></child>
+  </joint>
+  <link name="d1p"></link>
+  <joint name="orient1p" type="fixed">
+    <origin rpy="0 0 0" xyz="0 0 0"></origin>
+    <parent link="d1p"></parent>
+    <child link="base_linkp"></child>
+  </joint>
+  <link name="d2"></link>
+  <joint name="orient2" type="fixed">
+    <origin rpy="${pi/2} 0 ${2*pi/3}" xyz="0 0 0"></origin>
+    <parent link="base_link"></parent>
+    <child link="d2"></child>
+  </joint>
+  <link name="d3"></link>
+  <joint name="orient3" type="fixed">
+    <origin rpy="${pi/2} 0 ${2*2*pi/3}" xyz="0 0 0"></origin>
+    <parent link="base_link"></parent>
+    <child link="d3"></child>
+  </joint>
+  <joint name="fix1" type="fixed">
+    <origin rpy="0 ${pi/2} 0" xyz="${body_radius} 0 0"></origin>
+    <parent link="d1"></parent>
+    <child link="leg${limbfront}gripper1"></child>
+  </joint>
+  <joint name="fix1p" type="fixed">
+    <origin rpy="${pi} 0 ${pi}" xyz="${body_radius} 0 0"></origin>
+    <parent link="leg${limbfront}gripper2_straight"></parent>
+    <child link="d1p"></child>
+  </joint>
+  <joint name="fix2" type="fixed">
+    <origin rpy="0 ${pi/2} 0" xyz="${body_radius} 0 0"></origin>
+    <parent link="d3"></parent>
+    <child link="leg${limbleft}gripper1"></child>
+  </joint>
+  <joint name="fix3" type="fixed">
+    <origin rpy="0 ${pi/2} 0" xyz="${body_radius} 0 0"></origin>
+    <parent link="d2"></parent>
+    <child link="leg${limbright}gripper1"></child>
+  </joint>
+  <xacro:include filename="hero_7dof_arm_macro.xacro"></xacro:include>
+  <xacro:get_hero prefix="leg${limbfront}"></xacro:get_hero>
+  <xacro:get_hero prefix="leg${limbleft}"></xacro:get_hero>
+  <xacro:get_hero prefix="leg${limbright}"></xacro:get_hero>
 </robot>

File: src/ros2_m_hero_pkg/urdf/hero_3legwheel.xacro (robot description, xacro)
@@ -12,5 +12,5 @@
 <origin xyz="0 0 0"
 rpy="0 0 0"/>
-<parent link="leg1gripper2"/>
+<parent link="leg${limbfront}gripper2"/>
 <child link="${wheelfront}in"/>
 </joint>
@@ -20,5 +20,5 @@
 <origin xyz="0 0 0"
 rpy="0 0 0"/>
-<parent link="leg2gripper2"/>
+<parent link="leg${limbleft}gripper2"/>
 <child link="${wheelleft}in"/>
 </joint>
@@ -28,5 +28,5 @@
 <origin xyz="0 0 0"
 rpy="0 0 0"/>
-<parent link="leg4gripper2"/>
+<parent link="leg${limbright}gripper2"/>
 <child link="${wheelright}in"/>
 </joint>

File: src/ros2_m_hero_pkg/urdf/hero_7dof_macro.xacro (robot description, xacro)
@@ -7,19 +7,5 @@
     <xacro:property name="MeshPath" value="package://${ThisPackage}/meshes/hero_7dof_arm/optimised" />
     <xacro:property name="mesh_extension" value="STL" />
-    <xacro:macro name="get_hero" params="prefix off_base_link_link2 off_link2_link3 off_link3_link4 off_link4_link5 off_link5_link6 off_link6_link7 off_link7_link8">
-    <xacro:property name="max_base_link_link2" value="${-1 * off_base_link_link2}" />
-    <xacro:property name="max_link2_link3" value="${-1 * off_link2_link3}" />
-    <xacro:property name="max_link3_link4" value="${-1 * off_link3_link4}" />
-    <xacro:property name="max_link4_link5" value="${-1 * off_link4_link5}" />
-    <xacro:property name="max_link5_link6" value="${-1 * off_link5_link6}" />
-    <xacro:property name="max_link6_link7" value="${-1 * off_link6_link7}" />
-    <xacro:property name="max_link7_link8" value="${-1 * off_link7_link8}" />
-    <xacro:property name="min_base_link_link2" value="${-1 * off_base_link_link2 - pi}" />
-    <xacro:property name="min_link2_link3" value="${-1 * off_link2_link3 - pi}" />
-    <xacro:property name="min_link3_link4" value="${-1 * off_link3_link4 - pi}" />
-    <xacro:property name="min_link4_link5" value="${-1 * off_link4_link5 - pi}" />
-    <xacro:property name="min_link5_link6" value="${-1 * off_link5_link6 - pi}" />
-    <xacro:property name="min_link6_link7" value="${-1 * off_link6_link7 - pi}" />
-    <xacro:property name="min_link7_link8" value="${-1 * off_link7_link8 - pi}" />
+    <xacro:macro name="get_hero" params="prefix:=leg1">
     <xacro:property name="max_vel" value="0.15" />
     <!-- PREFIX BELOW IS FOR TESTING. TODO: REMOVE -->

File: src/ros2_m_hero_pkg/urdf/hero_all.xacro (robot description, xacro)
@@ -2,7 +2,11 @@
 <robot xmlns:xacro="http://www.ros.org/wiki/xacro" name="hero_dragon">
 <xacro:property name="ThisPackage" value="urdf_packer" />
-<xacro:property name="Filename" value="hero_7dof" />
 <xacro:property name="UrdfDataPath" value="package://${ThisPackage}/urdf" />
 <link name="base_link" />
+<xacro:include filename="hero_7dof_macro.xacro"/>
+<xacro:get_hero prefix="leg1"/>
+<xacro:get_hero prefix="leg2"/>
+<xacro:get_hero prefix="leg3"/>
+<xacro:get_hero prefix="leg4"/>
 <joint name="fix1" type="fixed">
 <origin xyz="-0.6 0 0" rpy="0 0 0"/>
@@ -25,10 +29,9 @@
 <child link="leg4gripper1"/>
 </joint>
-<xacro:include filename="hero_7dofm1.xacro"/>
-<xacro:include filename="hero_7dofm2.xacro"/>
-<xacro:include filename="hero_7dofm3.xacro"/>
-<xacro:include filename="hero_7dofm4.xacro"/>
-<xacro:include filename="hero_wheel_module.xacro"/>
+<xacro:include filename="hero_wheel_macro.xacro"/>
 <xacro:add_wheel prefix="wheel11_" />
+<xacro:add_wheel prefix="wheel12_" />
+<xacro:add_wheel prefix="wheel13_" />
+<xacro:add_wheel prefix="wheel14_" />
 <joint name="fix11" type="fixed">
 <origin xyz="0 2 0" rpy="0 0 0"/>
@@ -36,5 +39,4 @@
 <child link="wheel11_in"/>
 </joint>
-<xacro:add_wheel prefix="wheel12_" />
 <joint name="fix12" type="fixed">
 <origin xyz="0.6 2 0" rpy="0 0 0"/>
@@ -42,5 +44,4 @@
 <child link="wheel12_in"/>
 </joint>
-<xacro:add_wheel prefix="wheel13_" />
 <joint name="fix13" type="fixed">
 <origin xyz="1.2 2 0" rpy="0 0 0"/>
@@ -48,5 +49,4 @@
 <child link="wheel13_in"/>
 </joint>
-<xacro:add_wheel prefix="wheel14_" />
 <joint name="fix14" type="fixed">
 <origin xyz="1.8 2 0" rpy="0 0 0"/>

File: src/ros2_m_hero_pkg/urdf/hero_dragon.xacro (robot description, xacro)
@@ -1,70 +1,13 @@
-<?xml version="1.0" encoding="UTF-8"?>
+<?xml version="1.0" encoding="utf-8"?>
 <robot name="hero_dragon" xmlns:xacro="http://www.ros.org/wiki/xacro">
-  <!-- change what leg is where -->
-  <!--  -->
-  <!--  -->
-  <xacro:property name="wheelfront" value="wheel12_"></xacro:property>
-  <xacro:property name="wheelback" value="wheel14_"></xacro:property>
-  <xacro:property name="bridge_leg" value="4"></xacro:property>
-  <!-- also change that here !!!!    V   -->
-  <xacro:include filename="hero_7dofm4.xacro"></xacro:include>
-  <xacro:property name="manip_leg" value="3"></xacro:property>
-  <!-- also change that here !!!!    V   -->
-  <xacro:include filename="hero_7dofm3.xacro"></xacro:include>
-  <!--  -->
-  <!--  -->
-  <!--  -->
-  <link name="base_link"></link>
-  <xacro:include filename="hero_wheel_module.xacro"></xacro:include>
-  <joint name="bfix" type="fixed">
-  <origin rpy="0 ${pi/4 - pi/2} ${pi}" xyz="0 0 0"></origin>
-    <parent link="base_link"></parent>
-    <child link="base_link45"></child>
-  </joint>
-  <link name="base_link45"></link>
-  <joint name="bfixstraight" type="fixed">
-    <origin rpy="0 0 0" xyz="0 0 0.160"></origin>
-    <parent link="base_link45"></parent>
-    <child link="${wheelfront}in"></child>
-  </joint>
-  <!---->
-  <!---->
-  <xacro:add_wheel prefix="${wheelfront}"></xacro:add_wheel>
-  <!-- <link name="${wheelfront}c45"></link> -->
-  <!-- <joint name="${wheelfront}fix45" type="fixed"> -->
-  <!--   <origin rpy="${-pi/4} 0 0" xyz="0 0 0"></origin> -->
-  <!--   <parent link="${wheelfront}center"></parent> -->
-  <!--   <child link="${wheelfront}c45"></child> -->
-  <!-- </joint> -->
-  <joint name="${wheelfront}fixin" type="fixed">
-    <origin rpy="0 0 0" xyz="0 0 0"></origin>
-    <parent link="${wheelfront}in"></parent>
-    <child link="leg${manip_leg}gripper1"></child>
-  </joint>
-  <!---->
-  <!---->
-  <joint name="${wheelback}fix1" type="fixed">
-    <origin rpy="0 0 ${0*pi}" xyz="0 0 0"></origin>
-    <parent link="leg${bridge_leg}gripper2"></parent>
-    <child link="${wheelback}in"></child>
-  </joint>
-  <xacro:add_wheel prefix="${wheelback}"></xacro:add_wheel>
-  <link name="${wheelback}c45"></link>
-  <joint name="fix45${wheelback}" type="fixed">
-  <origin rpy="0 -${pi/4} ${pi}" xyz="0 0 0"></origin>
-    <parent link="${wheelback}center"></parent>
-    <child link="${wheelback}c45"></child>
-  </joint>
-  <joint name="${wheelfront}fix_out" type="fixed">
-    <origin rpy="0 0 0" xyz="0 0 0"></origin>
-    <parent link="${wheelfront}out"></parent>
-    <child link="leg${bridge_leg}gripper1"></child>
-  </joint>
-  <!-- <xacro:add_wheel  prefix="${manip_leg}" /> -->
-  <!---->
-  <!-- <joint name="fixwheel1-${manip_leg}" type="fixed"> -->
-  <!-- <origin xyz="0 0 0" rpy="0 0 0"/> -->
-  <!-- <parent link="leg4gripper2"/> -->
-  <!-- <child link="${manip_leg}wheel_in"/> -->
-  <!-- </joint> -->
+  <xacro:include filename="hero_dragon_macro.xacro"></xacro:include>
+  <xacro:arg default="4" name="bridge"></xacro:arg>
+  <xacro:arg default="3" name="manip"></xacro:arg>
+  <xacro:arg default="11" name="front_wheel"></xacro:arg>
+  <xacro:arg default="12" name="back_wheel"></xacro:arg>
+  <xacro:property name="bridge_value" value="$(arg bridge)"></xacro:property>
+  <xacro:property name="manip_value" value="$(arg manip)"></xacro:property>
+  <xacro:property name="front_value" value="$(arg front_wheel)"></xacro:property>
+  <xacro:property name="back_value" value="$(arg back_wheel)"></xacro:property>
+  <xacro:dragon bridge_limb="${bridge_value}" manip_limb="${manip_value}" wheel_back="${back_value}" wheel_front="${front_value}"></xacro:dragon>
 </robot>

File: src/ros2_m_hero_pkg/urdf/hero_minimal.xacro (robot description, xacro)
@@ -1,34 +1,9 @@
 <?xml version="1.0" encoding="UTF-8"?>
-<robot name="hero_vehicle" xmlns:xacro="http://www.ros.org/wiki/xacro">
-  <!-- change what leg is where -->
-  <!--  -->
-  <!--  -->
-  <xacro:property name="wheelfront" value="wheel11_"></xacro:property>
-  <xacro:property name="bridge_leg" value="1"></xacro:property>
-  <!-- also change that here !!!!    V   -->
-  <xacro:include filename="hero_7dofm1.xacro"></xacro:include>
-  <!--  -->
-  <!--  -->
-  <!--  -->
-  <link name="base_link"></link>
-  <xacro:include filename="hero_wheel_module.xacro"></xacro:include>
-  <joint name="bfix" type="fixed">
-  <origin rpy="0 ${- pi/2} ${pi}" xyz="0 0 0"></origin>
-    <parent link="base_link"></parent>
-    <child link="base_link45"></child>
-  </joint>
-  <link name="base_link45"></link>
-  <joint name="bfixstraight" type="fixed">
-    <origin rpy="0 0 0" xyz="0 0 0.160"></origin>
-    <parent link="base_link45"></parent>
-    <child link="${wheelfront}in"></child>
-  </joint>
-  <!---->
-  <!---->
-  <xacro:add_wheel prefix="${wheelfront}"></xacro:add_wheel>
-  <joint name="${wheelfront}fix_out" type="fixed">
-    <origin rpy="0 0 0" xyz="0 0 0"></origin>
-    <parent link="${wheelfront}out"></parent>
-    <child link="leg${bridge_leg}gripper1"></child>
-  </joint>
+<robot name="minimal" xmlns:xacro="http://www.ros.org/wiki/xacro">
+  <xacro:include filename="hero_minimal_macro.xacro"></xacro:include>
+  <xacro:arg default="1" name="limb"></xacro:arg>
+  <xacro:arg default="11" name="wheel"></xacro:arg>
+  <xacro:property name="limb_val" value="$(arg limb)"></xacro:property>
+  <xacro:property name="wheel_val" value="$(arg wheel)"></xacro:property>
+  <xacro:minimal limb="${limb_val}" wheel="${wheel_val}"></xacro:minimal>
 </robot>

File: src/ros2_m_hero_pkg/urdf/hero_vehicle.xacro (robot description, xacro)
@@ -1,54 +1,11 @@
-<?xml version="1.0" encoding="UTF-8"?>
+<?xml version="1.0" encoding="utf-8"?>
 <robot name="hero_vehicle" xmlns:xacro="http://www.ros.org/wiki/xacro">
-  <!-- change what leg is where -->
-  <!--  -->
-  <!--  -->
-  <xacro:property name="wheelfront" value="wheel11_"></xacro:property>
-  <xacro:property name="wheelback" value="wheel12_"></xacro:property>
-  <xacro:property name="bridge_leg" value="1"></xacro:property>
-  <!-- also change that here !!!!    V   -->
-  <xacro:include filename="hero_7dofm1.xacro"></xacro:include>
-  <!--  -->
-  <!--  -->
-  <!--  -->
-  <link name="base_link"></link>
-  <xacro:include filename="hero_wheel_module.xacro"></xacro:include>
-  <joint name="bfix" type="fixed">
-  <origin rpy="0 ${- pi/2} ${pi}" xyz="0 0 0"></origin>
-    <parent link="base_link"></parent>
-    <child link="base_link45"></child>
-  </joint>
-  <link name="base_link45"></link>
-  <joint name="bfixstraight" type="fixed">
-    <origin rpy="0 0 0" xyz="0 0 0.160"></origin>
-    <parent link="base_link45"></parent>
-    <child link="${wheelfront}in"></child>
-  </joint>
-  <!---->
-  <!---->
-  <xacro:add_wheel prefix="${wheelfront}"></xacro:add_wheel>
-  <joint name="${wheelback}fix1" type="fixed">
-    <origin rpy="0 0 ${0*pi}" xyz="0 0 0"></origin>
-    <parent link="leg${bridge_leg}gripper2"></parent>
-    <child link="${wheelback}in"></child>
-  </joint>
-  <xacro:add_wheel prefix="${wheelback}"></xacro:add_wheel>
-  <link name="${wheelback}c45"></link>
-  <joint name="fix45${wheelback}" type="fixed">
-    <origin rpy="${0} 0 0" xyz="0 0 0"></origin>
-    <parent link="${wheelback}center"></parent>
-    <child link="${wheelback}c45"></child>
-  </joint>
-  <joint name="${wheelfront}fix_out" type="fixed">
-    <origin rpy="0 0 0" xyz="0 0 0"></origin>
-    <parent link="${wheelfront}out"></parent>
-    <child link="leg${bridge_leg}gripper1"></child>
-  </joint>
-  <!-- <xacro:add_wheel  prefix="${manip_leg}" /> -->
-  <!---->
-  <!-- <joint name="fixwheel1-${manip_leg}" type="fixed"> -->
-  <!-- <origin xyz="0 0 0" rpy="0 0 0"/> -->
-  <!-- <parent link="leg4gripper2"/> -->
-  <!-- <child link="${manip_leg}wheel_in"/> -->
-  <!-- </joint> -->
+  <xacro:include filename="hero_vehicle_macro.xacro"></xacro:include>
+  <xacro:arg default="1" name="limb"></xacro:arg>
+  <xacro:arg default="11" name="front_wheel"></xacro:arg>
+  <xacro:arg default="12" name="back_wheel"></xacro:arg>
+  <xacro:property name="bridge_value" value="$(arg limb)"></xacro:property>
+  <xacro:property name="front_value" value="$(arg front_wheel)"></xacro:property>
+  <xacro:property name="back_value" value="$(arg back_wheel)"></xacro:property>
+  <xacro:vehicle bridge_limb="${bridge_value}" wheel_back="${back_value}" wheel_front="${front_value}"></xacro:vehicle>
 </robot>
