Commit message: dragon 45deg fixed

File: src/ros2_m_hero_pkg/urdf/hero_dragon.xacro (robot description, xacro)
@@ -52,5 +52,5 @@
   <link name="${wheelback}c45"></link>
   <joint name="fix45${wheelback}" type="fixed">
-    <origin rpy="${pi/4} 0 0" xyz="0 0 0"></origin>
+  <origin rpy="0 -${pi/4} ${pi}" xyz="0 0 0"></origin>
     <parent link="${wheelback}center"></parent>
     <child link="${wheelback}c45"></child>

Commit message: automated urdf

File: src/ros2_m_hero_pkg/urdf/hero_dragon.xacro (robot description, xacro)
@@ -2,6 +2,6 @@
 <robot name="hero_dragon" xmlns:xacro="http://www.ros.org/wiki/xacro">
   <xacro:include filename="hero_dragon_macro.xacro"></xacro:include>
-  <xacro:arg default="4" name="bridge"></xacro:arg>
-  <xacro:arg default="3" name="manip"></xacro:arg>
+  <xacro:arg default="1" name="bridge"></xacro:arg>
+  <xacro:arg default="2" name="manip"></xacro:arg>
   <xacro:arg default="11" name="front_wheel"></xacro:arg>
   <xacro:arg default="12" name="back_wheel"></xacro:arg>
@@ -10,4 +10,5 @@
   <xacro:property name="front_value" value="$(arg front_wheel)"></xacro:property>
   <xacro:property name="back_value" value="$(arg back_wheel)"></xacro:property>
+  <!-- <xacro:dragon bridge_limb="${bridge_value}" manip_limb="${manip_value}" wheel_back="${back_value}" wheel_front="${front_value}"></xacro:dragon> -->
   <xacro:dragon bridge_limb="${bridge_value}" manip_limb="${manip_value}" wheel_back="${back_value}" wheel_front="${front_value}"></xacro:dragon>
 </robot>

File: src/ros2_m_hero_pkg/urdf/hero_dragon_macro.xacro (robot description, xacro)
@@ -1,5 +1,5 @@
 <?xml version="1.0" encoding="UTF-8"?>
 <robot name="dragon" xmlns:xacro="http://www.ros.org/wiki/xacro">
-  <xacro:macro name="dragon" params="bridge_limb:=4 manip_limb:=3 wheel_front:=11 wheel_back:=12 ">
+  <xacro:macro name="dragon" params="bridge_limb:=1 manip_limb:=2 wheel_front:=11 wheel_back:=12 ">
     <xacro:property name="wheel_front_pre" value="wheel${wheel_front}_"></xacro:property>
     <xacro:property name="wheel_back_pre" value="wheel${wheel_back}_"></xacro:property>
@@ -22,13 +22,4 @@
       <child link="${wheel_front_pre}in"></child>
     </joint>
-    <!---->
-    <!---->
-    <xacro:add_wheel prefix="${wheel_front_pre}"></xacro:add_wheel>
-    <!-- <link name="${wheel_front_pre}c45"></link> -->
-    <!-- <joint name="${wheel_front_pre}fix45" type="fixed"> -->
-    <!--   <origin rpy="${-pi/4} 0 0" xyz="0 0 0"></origin> -->
-    <!--   <parent link="${wheel_front_pre}center"></parent> -->
-    <!--   <child link="${wheel_front_pre}c45"></child> -->
-    <!-- </joint> -->
     <joint name="${wheel_front_pre}fixin" type="fixed">
       <origin rpy="0 0 0" xyz="0 0 0"></origin>
@@ -36,6 +27,4 @@
       <child link="leg${manip_limb}gripper1"></child>
     </joint>
-    <!---->
-    <!---->
     <joint name="${wheel_back_pre}fix1" type="fixed">
       <origin rpy="0 0 ${0*pi}" xyz="0 0 0"></origin>
@@ -43,5 +32,4 @@
       <child link="${wheel_back_pre}in"></child>
     </joint>
-    <xacro:add_wheel prefix="${wheel_back_pre}"></xacro:add_wheel>
     <link name="${wheel_back_pre}c45"></link>
     <joint name="fix45${wheel_back_pre}" type="fixed">
@@ -55,11 +43,4 @@
       <child link="leg${bridge_limb}gripper1"></child>
     </joint>
-    <!-- <xacro:add_wheel  prefix="${manip_limb}" /> -->
-    <!---->
-    <!-- <joint name="fixwheel1-${manip_limb}" type="fixed"> -->
-    <!-- <origin xyz="0 0 0" rpy="0 0 0"/> -->
-    <!-- <parent link="leg4gripper2"/> -->
-    <!-- <child link="${manip_limb}wheel_in"/> -->
-    <!-- </joint> -->
   </xacro:macro>
 </robot>

File: src/ros2_m_hero_pkg/urdf/hero_minimal.xacro (robot description, xacro)
@@ -7,3 +7,9 @@
   <xacro:property name="wheel_val" value="$(arg wheel)"></xacro:property>
   <xacro:minimal limb="${limb_val}" wheel="${wheel_val}"></xacro:minimal>
+  <link name="base_link"/>
+  <joint name="base_fix" type="fixed">
+    <origin rpy="0 0 0" xyz="0 0 0"></origin>
+    <parent link="base_link"></parent>
+    <child link="leg${limb_val}gripper1"></child>
+  </joint>
 </robot>

File: src/ros2_m_hero_pkg/urdf/hero_minimal_macro.xacro (robot description, xacro)
@@ -3,27 +3,13 @@
   <xacro:macro name="minimal" params="limb:=1 wheel:=11">
   <xacro:include filename="hero_wheel_macro.xacro"></xacro:include>
-  <xacro:property name="wheelfront" value="wheel${wheel}_"></xacro:property>
-  <xacro:add_wheel prefix="${wheelfront}"></xacro:add_wheel>
+  <xacro:property name="wheel_pre" value="wheel${wheel}_"></xacro:property>
+  <xacro:add_wheel prefix="${wheel_pre}"></xacro:add_wheel>
   <xacro:include filename="hero_7dof_macro.xacro"></xacro:include>
   <xacro:property name="bridge_leg" value="${limb}"></xacro:property>
   <xacro:get_hero prefix="leg${limb}"></xacro:get_hero>
-  <link name="base_link"></link>
-  <joint name="bfix" type="fixed">
-  <origin rpy="0 ${- pi/2} ${pi}" xyz="0 0 0"></origin>
-    <parent link="base_link"></parent>
-    <child link="base_link45"></child>
-  </joint>
-  <link name="base_link45"></link>
-  <joint name="bfixstraight" type="fixed">
-    <origin rpy="0 0 0" xyz="0 0 0.160"></origin>
-    <parent link="base_link45"></parent>
-    <child link="${wheelfront}in"></child>
-  </joint>
-  <!---->
-  <!---->
-  <joint name="${wheelfront}fix_out" type="fixed">
+  <joint name="leg${bridge_leg}_${wheel_pre}_fix" type="fixed">
     <origin rpy="0 0 0" xyz="0 0 0"></origin>
-    <parent link="${wheelfront}out"></parent>
-    <child link="leg${bridge_leg}gripper1"></child>
+    <parent link="leg${bridge_leg}gripper2"></parent>
+    <child link="${wheel_pre}in"></child>
   </joint>
   </xacro:macro>

File: src/ros2_m_hero_pkg/urdf/hero_tricycle.xacro (robot description, xacro)
@@ -22,3 +22,9 @@
   right_wheel="${right_wheel_val}"
   ></xacro:tricycle>
+  <link name="base_link"/>
+  <joint name="base_fix" type="fixed">
+    <origin rpy="0 0 0" xyz="0 0 0"></origin>
+    <parent link="base_link"></parent>
+    <child link="tri_body"></child>
+  </joint>
 </robot>

File: src/ros2_m_hero_pkg/urdf/hero_tricycle_macro.xacro (robot description, xacro)
@@ -1,13 +1,13 @@
 <?xml version="1.0" encoding="UTF-8"?>
 <robot name="hero_tricycle" xmlns:xacro="http://www.ros.org/wiki/xacro">
+  <xacro:macro name="tricycle" params="front_limb:=1 left_limb:=2 right_limb:=3 front_wheel:=11 left_wheel:=12 right_wheel:=13">
     <xacro:property name="ThisPackage" value="ros2_m_hero_pkg" />
-    <xacro:property name="MeshPath" value="package://${ThisPackage}/meshes/hero_7dof_arm/optimised" />
+    <xacro:property name="MeshPath" value="package://${ThisPackage}/meshes" />
   <xacro:property name="body_radius" value="0.200"></xacro:property>
     <xacro:include filename="hero_minimal_macro.xacro"></xacro:include>
-  <xacro:macro name="tricycle" params="front_limb:=1 left_limb:=2 right_limb:=3 front_wheel:=11 left_wheel:=12 right_wheel:=13">
     <xacro:minimal limb="${front_limb}" wheel="${front_wheel}"></xacro:minimal>
     <xacro:minimal limb="${left_limb}" wheel="${left_wheel}"></xacro:minimal>
     <xacro:minimal limb="${right_limb}" wheel="${right_wheel}"></xacro:minimal>
-    <link name="base_link">
+    <link name="tri_body">
       <visual>
         <origin rpy="0 0 1.04" xyz="0 0 0"></origin>
@@ -25,5 +25,5 @@
     <joint name="orient1" type="fixed">
       <origin rpy="${pi/2} 0 0" xyz="0 0 0"></origin>
-      <parent link="base_link"></parent>
+      <parent link="tri_body"></parent>
       <child link="d1"></child>
     </joint>
@@ -37,5 +37,5 @@
     <joint name="orient2" type="fixed">
       <origin rpy="${pi/2} 0 ${2*pi/3}" xyz="0 0 0"></origin>
-      <parent link="base_link"></parent>
+      <parent link="tri_body"></parent>
       <child link="d2"></child>
     </joint>
@@ -43,5 +43,5 @@
     <joint name="orient3" type="fixed">
       <origin rpy="${pi/2} 0 ${2*2*pi/3}" xyz="0 0 0"></origin>
-      <parent link="base_link"></parent>
+      <parent link="tri_body"></parent>
       <child link="d3"></child>
     </joint>

File: src/ros2_m_hero_pkg/urdf/hero_vehicle.xacro (robot description, xacro)
@@ -2,8 +2,8 @@
 <robot name="hero_vehicle" xmlns:xacro="http://www.ros.org/wiki/xacro">
   <xacro:include filename="hero_vehicle_macro.xacro"></xacro:include>
-  <xacro:arg default="1" name="limb"></xacro:arg>
+  <xacro:arg default="1" name="bridge"></xacro:arg>
   <xacro:arg default="11" name="front_wheel"></xacro:arg>
   <xacro:arg default="12" name="back_wheel"></xacro:arg>
-  <xacro:property name="bridge_value" value="$(arg limb)"></xacro:property>
+  <xacro:property name="bridge_value" value="$(arg bridge)"></xacro:property>
   <xacro:property name="front_value" value="$(arg front_wheel)"></xacro:property>
   <xacro:property name="back_value" value="$(arg back_wheel)"></xacro:property>

File: src/ros2_m_hero_pkg/urdf/hero_wheel.xacro (robot description, xacro)
@@ -6,3 +6,9 @@
   <xacro:property name="number_value" value="$(arg number)"></xacro:property>
   <xacro:add_wheel prefix="wheel${number_value}_"/>
+  <link name="base_link"/>
+  <joint name="base_fix" type="fixed">
+    <origin rpy="0 0 0" xyz="0 0 0"></origin>
+    <parent link="base_link"></parent>
+    <child link="wheel${limb_val}_in"></child>
+  </joint>
 </robot>

File: src/ros2_m_hero_pkg/urdf/hero_wheel_macro.xacro (robot description, xacro)
@@ -4,8 +4,8 @@
      For more information, please see http://wiki.ros.org/sw_urdf_exporter -->
 <robot xmlns:xacro="http://www.ros.org/wiki/xacro" name="hero_wheel_module">
+  <xacro:macro name="add_wheel" params="prefix:=11">
   <xacro:property name="ThisPackage" value="ros2_m_hero_pkg" />
   <xacro:property name="MeshPath" value="package://${ThisPackage}/meshes/hero_wheel_module/optimised" />
   <xacro:property name="mesh_extension" value="STL" />
-  <xacro:macro name="add_wheel" params="prefix">
   <!-- PREFIX BELOW IS FOR TESTING. TODO: REMOVE -->
   <!-- <xacro:property name="prefix" value = "wm1"/> -->
