Commit message: urdf minifix and deleted old

File: src/ros2_m_hero_pkg/urdf/hero_wheel.xacro (robot description, xacro)
@@ -10,5 +10,5 @@
     <origin rpy="0 0 0" xyz="0 0 0"></origin>
     <parent link="base_link"></parent>
-    <child link="wheel${limb_val}_in"></child>
+    <child link="wheel${number_value}_in"></child>
   </joint>
 </robot>
