Commit message: realsense xmacro update

File: src/ros2_m_hero_pkg/urdf/hero_dragon_realsense.xacro (robot description, xacro)
@@ -4,6 +4,6 @@
     <xacro:include filename="hero_dragon.xacro"></xacro:include>
     <xacro:include filename="realsense_macro.xacro"></xacro:include>
-    <xacro:realsense_d435i parent_link='leg4gripper2'
-                           camera_xyz='0.08 -0.01 0.02'
-                           camera_rpy='${PI} ${PI/2} 0'/>
+    <xacro:realsense_d435i parent_link="leg${manip_value}gripper2"
+                           camera_xyz='-0.01 0.06 0.02'
+    camera_rpy='${-pi/2} ${pi/2} 0'/>
 </robot>

File: src/ros2_m_hero_pkg/urdf/realsense_macro.xacro (robot description, xacro)
@@ -6,5 +6,5 @@
     <joint name="robot_to_camera_joint" type="fixed">
       <origin xyz="${camera_xyz}" rpy="${camera_rpy}"/>
-      <parent link="leg4gripper2"/>
+      <parent link="${parent_link}"/>
       <child link="robot_to_camera_link"/>
     </joint>
