Commit message: not much

File: src/ros2_m_hero_pkg/urdf/hero_7dof_macro.xacro (robot description, xacro)
@@ -6,4 +6,5 @@
     <xacro:property name="ThisPackage" value="ros2_m_hero_pkg" />
     <xacro:property name="MeshPath" value="package://${ThisPackage}/meshes/hero_7dof_arm/optimised" />
+    <!-- <xacro:property name="MeshPath" value="package://${ThisPackage}/meshes/hero_7dof_arm/raw" /> -->
     <xacro:property name="mesh_extension" value="STL" />
     <xacro:macro name="get_hero" params="prefix:=leg1">

File: src/ros2_m_hero_pkg/urdf/hero_dragon.xacro (robot description, xacro)
@@ -10,5 +10,4 @@
   <xacro:property name="front_value" value="$(arg front_wheel)"></xacro:property>
   <xacro:property name="back_value" value="$(arg back_wheel)"></xacro:property>
-  <!-- <xacro:dragon bridge_limb="${bridge_value}" manip_limb="${manip_value}" wheel_back="${back_value}" wheel_front="${front_value}"></xacro:dragon> -->
   <xacro:dragon bridge_limb="${bridge_value}" manip_limb="${manip_value}" wheel_back="${back_value}" wheel_front="${front_value}"></xacro:dragon>
 </robot>

File: src/ros2_m_hero_pkg/urdf/hero_wheel_macro.xacro (robot description, xacro)
@@ -7,4 +7,5 @@
   <xacro:property name="ThisPackage" value="ros2_m_hero_pkg" />
   <xacro:property name="MeshPath" value="package://${ThisPackage}/meshes/hero_wheel_module/optimised" />
+  <!-- <xacro:property name="MeshPath" value="package://${ThisPackage}/meshes/hero_wheel_module/raw" /> -->
   <xacro:property name="mesh_extension" value="STL" />
   <!-- PREFIX BELOW IS FOR TESTING. TODO: REMOVE -->

Commit message: update

File: src/ros2_m_hero_pkg/urdf/hero_7dof_macro.xacro (robot description, xacro)
@@ -5,5 +5,5 @@
 <robot xmlns:xacro="http://www.ros.org/wiki/xacro" name="hero_7dof_arm">
     <xacro:property name="ThisPackage" value="ros2_m_hero_pkg" />
-    <xacro:property name="MeshPath" value="package://${ThisPackage}/meshes/hero_7dof_arm/optimised" />
+    <xacro:property name="MeshPath" value="package://${ThisPackage}/meshes/hero_7dof_arm/raw" />
     <xacro:property name="mesh_extension" value="STL" />
     <xacro:macro name="get_hero" params="prefix:=leg1">

File: src/ros2_m_hero_pkg/urdf/hero_wheel_macro.xacro (robot description, xacro)
@@ -6,5 +6,5 @@
   <xacro:macro name="add_wheel" params="prefix:=11">
   <xacro:property name="ThisPackage" value="ros2_m_hero_pkg" />
-  <xacro:property name="MeshPath" value="package://${ThisPackage}/meshes/hero_wheel_module/optimised" />
+  <xacro:property name="MeshPath" value="package://${ThisPackage}/meshes/hero_wheel_module/raw" />
   <xacro:property name="mesh_extension" value="STL" />
   <!-- PREFIX BELOW IS FOR TESTING. TODO: REMOVE -->

Commit message: ns method

File: src/ros2_m_hero_pkg/urdf/hero_7dof_macro.xacro (robot description, xacro)
@@ -274,26 +274,4 @@
         <limit lower="-9999" upper="9999" effort="9999" velocity="${max_vel}" />
     </joint>
-    <link name="${prefix}gripper2_base">
-        <inertial>
-            <origin xyz="0 0 0.034092" rpy="0 0 0" />
-            <mass value="1" />
-            <inertia ixx="0.00037818" ixy="-7.3501E-08" ixz="9.8348E-07" iyy="0.0011423" iyz="1.9396E-08" izz="0.0012608" />
-        </inertial>
-        <visual>
-            <origin xyz="0 0 0" rpy="0 0 0" />
-            <geometry>
-                <mesh filename="${MeshPath}/gripper_base.${mesh_extension}" />
-            </geometry>
-            <material name="">
-                <color rgba="0.79216 0.81961 0.93333 1" />
-            </material>
-        </visual>
-        <collision>
-            <origin xyz="0 0 0" rpy="0 0 0" />
-            <geometry>
-                <mesh filename="${MeshPath}/gripper_base.${mesh_extension}" />
-            </geometry>
-        </collision>
-    </link>
     <joint name="${prefix}joint7" type="continuous">
     <origin xyz="0.1646 0 0.072902" rpy="${-pi/2} 0 ${-pi/2}" />
@@ -303,4 +281,26 @@
         <limit lower="-9999" upper="9999" effort="9999" velocity="${max_vel}" />
     </joint>
+    <link name="${prefix}gripper2_base">
+        <inertial>
+            <origin xyz="0 0 0.034092" rpy="0 0 0" />
+            <mass value="1" />
+            <inertia ixx="0.00037818" ixy="-7.3501E-08" ixz="9.8348E-07" iyy="0.0011423" iyz="1.9396E-08" izz="0.0012608" />
+        </inertial>
+        <visual>
+            <origin xyz="0 0 0" rpy="0 0 0" />
+            <geometry>
+                <mesh filename="${MeshPath}/gripper_base.${mesh_extension}" />
+            </geometry>
+            <material name="">
+                <color rgba="0.79216 0.81961 0.93333 1" />
+            </material>
+        </visual>
+        <collision>
+            <origin xyz="0 0 0" rpy="0 0 0" />
+            <geometry>
+                <mesh filename="${MeshPath}/gripper_base.${mesh_extension}" />
+            </geometry>
+        </collision>
+    </link>
     <link name="${prefix}gripper2_jaw_left">
         <inertial>
