Commit message: renamed tuto, docs and auto pakge ms

File: src/motion_stack_tuto/urdf/moonbot_zero.xacro (robot description, xacro)
@@ -1,5 +1,5 @@
 <?xml version="1.0" ?>
 <robot name="moonbot_zero" xmlns:xacro="http://www.ros.org/wiki/xacro">
-<xacro:property name="ThisPackage" value="moonbot_zero_tuto" />
+<xacro:property name="ThisPackage" value="motion_stack_tuto" />
 <xacro:property name="UrdfDataPath" value="package://${ThisPackage}/urdf" />
 <xacro:property name="MeshPath" value="package://${ThisPackage}/meshes" />
